Commit message: modified pelvis IMU rpy

File: alexander-models/alexander_V1_description/urdf/alexander_v1.lowerBodyOnly.urdf (robot description, URDF)
Before this commit: robot Alexander, 23 links, 22 joints
Joints:
- joint LEFT_THIGH_IMU_JOINT: origin xyz=0.10004 0.03746 -0.21194 rpy=1.6947717585 0 1.570796 -> xyz=0.10004 0.03746 -0.21194 rpy=1.437982 0 1.570796
- joint PELVIS_STIM_IMU_JOINT: origin xyz=-0.08687724 0.01225028 -0.08051472 rpy=0.0 0.0 1.570796 -> xyz=-0.08687724 0.01225028 -0.08051472 rpy=-0.01399 -0.013054 1.570796

Commit message: updated individual body part urdfs to include IMU information

File: alexander-models/alexander_V1_description/urdf/alexander_v1.lowerBodyOnly.urdf (robot description, URDF)
Before this commit: robot Alexander, 23 links, 22 joints
Links:
- added link TORSO_IMU_LINK, mass 0
Joints:
- added joint TORSO_IMU_JOINT: type fixed, parent TORSO_LINK, child TORSO_IMU_LINK, origin xyz=0.0 0.0 0.0 rpy=0.0 0 0.0, axis 0 0 1

Commit message: updated torso mass to include delta between expected and measured whole robot mass. scaled inertias too

File: alexander-models/alexander_V1_description/urdf/alexander_v1.lowerBodyOnly.urdf (robot description, URDF)
Before this commit: robot Alexander, 24 links, 23 joints
Links:
- link TORSO_LINK: mass 4.352 -> 7.0081
