Commit message: did some general URDF cleanup

File: alexander-models/alexander_V1_description/urdf/alexander_v1.leftUpperArm.urdf (robot description, URDF)
Before this commit: robot Alexander, 6 links, 6 joints
Links:
- removed link LEFT_ELBOW_PITCH_LINK
Joints:
- removed joint LEFT_ELBOW_Y

File: alexander-models/alexander_V1_description/urdf/alexander_v1.lowerBody.urdf (robot description, URDF)
Before this commit: robot Alexander, 24 links, 23 joints
Links:
- link TORSO_IMU_LINK: mass 0.0 -> 0
- link TORSO_LINK: mass 4.806 -> 7.0081
Joints:
- joint TORSO_IMU_JOINT: axis (none) -> 0 0 1; origin xyz=0.04529 -0.02427 0.33757 rpy=3.141592 0 0 -> xyz=0.0 0.0 0.0 rpy=0.0 0 0.0

File: alexander-models/alexander_V1_description/urdf/alexander_v1.rightUpperArm.urdf (robot description, URDF)
Before this commit: robot Alexander, 6 links, 6 joints
Links:
- removed link RIGHT_ELBOW_PITCH_LINK
Joints:
- removed joint RIGHT_ELBOW_Y
