Commit message: Feature/alexander long (#38)
* did some general URDF cleanup

* set up a long bicep version

File: alexander-models/alexander_V1_description/urdf/alexander_v1.rightLongUpperArm.urdf (robot description, URDF)
Before this commit: robot Alexander, 6 links, 6 joints
Links:
- removed link RIGHT_ELBOW_PITCH_LINK
- link RIGHT_SHOULDER_X_LINK: mass 0.972 -> 1.17068
Joints:
- removed joint RIGHT_ELBOW_Y
- joint RIGHT_SHOULDER_Z: origin xyz=0.0 -0.035 0.0 rpy=0.0 0.0 0.0 -> xyz=0.0 -0.035 -0.08 rpy=0.0 0.0 0.0
