Commit message: Updated urdf formatting and made full body w hands vs nubs

File: alexander-models/alexander_V1_description/urdf/alexander_v1.fullBodyNubForearms.urdf (robot description, URDF)
Before this commit: robot Alexander, 51 links, 50 joints
Links:
- removed link LEFT_GRIPPER_ATTACHMENT_FIXED_LINK
- removed link LEFT_GRIPPER_YAW_IMU_LINK
- removed link LEFT_GRIPPER_Z_LINK
- removed link LEFT_WRIST_X_LINK
- removed link LEFT_WRIST_YAW_IMU_LINK
- removed link LEFT_WRIST_Z_LINK
- removed link RIGHT_GRIPPER_ATTACHMENT_FIXED_LINK
- removed link RIGHT_GRIPPER_YAW_IMU_LINK
- removed link RIGHT_GRIPPER_Z_LINK
- removed link RIGHT_WRIST_X_LINK
- removed link RIGHT_WRIST_YAW_IMU_LINK
- removed link RIGHT_WRIST_Z_LINK
- link LEFT_ELBOW_Y_LINK: mass 0.45 -> 0.616; geometry visual mesh filename=package://alexander_V1_description/meshes/cycloidal_arm/LEF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
- link LEFT_SHOULDER_X_LINK: mass 0.972 -> 1.17068
- link RIGHT_ELBOW_Y_LINK: mass 0.45 -> 0.616; geometry visual mesh filename=package://alexander_V1_description/meshes/cycloidal_arm/RIG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
- link RIGHT_SHOULDER_X_LINK: mass 0.972 -> 1.17068
Joints:
- removed joint LEFT_GRIPPER_ATTACHMENT_FIXED
- removed joint LEFT_GRIPPER_YAW_IMU_JOINT
- removed joint LEFT_GRIPPER_Z
- removed joint LEFT_WRIST_X
- removed joint LEFT_WRIST_YAW_IMU_JOINT
- removed joint LEFT_WRIST_Z
- removed joint RIGHT_GRIPPER_ATTACHMENT_FIXED
- removed joint RIGHT_GRIPPER_YAW_IMU_JOINT
- removed joint RIGHT_GRIPPER_Z
- removed joint RIGHT_WRIST_X
- removed joint RIGHT_WRIST_YAW_IMU_JOINT
- removed joint RIGHT_WRIST_Z

File: alexander-models/alexander_V1_description/urdf/alexander_v1.head.urdf (robot description, URDF)
Before this commit: robot Alexander, 3 links, 3 joints
Joints:
- joint HEAD_IMU_JOINT: origin xyz=0.0 0.0 0.0 rpy=0.0 0 0.0 -> xyz=0.040556 -0.14155 0.057016 rpy=0.0 0 0.0

File: alexander-models/alexander_V1_description/urdf/alexander_v1.leftFixedForearm.urdf (robot description, URDF)
Before this commit: robot Alexander, 1 links, 1 joints
Links:
- removed link LEFT_ELBOW_PITCH_LINK
- added link LEFT_ELBOW_Y_LINK, mass 0.616; visual mesh filename=package://alexander_V1_description/meshes/cycloidal_arm/LEF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
Joints:
- joint LEFT_ELBOW_Y: child LEFT_ELBOW_PITCH_LINK -> LEFT_ELBOW_Y_LINK

File: alexander-models/alexander_V1_description/urdf/alexander_v1.rightFixedForearm.urdf (robot description, URDF)
Before this commit: robot Alexander, 1 links, 1 joints
Links:
- removed link RIGHT_ELBOW_PITCH_LINK
- added link RIGHT_ELBOW_Y_LINK, mass 0.616; visual mesh filename=package://alexander_V1_description/meshes/cycloidal_arm/RIG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
Joints:
- joint RIGHT_ELBOW_Y: child RIGHT_ELBOW_PITCH_LINK -> RIGHT_ELBOW_Y_LINK

Commit message: Missing z offset for shoulder z on full body nub arms urdf

File: alexander-models/alexander_V1_description/urdf/alexander_v1.fullBodyNubForearms.urdf (robot description, URDF)
Before this commit: robot Alexander, 39 links, 38 joints
Joints:
- joint LEFT_SHOULDER_Z: origin xyz=0.0 0.035 0.0 rpy=0.0 0.0 0.0 -> xyz=0.0 0.035 -0.08 rpy=0.0 0.0 0.0
- joint RIGHT_SHOULDER_Z: origin xyz=0.0 -0.035 0.0 rpy=0.0 0.0 0.0 -> xyz=0.0 -0.035 -0.08 rpy=0.0 0.0 0.0

Commit message: Adding collisions

File: alexander-models/alexander_V1_description/urdf/alexander_v1.fullBodyNubForearms.urdf (robot description, URDF)
Before this commit: robot Alexander, 39 links, 38 joints
Links:
- link PELVIS_LINK: geometry collision box size=0.15 0.10 0.12; visual mesh filename=package://alexander_V1_description/meshes/legs/Pelvis.obj
- link RIGHT_FOOT: geometry collision box size=0.22 0.1 0.02; visual mesh filename=package://alexander_V1_description/meshes/legs/Foot.obj

Commit message: Changed to x y z naming on urdfs and xmls

File: alexander-models/alexander_V1_description/urdf/alexander_v1.fullBodyNubForearms.urdf (robot description, URDF)
Before this commit: robot Alexander, 39 links, 38 joints
Links:
- removed link PELVIS_STIM_IMU_LINK
- added link PELVIS_IMU_LINK, mass 0.0
Joints:
- removed joint PELVIS_STIM_IMU_JOINT
- added joint PELVIS_IMU_JOINT: type fixed, parent PELVIS_LINK, child PELVIS_IMU_LINK, origin xyz=-0.08687724 0.01225028 -0.08051472 rpy=-0.01399 -0.013054 1.570796

Commit message: Merge/ahs to develop 08152025 (#39)
* updated FT offsets for left FT

* Fixed ankle RoM issues

* Added scalars to FTs

* changed gear ratios for actuator packages to measured exact ones. set default damping compensation scalar to 0.0

* Feature/use mahony gyro bias (#31)

* Added mahony filter biases to the xmls

* Fixed angular velocity bias names

* updated angular vel IMU biases in xml

---------

Co-authored-by: Biomech OCU <jli@ihmc.org>

* fixed neck cycloid manager in torso xml from pitch to yaw

* Feature/urdf update (#33)

* updated the urdf model a bit

* moved torso CoM offset

* modified pelvis IMU rpy

* Modified imu origins in lowerBody

---------

Co-authored-by: Robert <rgriffin@ihmc.org>
Co-authored-by: Stefan Fasano <sfasano@ihmc.org>
Co-authored-by: Biomech OCU <jli@ihmc.org>

* Feature/adding arms (#36)

* Added information for arms and split arms into fore and aft

* Updated all the joint limits and added new cycloid configs

* Modified xmls to check if using latest codes for twitters, formatting for ethersnacks

* Added imus to arms, switched to nadia ethersnacks boards

* added some imu definitions into urdf. added missing things into xml. reversed motor directions for right J1 and J4

* updated individual body part urdfs to include IMU information

* added raw zero offsets to xmls for arms and neck actuators

* updated torso mass to include delta between expected and measured whole robot mass. scaled inertias too

* Fixed xml names for upper arm

---------

Co-authored-by: Biomech OCU <jli@ihmc.org>
Co-authored-by: Alexander OCU <rpeterson@ihmc.org>

* Adding pelvis imu orientation offset to fullbody urdf

* Prep for creating initial release of ihmc-common-hardware (#32)

* Altered cycloid mechanism name in xml

* Changed xml descriptions for cycloids in arms

* Modified names of xml cycloid mechanisms

---------

Co-authored-by: Biomech OCU <jli@ihmc.org>
Co-authored-by: Stefan Fasano <sfasano@ihmc.org>

* Merge/develop to ahs 08132025 (#37)

* Retopologized meshes (#35)

* Swapping in retopologized meshes and increasing diffuse of mtl's.

* Replace .g3djs with new .glbs from Louis.

* Capitalizing Pelvis obj

---------

Co-authored-by: Duncan Calvert <dcalvert@ihmc.org>

* Added imus for forearm to full body urdf

* Altered masses of full body urdf to match edits in lower body

* Feature/alexander long (#38)

* did some general URDF cleanup

* set up a long bicep version

---------

Co-authored-by: Stephen McCrory <smccrory@ihmc.us>
Co-authored-by: Duncan Calvert <dcalvert@ihmc.org>
Co-authored-by: Robert Griffin <rjgriffin42@gmail.com>

* Added angular velocity biases

* Fixed upper arm encoder offsets

* Updated urdf formatting and made full body w hands vs nubs

* Updated urdf formatting and made full body w hands vs nubs

* Updated Hand Submodules (#30)

* Updated hand submodules

* Use ihmc_hands_ros2

* Merge/develop to ahs 08132025 (#37)

* Retopologized meshes (#35)

* Swapping in retopologized meshes and increasing diffuse of mtl's.

* Replace .g3djs with new .glbs from Louis.

* Capitalizing Pelvis obj

---------

Co-authored-by: Duncan Calvert <dcalvert@ihmc.org>

* Added imus for forearm to full body urdf

* Altered masses of full body urdf to match edits in lower body

* Feature/alexander long (#38)

* did some general URDF cleanup

* set up a long bicep version

---------

Co-authored-by: Stephen McCrory <smccrory@ihmc.us>
Co-authored-by: Duncan Calvert <dcalvert@ihmc.org>
Co-authored-by: Robert Griffin <rjgriffin42@gmail.com>

* Missed some merge conflicts

* Missing z offset for shoulder z on full body nub arms urdf

* Fixed material appearance issues for long biceps

* Updated MuJoCo XMLs to match URDFs.

* resetting ankle motor kt to spreadsheet

* resetting ankle motor kt to spreadsheet

* Adding collisions

* Fixed difference in inertia positions for shoulder z

* Fixed difference in inertia positions for shoulder z

* Added collisions to nubs

* Fixed head imu orientation and position

* Fixed head IMU position and orientation in mujoco files

* Fixed some of the positions of shoulder y, neck z, neck y, and the visual torso link

* Updated MuJoCo XMLs to match URDFs.

* Increased the torque break freqs to 100 Hz

* Fixed neck y y offset

* Increased the torque break freqs to 100 Hz

* Fixed neck y y offset

* Fixed head y position in mujoco files

* Fixed some incorrect link names, fixed formatting

* Finally fixed naming convention from ROLL PITCH YAW links, IMUs, to X Y Z links, IMUs

* Fixed right shoulder z inertias

* Fixed IMU names to match x y z link convention

* Changed to x y z naming on urdfs and xmls

---------

Co-authored-by: Stefan Fasano <sfasano@ihmc.org>
Co-authored-by: Biomech OCU <jli@ihmc.org>
Co-authored-by: Stefan <161661671+stefanfasano@users.noreply.github.com>
Co-authored-by: Robert <rgriffin@ihmc.org>
Co-authored-by: Stephen McCrory <smccrory@ihmc.us>
Co-authored-by: Duncan Calvert <dcalvert@ihmc.org>
Co-authored-by: Robert Griffin <rjgriffin42@gmail.com>
Co-authored-by: Tomasz Bialek <103042423+TomaszTB@users.noreply.github.com>
Co-authored-by: jeh15 <jeh15@fsu.edu>

File: alexander-models/alexander_V1_description/urdf/alexander_v1.fullBodyNubForearms.urdf (robot description, URDF)
Before this commit: robot Alexander, 51 links, 50 joints
Links:
- removed link LEFT_GRIPPER_ATTACHMENT_FIXED_LINK
- removed link LEFT_GRIPPER_Z_IMU_LINK
- removed link LEFT_GRIPPER_Z_LINK
- removed link LEFT_WRIST_X_LINK
- removed link LEFT_WRIST_Z_IMU_LINK
- removed link LEFT_WRIST_Z_LINK
- removed link RIGHT_GRIPPER_ATTACHMENT_FIXED_LINK
- removed link RIGHT_GRIPPER_Z_IMU_LINK
- removed link RIGHT_GRIPPER_Z_LINK
- removed link RIGHT_WRIST_X_LINK
- removed link RIGHT_WRIST_Z_IMU_LINK
- removed link RIGHT_WRIST_Z_LINK
- link LEFT_ELBOW_Y_LINK: mass 0.45 -> 0.616; geometry collision cylinder length=0.34 radius=0.033; visual mesh filename=package://alexander_V1_description/meshes/cycloidal_arm/LEF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
- link LEFT_SHOULDER_X_LINK: mass 0.972 -> 1.17068
- link LEFT_SHOULDER_Z_LINK: geometry collision cylinder length=0.26 radius=0.05; visual mesh filename=package://alexander_V1_description/meshes/cycloidal_arm/Lef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
- link RIGHT_ELBOW_Y_LINK: mass 0.45 -> 0.616; geometry collision cylinder length=0.34 radius=0.033; visual mesh filename=package://alexander_V1_description/meshes/cycloidal_arm/RIG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
- link RIGHT_SHOULDER_X_LINK: mass 0.972 -> 1.17068
- link RIGHT_SHOULDER_Z_LINK: geometry collision cylinder length=0.26 radius=0.05; visual mesh filename=package://alexander_V1_description/meshes/cycloidal_arm/Rig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
Joints:
- removed joint LEFT_GRIPPER_ATTACHMENT_FIXED
- removed joint LEFT_GRIPPER_Z
- removed joint LEFT_GRIPPER_Z_IMU_JOINT
- removed joint LEFT_WRIST_X
- removed joint LEFT_WRIST_Z
- removed joint LEFT_WRIST_Z_IMU_JOINT
- removed joint RIGHT_GRIPPER_ATTACHMENT_FIXED
- removed joint RIGHT_GRIPPER_Z
- removed joint RIGHT_GRIPPER_Z_IMU_JOINT
- removed joint RIGHT_HIP_X_IMU_JOINT
- removed joint RIGHT_WRIST_X
- removed joint RIGHT_WRIST_Z
- removed joint RIGHT_WRIST_Z_IMU_JOINT
- added joint RIGHT_HIP_ROLL_IMU_JOINT: type fixed, parent RIGHT_HIP_X_LINK, child RIGHT_HIP_X_IMU_LINK, origin xyz=-0.01922309 -0.07694987 -0.01488788 rpy=-1.570796 0 1.570796, axis 0 0 1
- joint LEFT_SHOULDER_Z: origin xyz=0.0 0.035 0.0 rpy=0.0 0.0 0.0 -> xyz=0.0 0.035 -0.08 rpy=0.0 0.0 0.0
- joint RIGHT_SHOULDER_Z: origin xyz=0.0 -0.035 0.0 rpy=0.0 0.0 0.0 -> xyz=0.0 -0.035 -0.08 rpy=0.0 0.0 0.0

File: alexander-models/alexander_V1_description/urdf/alexander_v1.head.urdf (robot description, URDF)
Before this commit: robot Alexander, 2 links, 2 joints
Links:
- added link HEAD_IMU_LINK, mass 0
Joints:
- added joint HEAD_IMU_JOINT: type fixed, parent HEAD_LINK, child HEAD_IMU_LINK, origin xyz=0.040556 -0.014155 0.057016 rpy=0.56723 0.0 1.5708 , axis 0 0 1
- joint NECK_Y: limit lower=-1.0472 upper=1.0472 effort=20 velocity=20 -> lower=-0.488692 upper=0.488692 effort=20 velocity=20; origin xyz=0.025 0.01 0.207252 rpy=0 0 0 -> xyz=0.025 0.01 0.189597 rpy=0 0 0
- joint NECK_Z: origin xyz=0 0 0.307953 rpy=0 0 0 -> xyz=-0.015 0 0.450403 rpy=0 0 0

File: alexander-models/alexander_V1_description/urdf/alexander_v1.leftForearm.urdf (robot description, URDF)
Before this commit: robot Alexander, 7 links, 7 joints
Links:
- removed link LEFT_SHOULDER_X_LINK
- removed link LEFT_SHOULDER_Y_LINK
- removed link LEFT_SHOULDER_Z_LINK
- added link LEFT_GRIPPER_Z_IMU_LINK, mass 0
- added link LEFT_WRIST_Z_IMU_LINK, mass 0
Joints:
- removed joint LEFT_SHOULDER_X
- removed joint LEFT_SHOULDER_Y
- removed joint LEFT_SHOULDER_Z
- added joint LEFT_GRIPPER_Z_IMU_JOINT: type fixed, parent LEFT_GRIPPER_Z_LINK, child LEFT_GRIPPER_Z_IMU_LINK, origin xyz=0 0 0 rpy=0 0 0, axis 0 0 1
- added joint LEFT_WRIST_Z_IMU_JOINT: type fixed, parent LEFT_WRIST_Z_LINK, child LEFT_WRIST_Z_IMU_LINK, origin xyz=-0.033554 0.010450 -0.148527 rpy=1.571 0.0 1.571, axis 0 0 1

File: alexander-models/alexander_V1_description/urdf/alexander_v1.leftUpperArm.urdf (robot description, URDF)
Before this commit: robot Alexander, 4 links, 4 joints
Links:
- removed link LEFT_ELBOW_PITCH_LINK
- added link LEFT_SHOULDER_Y_IMU_LINK, mass 0
- added link LEFT_SHOULDER_Z_IMU_LINK, mass 0
Joints:
- removed joint LEFT_ELBOW_Y
- added joint LEFT_SHOULDER_Y_IMU_JOINT: type fixed, parent LEFT_SHOULDER_Y_LINK, child LEFT_SHOULDER_Y_IMU_LINK, origin xyz=0.0174 0.06944 -0.03025 rpy=-1.570796 1.570796 0, axis 0 0 1
- added joint LEFT_SHOULDER_Z_IMU_JOINT: type fixed, parent LEFT_SHOULDER_Z_LINK, child LEFT_SHOULDER_Z_IMU_LINK, origin xyz=-0.00763459 -0.0123324 -0.318 rpy=-1.570796 3.1415926 -0.314159, axis 0 0 1
- joint LEFT_SHOULDER_Y: origin xyz=-0.025 0.1 0.214 rpy=0.698132 0.0 0.0 -> xyz=-0.015 0.115474 0.352984 rpy=0.698132 0.0 0.0

File: alexander-models/alexander_V1_description/urdf/alexander_v1.lowerBody.urdf (robot description, URDF)
Before this commit: robot Alexander, 24 links, 23 joints
Links:
- removed link PELVIS_STIM_IMU_LINK
- added link PELVIS_IMU_LINK, mass 0.0
- link LEFT_ANKLE_Y_LINK: mass 0.04972436486 -> 0.05045632
- link LEFT_FOOT: mass 1.264275635 -> 1.28288609; geometry collision box size=0.22 0.1 0.02; visual mesh filename=package://alexander_V1_description/meshes/legs/Foot.obj
- link LEFT_HIP_X_LINK: mass 1.933 -> 2.32977961; geometry collision box size=0.02 0.12 0.10; visual mesh filename=package://alexander_V1_description/meshes/legs/LeftHipRollL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
- link LEFT_HIP_Z_LINK: mass 0.777 -> 0.77281362
- link LEFT_SHIN: mass 7.400 -> 6.31087157; geometry collision cylinder length=0.3 radius=0.08; visual mesh filename=package://alexander_V1_description/meshes/legs/LeftShin.obj
- link LEFT_THIGH: mass 8.200 -> 7.75; geometry collision box size=0.16 0.13 0.29; visual mesh filename=package://alexander_V1_description/meshes/legs/LeftThigh.obj
- link PELVIS_LINK: mass 7.700 -> 9.50083635; geometry collision box size=0.15 0.10 0.12; visual mesh filename=package://alexander_V1_description/meshes/legs/Pelvis.obj
- link RIGHT_ANKLE_Y_LINK: mass 0.04972436486 -> 0.05045632
- link RIGHT_FOOT: mass 1.264275635 -> 1.28288609; geometry collision box size=0.22 0.1 0.02; visual mesh filename=package://alexander_V1_description/meshes/legs/Foot.obj
- link RIGHT_HIP_X_LINK: mass 1.933 -> 2.32977248; geometry collision box size=0.02 0.12 0.10; visual mesh filename=package://alexander_V1_description/meshes/legs/RightHipRoll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
- link RIGHT_HIP_Z_LINK: mass 0.777 -> 0.77281055
- link RIGHT_SHIN: mass 7.400 -> 6.31087157; geometry collision cylinder length=0.3 radius=0.08; visual mesh filename=package://alexander_V1_description/meshes/legs/RightShin.obj
- link RIGHT_THIGH: mass 8.200 -> 7.75; geometry collision box size=0.16 0.13 0.29; visual mesh filename=package://alexander_V1_description/meshes/legs/RightThigh.o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
- link TORSO_IMU_LINK: mass 0.0 -> 0
- link TORSO_LINK: mass 2.13269743 -> 7.0081; geometry collision box size=0.275 0.33 0.43; visual mesh filename=package://alexander_V1_description/meshes/torso.obj
Joints:
- removed joint PELVIS_STIM_IMU_JOINT
- removed joint RIGHT_HIP_ROLL_IMU_JOINT
- added joint PELVIS_IMU_JOINT: type fixed, parent PELVIS_LINK, child PELVIS_IMU_LINK, origin xyz=-0.08687724 0.01225028 -0.08051472 rpy=-0.01399 -0.013054 1.570796
- added joint RIGHT_HIP_X_IMU_JOINT: type fixed, parent RIGHT_HIP_X_LINK, child RIGHT_HIP_X_IMU_LINK, origin xyz=-0.01922309 -0.07694987 -0.01488788 rpy=-1.570796 0 1.570796, axis 0 0 1
- joint LEFT_THIGH_IMU_JOINT: origin xyz=0.10004 0.03746 -0.21194 rpy=1.6947717585 0 1.570796 -> xyz=0.10004 0.03746 -0.21194 rpy=1.437982 0 1.570796
- joint TORSO_IMU_JOINT: axis (none) -> 0 0 1; origin xyz=0.04529 -0.02427 0.33757 rpy=3.141592 0 0 -> xyz=-0.009753 -0.01075 0.373405 rpy=0.0 0.0 -1.5708

File: alexander-models/alexander_V1_description/urdf/alexander_v1.rightForearm.urdf (robot description, URDF)
Before this commit: robot Alexander, 7 links, 7 joints
Links:
- removed link RIGHT_SHOULDER_X_LINK
- removed link RIGHT_SHOULDER_Y_LINK
- removed link RIGHT_SHOULDER_Z_LINK
- added link RIGHT_GRIPPER_Z_IMU_LINK, mass 0
- added link RIGHT_WRIST_Z_IMU_LINK, mass 0
Joints:
- removed joint RIGHT_SHOULDER_X
- removed joint RIGHT_SHOULDER_Y
- removed joint RIGHT_SHOULDER_Z
- added joint RIGHT_GRIPPER_Z_IMU_JOINT: type fixed, parent RIGHT_GRIPPER_Z_LINK, child RIGHT_GRIPPER_Z_IMU_LINK, origin xyz=0 0 0 rpy=0 0 0, axis 0 0 1
- added joint RIGHT_WRIST_Z_IMU_JOINT: type fixed, parent RIGHT_WRIST_Z_LINK, child RIGHT_WRIST_Z_IMU_LINK, origin xyz=-0.033554 0.010450 -0.148527 rpy=1.571  0.0 1.571, axis 0 0 1

File: alexander-models/alexander_V1_description/urdf/alexander_v1.rightUpperArm.urdf (robot description, URDF)
Before this commit: robot Alexander, 4 links, 4 joints
Links:
- removed link RIGHT_ELBOW_PITCH_LINK
- added link RIGHT_SHOULDER_Y_IMU_LINK, mass 0
- added link RIGHT_SHOULDER_Z_IMU_LINK, mass 0
Joints:
- removed joint RIGHT_ELBOW_Y
- added joint RIGHT_SHOULDER_Y_IMU_JOINT: type fixed, parent RIGHT_SHOULDER_Y_LINK, child RIGHT_SHOULDER_Y_IMU_LINK, origin xyz=0.0175 -0.0704 -0.00778 rpy=1.570796 -1.570796 0, axis 0 0 1
- added joint RIGHT_SHOULDER_Z_IMU_JOINT: type fixed, parent RIGHT_SHOULDER_Z_LINK, child RIGHT_SHOULDER_Z_IMU_LINK, origin xyz=0.002 0.016 -0.318 rpy=1.570796 0 0.314159, axis 0 0 1
- joint RIGHT_SHOULDER_Y: origin xyz=-0.025 -0.1 0.214 rpy=-0.698132 0.0 0.0 -> xyz=-0.015 -0.115474 0.352984 rpy=-0.698132 0.0 0.0
