Commit message: Adding hand URDF files

File: alexander-models/alexander_V1_description/urdf/alexander_v1.leftForearm.urdf (robot description, URDF)
Before this commit: robot Alexander, 6 links, 6 joints
Links:
- link LEFT_GRIPPER_Z_LINK: mass 0.251 -> 0.144; geometry visual mesh filename=package://alexander_V1_description/meshes/cycloidal_arm/Lef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

File: alexander-models/alexander_V1_description/urdf/alexander_v1.rightForearm.urdf (robot description, URDF)
Before this commit: robot Alexander, 6 links, 6 joints
Links:
- link RIGHT_GRIPPER_Z_LINK: mass 0.251 -> 0.144; geometry visual mesh filename=package://alexander_V1_description/meshes/cycloidal_arm/Rig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

Commit message: Revert "Adding hand URDF files"
This reverts commit 9e6ae99f73a85d4310eca5710e8b08d12bc4b1b1.

File: alexander-models/alexander_V1_description/urdf/alexander_v1.leftForearm.urdf (robot description, URDF)
Before this commit: robot Alexander, 6 links, 6 joints
Links:
- link LEFT_GRIPPER_Z_LINK: mass 0.144 -> 0.251; geometry visual mesh filename=package://alexander_V1_description/meshes/cycloidal_arm/nub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

File: alexander-models/alexander_V1_description/urdf/alexander_v1.rightForearm.urdf (robot description, URDF)
Before this commit: robot Alexander, 6 links, 6 joints
Links:
- link RIGHT_GRIPPER_Z_LINK: mass 0.144 -> 0.251; geometry visual mesh filename=package://alexander_V1_description/meshes/cycloidal_arm/nub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
