Commit message: Added angular velocity biases

File: alexander-models/alexander_V1_description/urdf/alexander_v1.head.urdf (robot description, URDF)
Before this commit: robot Alexander, 3 links, 3 joints
Joints:
- joint NECK_Y: limit lower=-1.0472 upper=1.0472 effort=20 velocity=20 -> lower=-0.488692 upper=0.488692 effort=20 velocity=20

File: alexander-models/alexander_V1_description/urdf/alexander_v1.lowerBody.urdf (robot description, URDF)
Before this commit: robot Alexander, 24 links, 23 joints
Joints:
- joint TORSO_IMU_JOINT: origin xyz=0.0 0.0 0.0 rpy=0.0 0 0.0 -> xyz=-0.009753 -0.01075 0.373405 rpy=0.0 0.0 -1.57

Commit message: Fixed head imu orientation and position

File: alexander-models/alexander_V1_description/urdf/alexander_v1.head.urdf (robot description, URDF)
Before this commit: robot Alexander, 3 links, 3 joints
Joints:
- joint HEAD_IMU_JOINT: origin xyz=0.040556 -0.14155 0.057016 rpy=0.0 0 0.0 -> xyz=0.040556 -0.014155 0.057016 rpy=0.56723 0.0 1.5708 

File: alexander-models/alexander_V1_description/urdf/alexander_v1.lowerBody.urdf (robot description, URDF)
Before this commit: robot Alexander, 24 links, 23 joints
Joints:
- joint TORSO_IMU_JOINT: origin xyz=-0.009753 -0.01075 0.373405 rpy=0.0 0.0 -1.57 -> xyz=-0.009753 -0.01075 0.373405 rpy=0.0 0.0 -1.5708

Commit message: Fixed some of the positions of shoulder y, neck z, neck y, and the visual torso link

File: alexander-models/alexander_V1_description/urdf/alexander_v1.head.urdf (robot description, URDF)
Before this commit: robot Alexander, 3 links, 3 joints
Joints:
- joint NECK_Y: origin xyz=0.025 0.01 0.207252 rpy=0 0 0 -> xyz=0.025 0.024 0.189597 rpy=0 0 0
- joint NECK_Z: origin xyz=0 0 0.307953 rpy=0 0 0 -> xyz=-0.015 0 0.450403 rpy=0 0 0

File: alexander-models/alexander_V1_description/urdf/alexander_v1.leftLongUpperArm.urdf (robot description, URDF)
Before this commit: robot Alexander, 5 links, 5 joints
Joints:
- joint LEFT_SHOULDER_Y: origin xyz=-0.025 0.1 0.214 rpy=0.698132 0.0 0.0 -> xyz=-0.015 0.115474 0.352984 rpy=0.698132 0.0 0.0

File: alexander-models/alexander_V1_description/urdf/alexander_v1.leftUpperArm.urdf (robot description, URDF)
Before this commit: robot Alexander, 5 links, 5 joints
Joints:
- joint LEFT_SHOULDER_Y: origin xyz=-0.025 0.1 0.214 rpy=0.698132 0.0 0.0 -> xyz=-0.015 0.115474 0.352984 rpy=0.698132 0.0 0.0

File: alexander-models/alexander_V1_description/urdf/alexander_v1.rightLongUpperArm.urdf (robot description, URDF)
Before this commit: robot Alexander, 5 links, 5 joints
Joints:
- joint RIGHT_SHOULDER_Y: origin xyz=-0.025 -0.1 0.214 rpy=-0.698132 0.0 0.0 -> xyz=-0.015 -0.115474 0.352984 rpy=-0.698132 0.0 0.0

File: alexander-models/alexander_V1_description/urdf/alexander_v1.rightUpperArm.urdf (robot description, URDF)
Before this commit: robot Alexander, 5 links, 5 joints
Joints:
- joint RIGHT_SHOULDER_Y: origin xyz=-0.025 -0.1 0.214 rpy=-0.698132 0.0 0.0 -> xyz=-0.015 -0.115474 0.352984 rpy=-0.698132 0.0 0.0

Commit message: Fixed neck y y offset

File: alexander-models/alexander_V1_description/urdf/alexander_v1.head.urdf (robot description, URDF)
Before this commit: robot Alexander, 3 links, 3 joints
Joints:
- joint NECK_Y: origin xyz=0.025 0.024 0.189597 rpy=0 0 0 -> xyz=0.025 0.01 0.189597 rpy=0 0 0

Commit message: Updated the inertia parameters to match real life urdfs

File: alexander-models/alexander_V1_description/urdf/alexander_v1.head.urdf (robot description, URDF)
Before this commit: robot Alexander, 3 links, 3 joints
Links:
- link HEAD_LINK: mass 1.677 -> 1.27065932
- link NECK_Z_LINK: mass 1.141 -> 1.03172573

File: alexander-models/alexander_V1_description/urdf/alexander_v1.leftUpperArm.urdf (robot description, URDF)
Before this commit: robot Alexander, 5 links, 5 joints
Links:
- link LEFT_SHOULDER_X_LINK: mass 0.972 -> 1.16160776 
- link LEFT_SHOULDER_Y_LINK: mass 2.99 -> 3.0331992
- link LEFT_SHOULDER_Z_LINK: mass 2.91 -> 3.134 

File: alexander-models/alexander_V1_description/urdf/alexander_v1.lowerBody.urdf (robot description, URDF)
Before this commit: robot Alexander, 24 links, 23 joints
Links:
- link LEFT_FOOT: mass 1.28288609 -> 1.28831268
- link LEFT_HIP_X_LINK: mass 2.32977961 -> 2.332078
- link LEFT_HIP_Z_LINK: mass 0.77281362 -> 0.74972192 
- link LEFT_SHIN: mass 6.31087157 -> 6.3405718 
- link LEFT_THIGH: mass 7.75 -> 8.286
- link PELVIS_LINK: mass 9.50083635 -> 7.161
- link RIGHT_FOOT: mass 1.28288609 -> 1.28831268
- link RIGHT_HIP_X_LINK: mass 2.32977248 -> 2.33123426 
- link RIGHT_HIP_Z_LINK: mass 0.77281055 -> 0.77280715
- link RIGHT_SHIN: mass 6.31087157 -> 6.33633928 
- link RIGHT_THIGH: mass 7.75 -> 8.27617423 
- link TORSO_LINK: mass 7.0081 -> 11.478322779

File: alexander-models/alexander_V1_description/urdf/alexander_v1.rightUpperArm.urdf (robot description, URDF)
Before this commit: robot Alexander, 5 links, 5 joints
Links:
- link RIGHT_SHOULDER_X_LINK: mass 0.972 -> 1.1615873 
- link RIGHT_SHOULDER_Y_LINK: mass 2.99 -> 3.00752318
- link RIGHT_SHOULDER_Z_LINK: mass 2.91 -> 3.10111287
