Commit message: added forearms and created new urdf with psynoic hands

File: alexander-models/alexander_V1_description/urdf/alexander_v1_cad_accurate_total.urdf (robot description, URDF)
Before this commit: robot Alexander, 39 links, 38 joints
Links:
- added link LEFT_WRIST_X_LINK, mass 0.72320613; visual mesh filename=package://alexander_V1_description/meshes/cycloidal_arm/Lef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
- added link LEFT_WRIST_Z_LINK, mass 1.59997504; collision box size=0.01 0.06 0.1; collision cylinder length=0.12 radius=0.044
- added link RIGHT_WRIST_X_LINK, mass 0.72320613; visual mesh filename=package://alexander_V1_description/meshes/cycloidal_arm/Rig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
- added link RIGHT_WRIST_Z_LINK, mass 1.83740267 kg; collision box size=0.01 0.06 0.1; collision cylinder length=0.12 radius=0.044
- link HEAD_LINK: geometry collision sphere radius=0.14; visual mesh filename=package://alexander_V1_description/meshes/ALX02_01_A02_Head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
- link LEFT_ELBOW_Y_LINK: mass 0.69372585 -> 0.579 ; geometry visual mesh filename=package://alexander_V1_description/meshes/cycloidal_arm/Lef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
- link RIGHT_ELBOW_Y_LINK: mass 0.69372166  -> 0.579 ; geometry visual mesh filename=package://alexander_V1_description/meshes/cycloidal_arm/Rig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
- link TORSO_LINK: geometry collision box size=0.27 0.24 0.4; visual mesh filename=package://alexander_V1_description/meshes/torso.obj
Joints:
- added joint LEFT_GRIPPER_Z: type revolute, parent LEFT_WRIST_X_LINK, child LEFT_GRIPPER_Z_LINK, origin xyz=0.0 0.013 -0.031 rpy=0.0 0.0 0.0, axis 0.0 0.0 1.0, limit lower=-2.61799 upper=2.61799 effort=20.0 velocity=25.0
- added joint LEFT_WRIST_X: type revolute, parent LEFT_WRIST_Z_LINK, child LEFT_WRIST_X_LINK, origin xyz=0.0 -0.013 -0.25 rpy=0.0 0.0 0.0, axis 1 0 0, limit lower=-1.8326 upper=0.610865 effort=20.0 velocity=25.0
- added joint LEFT_WRIST_Z: type revolute, parent LEFT_ELBOW_Y_LINK, child LEFT_WRIST_Z_LINK, origin xyz=-0.015 0.0 0.0 rpy=0.0 0.0 0.0, axis 0.0 0.0 1.0, limit lower=-2.61799 upper=2.61799 effort=20.0 velocity=25.0
- added joint RIGHT_GRIPPER_Z: type revolute, parent RIGHT_WRIST_X_LINK, child RIGHT_GRIPPER_Z_LINK, origin xyz=0.0 -0.013 -0.031 rpy=0.0 0.0 0.0, axis 0.0 0.0 1.0, limit lower=-2.61799 upper=2.61799 effort=20.0 velocity=25.0
- added joint RIGHT_WRIST_X: type revolute, parent RIGHT_WRIST_Z_LINK, child RIGHT_WRIST_X_LINK, origin xyz=0.0 0.013 -0.25 rpy=0.0 0.0 0.0, axis 1 0 0, limit lower=-0.610865 upper=1.8326 effort=20.0 velocity=25.0
- added joint RIGHT_WRIST_Z: type revolute, parent RIGHT_ELBOW_Y_LINK, child RIGHT_WRIST_Z_LINK, origin xyz=-0.015 0.0 0.0 rpy=0.0 0.0 0.0, axis 0.0 0.0 1.0, limit lower=-2.61799 upper=2.61799 effort=20.0 velocity=25.0
