Commit message: added forearms and created new urdf with psynoic hands

File: alexander-models/alexander_V1_description/urdf/alexander_v1_realLife_accurate_total_hands.urdf (robot description, URDF)
Before this commit: robot Alexander, 45 links, 44 joints
Links:
- removed link LEFT_GRIPPER_Z_LINK
- removed link RIGHT_GRIPPER_Z_LINK
- added link base, mass 0.37511000; collision mesh filename=package://alexander_V1_description/meshes/abilityHand/palm_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; visual mesh filename=package://alexander_V1_description/meshes/abilityHand/FB_pa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
- added link base_right, mass 0.37511000; collision mesh filename=package://alexander_V1_description/meshes/abilityHand/palm_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; visual mesh filename=package://alexander_V1_description/meshes/abilityHand/FB_pa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
- added link fsr0
- added link fsr0_right
- added link fsr1
- added link fsr10
- added link fsr10_right
- added link fsr11
- added link fsr11_right
- added link fsr12
- added link fsr12_right
- added link fsr13
- added link fsr13_right
- added link fsr14
- added link fsr14_right
- added link fsr15
- added link fsr15_right
- added link fsr16
- added link fsr16_right
- added link fsr17
- added link fsr17_right
- added link fsr18
- added link fsr18_right
- added link fsr19
- added link fsr19_right
- added link fsr1_right
- added link fsr2
- added link fsr20
- added link fsr20_right
- added link fsr21
- added link fsr21_right
- added link fsr22
- added link fsr22_right
- added link fsr23
- added link fsr23_right
- added link fsr24
- added link fsr24_right
- added link fsr25
- added link fsr25_right
- added link fsr26
- added link fsr26_right
- added link fsr27
- added link fsr27_right
- added link fsr28
- added link fsr28_right
- added link fsr29
- added link fsr29_right
- added link fsr2_right
- added link fsr3
- added link fsr3_right
- added link fsr4
- added link fsr4_right
- added link fsr5
- added link fsr5_right
- added link fsr6
- added link fsr6_right
- added link fsr7
- added link fsr7_right
- added link fsr8
- added link fsr8_right
- added link fsr9
- added link fsr9_right
- added link index_L1, mass 0.00636000; collision mesh filename=package://alexander_V1_description/meshes/abilityHand/idx-F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; visual mesh filename=package://alexander_V1_description/meshes/abilityHand/idx-F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
- added link index_L1_right, mass 0.00636000; collision mesh filename=package://alexander_V1_description/meshes/abilityHand/idx-F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; visual mesh filename=package://alexander_V1_description/meshes/abilityHand/idx-F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
- added link index_L2, mass 0.00600000; collision mesh filename=package://alexander_V1_description/meshes/abilityHand/idx-F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; visual mesh filename=package://alexander_V1_description/meshes/abilityHand/idx-F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
- added link index_L2_right, mass 0.00600000; collision mesh filename=package://alexander_V1_description/meshes/abilityHand/idx-F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; visual mesh filename=package://alexander_V1_description/meshes/abilityHand/idx-F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
- added link index_anchor
- added link index_anchor_right
- added link middle_L1, mass 0.00636000; collision mesh filename=package://alexander_V1_description/meshes/abilityHand/idx-F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; visual mesh filename=package://alexander_V1_description/meshes/abilityHand/idx-F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
- added link middle_L1_right, mass 0.00636000; collision mesh filename=package://alexander_V1_description/meshes/abilityHand/idx-F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; visual mesh filename=package://alexander_V1_description/meshes/abilityHand/idx-F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
- added link middle_L2, mass 0.00600000; collision mesh filename=package://alexander_V1_description/meshes/abilityHand/idx-F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; visual mesh filename=package://alexander_V1_description/meshes/abilityHand/idx-F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
- added link middle_L2_right, mass 0.00600000; collision mesh filename=package://alexander_V1_description/meshes/abilityHand/idx-F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; visual mesh filename=package://alexander_V1_description/meshes/abilityHand/idx-F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
- added link middle_anchor
- added link middle_anchor_right
- added link pinky_L1, mass 0.00636000; collision mesh filename=package://alexander_V1_description/meshes/abilityHand/idx-F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; visual mesh filename=package://alexander_V1_description/meshes/abilityHand/idx-F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
- added link pinky_L1_right, mass 0.00636000; collision mesh filename=package://alexander_V1_description/meshes/abilityHand/idx-F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; visual mesh filename=package://alexander_V1_description/meshes/abilityHand/idx-F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
- added link pinky_L2, mass 0.00600000; collision mesh filename=package://alexander_V1_description/meshes/abilityHand/idx-F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; visual mesh filename=package://alexander_V1_description/meshes/abilityHand/idx-F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
- added link pinky_L2_right, mass 0.00600000; collision mesh filename=package://alexander_V1_description/meshes/abilityHand/idx-F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; visual mesh filename=package://alexander_V1_description/meshes/abilityHand/idx-F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
- added link pinky_anchor
- added link pinky_anchor_right
- added link ring_L1, mass 0.00636000; collision mesh filename=package://alexander_V1_description/meshes/abilityHand/idx-F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; visual mesh filename=package://alexander_V1_description/meshes/abilityHand/idx-F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
- added link ring_L1_right, mass 0.00636000; collision mesh filename=package://alexander_V1_description/meshes/abilityHand/idx-F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; visual mesh filename=package://alexander_V1_description/meshes/abilityHand/idx-F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
- added link ring_L2, mass 0.00600000; collision mesh filename=package://alexander_V1_description/meshes/abilityHand/idx-F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; visual mesh filename=package://alexander_V1_description/meshes/abilityHand/idx-F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
- added link ring_L2_right, mass 0.00600000; collision mesh filename=package://alexander_V1_description/meshes/abilityHand/idx-F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; visual mesh filename=package://alexander_V1_description/meshes/abilityHand/idx-F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
- added link ring_anchor
- added link ring_anchor_right
- added link thumb_L1, mass 0.00200000; collision mesh filename=package://alexander_V1_description/meshes/abilityHand/thumb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; visual mesh filename=package://alexander_V1_description/meshes/abilityHand/thumb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
- added link thumb_L1_right, mass 0.00200000; collision mesh filename=package://alexander_V1_description/meshes/abilityHand/thumb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; visual mesh filename=package://alexander_V1_description/meshes/abilityHand/thumb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
- added link thumb_L2, mass 0.06000000; collision mesh filename=package://alexander_V1_description/meshes/abilityHand/thumb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; visual mesh filename=package://alexander_V1_description/meshes/abilityHand/thumb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
- added link thumb_L2_right, mass 0.06000000; collision mesh filename=package://alexander_V1_description/meshes/abilityHand/thumb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; visual mesh filename=package://alexander_V1_description/meshes/abilityHand/thumb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
- added link thumb_anchor
- added link thumb_anchor_right
Joints:
- added joint fsr0: type fixed, parent index_L2, child fsr0, origin xyz=0.02936 -0.01697 -0.00435 rpy=3.14 0 -0.1848
- added joint fsr0_right: type fixed, parent index_L2_right, child fsr0_right, origin xyz=0.02936 -0.01697 -0.00435 rpy=3.14 0 -0.1848
- added joint fsr1: type fixed, parent index_L2, child fsr1, origin xyz=0.02961 -0.01394 0.0 rpy=-1.5708 0.0 -0.2316
- added joint fsr10: type fixed, parent middle_L2, child fsr10, origin xyz=0.01472 -0.01099 0.00435 rpy=0.00000 0.00000 -0.57199
- added joint fsr10_right: type fixed, parent middle_L2_right, child fsr10_right, origin xyz=0.01472 -0.01099 0.00435 rpy=0.00000 0.00000 -0.57199
- added joint fsr11: type fixed, parent middle_L2, child fsr11, origin xyz=0.03704 -0.01785 0.00000 rpy=-2.66907 -1.57080 0.00000
- added joint fsr11_right: type fixed, parent middle_L2_right, child fsr11_right, origin xyz=0.03704 -0.01785 0.00000 rpy=-2.66907 -1.57080 0.00000
- added joint fsr12: type fixed, parent ring_L2, child fsr12, origin xyz=0.02936 -0.01697 -0.00435 rpy=3.14 0 -0.1848
- added joint fsr12_right: type fixed, parent ring_L2_right, child fsr12_right, origin xyz=0.02936 -0.01697 -0.00435 rpy=3.14 0 -0.1848
- added joint fsr13: type fixed, parent ring_L2, child fsr13, origin xyz=0.02961 -0.01394 0.0 rpy=-1.5708 0.0 -0.2316
- added joint fsr13_right: type fixed, parent ring_L2_right, child fsr13_right, origin xyz=0.02961 -0.01394 0.0 rpy=-1.5708 0.0 -0.2316
- added joint fsr14: type fixed, parent ring_L2, child fsr14, origin xyz=0.02936 -0.01697 0.00435 rpy=0.0 0.0 -0.1848036056311012
- added joint fsr14_right: type fixed, parent ring_L2_right, child fsr14_right, origin xyz=0.02936 -0.01697 0.00435 rpy=0.0 0.0 -0.1848036056311012
- added joint fsr15: type fixed, parent ring_L2, child fsr15, origin xyz=0.01472 -0.01100 -0.00435 rpy=3.14159 0.00000 -0.57092
- added joint fsr15_right: type fixed, parent ring_L2_right, child fsr15_right, origin xyz=0.01472 -0.01100 -0.00435 rpy=3.14159 0.00000 -0.57092
- added joint fsr16: type fixed, parent ring_L2, child fsr16, origin xyz=0.01472 -0.01099 0.00435 rpy=0.00000 0.00000 -0.57199
- added joint fsr16_right: type fixed, parent ring_L2_right, child fsr16_right, origin xyz=0.01472 -0.01099 0.00435 rpy=0.00000 0.00000 -0.57199
- added joint fsr17: type fixed, parent ring_L2, child fsr17, origin xyz=0.03704 -0.01785 0.00000 rpy=-2.66907 -1.57080 0.00000
- added joint fsr17_right: type fixed, parent ring_L2_right, child fsr17_right, origin xyz=0.03704 -0.01785 0.00000 rpy=-2.66907 -1.57080 0.00000
- added joint fsr18: type fixed, parent pinky_L2, child fsr18, origin xyz=0.02556 -0.01391 -0.00435 rpy=3.14 0 -0.1848
- added joint fsr18_right: type fixed, parent pinky_L2_right, child fsr18_right, origin xyz=0.02556 -0.01391 -0.00435 rpy=3.14 0 -0.1848
- added joint fsr19: type fixed, parent pinky_L2, child fsr19, origin xyz=0.02517 -0.01110 -0.00000 rpy=-1.5708 0.0 -0.2316
- added joint fsr19_right: type fixed, parent pinky_L2_right, child fsr19_right, origin xyz=0.02517 -0.01110 -0.00000 rpy=-1.5708 0.0 -0.2316
- added joint fsr1_right: type fixed, parent index_L2_right, child fsr1_right, origin xyz=0.02961 -0.01394 0.0 rpy=-1.5708 0.0 -0.2316
- added joint fsr2: type fixed, parent index_L2, child fsr2, origin xyz=0.02936 -0.01697 0.00435 rpy=0.0 0.0 -0.1848036056311012
- added joint fsr20: type fixed, parent pinky_L2, child fsr20, origin xyz=0.02556 -0.01391 0.00435 rpy=0.0 0.0 -0.1848036056311012
- added joint fsr20_right: type fixed, parent pinky_L2_right, child fsr20_right, origin xyz=0.02556 -0.01391 0.00435 rpy=0.0 0.0 -0.1848036056311012
- added joint fsr21: type fixed, parent pinky_L2, child fsr21, origin xyz=0.01310 -0.00943 -0.00435 rpy=3.14159 0.00000 -0.57092
- added joint fsr21_right: type fixed, parent pinky_L2_right, child fsr21_right, origin xyz=0.01310 -0.00943 -0.00435 rpy=3.14159 0.00000 -0.57092
- added joint fsr22: type fixed, parent pinky_L2, child fsr22, origin xyz=0.01310 -0.00943 0.00435 rpy=0.00000 0.00000 -0.57199
- added joint fsr22_right: type fixed, parent pinky_L2_right, child fsr22_right, origin xyz=0.01310 -0.00943 0.00435 rpy=0.00000 0.00000 -0.57199
- added joint fsr23: type fixed, parent pinky_L2, child fsr23, origin xyz=0.03142 -0.01438 0.00000 rpy=-2.66907 -1.57080 0.00000
- added joint fsr23_right: type fixed, parent pinky_L2_right, child fsr23_right, origin xyz=0.03142 -0.01438 0.00000 rpy=-2.66907 -1.57080 0.00000
- added joint fsr24: type fixed, parent thumb_L2, child fsr24, origin xyz=0.04747 0.01988 -0.00874 rpy=-2.29074 0.00001 0.41769
- added joint fsr24_right: type fixed, parent thumb_L2_right, child fsr24_right, origin xyz=0.04747 0.01988 -0.001239 rpy=-2.29074 0.00001 0.41769
- added joint fsr25: type fixed, parent thumb_L2, child fsr25, origin xyz=0.04721 0.02124 -0.00106 rpy=-1.30899 0.00001 0.41769
- added joint fsr25_right: type fixed, parent thumb_L2_right, child fsr25_right, origin xyz=0.04721 0.02124 0.006439 rpy=-1.30899 0.00001 0.41769
- added joint fsr26: type fixed, parent thumb_L2, child fsr26, origin xyz=0.04896 0.01654 0.00491 rpy=-0.32726 0.00001 0.41769
- added joint fsr26_right: type fixed, parent thumb_L2_right, child fsr26_right, origin xyz=0.04896 0.01654 0.01241 rpy=-0.32726 0.00001 0.41769
- added joint fsr27: type fixed, parent thumb_L2, child fsr27, origin xyz=0.03739 0.01536 -0.00879 rpy=-2.29074 0.00001 0.41769
- added joint fsr27_right: type fixed, parent thumb_L2_right, child fsr27_right, origin xyz=0.03739 0.01536 -0.001289 rpy=-2.29074 0.00001 0.41769
- added joint fsr28: type fixed, parent thumb_L2, child fsr28, origin xyz=0.03888 0.01200 0.00494 rpy=-0.32726 0.00001 0.41769
- added joint fsr28_right: type fixed, parent thumb_L2_right, child fsr28_right, origin xyz=0.03888 0.01200 0.01244 rpy=-0.32726 0.00001 0.41769
- added joint fsr29: type fixed, parent thumb_L2, child fsr29, origin xyz=0.05591 0.02160 -0.00192
- added joint fsr29_right: type fixed, parent thumb_L2_right, child fsr29_right, origin xyz=0.05591 0.02160 0.00558
- added joint fsr2_right: type fixed, parent index_L2_right, child fsr2_right, origin xyz=0.02936 -0.01697 0.00435 rpy=0.0 0.0 -0.1848036056311012
- added joint fsr3: type fixed, parent index_L2, child fsr3, origin xyz=0.01472 -0.01100 -0.00435 rpy=3.14159 0.00000 -0.57092
- added joint fsr3_right: type fixed, parent index_L2_right, child fsr3_right, origin xyz=0.01472 -0.01100 -0.00435 rpy=3.14159 0.00000 -0.57092
- added joint fsr4: type fixed, parent index_L2, child fsr4, origin xyz=0.01472 -0.01099 0.00435 rpy=0.00000 0.00000 -0.57199
- added joint fsr4_right: type fixed, parent index_L2, child fsr4_right, origin xyz=0.01472 -0.01099 0.00435 rpy=0.00000 0.00000 -0.57199
- added joint fsr5: type fixed, parent index_L2, child fsr5, origin xyz=0.03704 -0.01785 0.00000 rpy=-2.66907 -1.57080 0.00000
- added joint fsr5_right: type fixed, parent index_L2_right, child fsr5_right, origin xyz=0.03704 -0.01785 0.00000 rpy=-2.66907 -1.57080 0.00000
- added joint fsr6: type fixed, parent middle_L2, child fsr6, origin xyz=0.02936 -0.01697 -0.00435 rpy=3.14 0 -0.1848
- added joint fsr6_right: type fixed, parent middle_L2_right, child fsr6_right, origin xyz=0.02936 -0.01697 -0.00435 rpy=3.14 0 -0.1848
- added joint fsr7: type fixed, parent middle_L2, child fsr7, origin xyz=0.02961 -0.01394 0.0 rpy=-1.5708 0.0 -0.2316
- added joint fsr7_right: type fixed, parent middle_L2_right, child fsr7_right, origin xyz=0.02961 -0.01394 0.0 rpy=-1.5708 0.0 -0.2316
- added joint fsr8: type fixed, parent middle_L2, child fsr8, origin xyz=0.02936 -0.01697 0.00435 rpy=0.0 0.0 -0.1848036056311012
- added joint fsr8_right: type fixed, parent middle_L2_right, child fsr8_right, origin xyz=0.02936 -0.01697 0.00435 rpy=0.0 0.0 -0.1848036056311012
- added joint fsr9: type fixed, parent middle_L2, child fsr9, origin xyz=0.01472 -0.01100 -0.00435 rpy=3.14159 0.00000 -0.57092
- added joint fsr9_right: type fixed, parent middle_L2_right, child fsr9_right, origin xyz=0.01472 -0.01100 -0.00435 rpy=3.14159 0.00000 -0.57092
- added joint idx_anchor: type fixed, parent index_L2, child index_anchor, origin xyz=31.5541e-3  -10.44e-3 0.14e-3 rpy=0 0 0
- added joint idx_anchor_right: type fixed, parent index_L2_right, child index_anchor_right, origin xyz=31.5541e-3  -10.44e-3 0.14e-3 rpy=0 0 0
- added joint index_q1: type revolute, parent base, child index_L1, origin xyz=0.028 -0.009 0.096 rpy=1.470 -1.317 -1.352, axis 0 0 1, limit lower=0 upper=1.74 effort=6.0 velocity=8.0677777442
- added joint index_q1_right: type revolute, parent base_right, child index_L1_right, origin xyz=-2.8e-2 -9e-3 9.6e-2 rpy= 1.672 -1.317 -1.790 , axis 0 0 1, limit lower=0 upper=1.74 effort=6.0 velocity=8.0677777442
- added joint index_q2: type revolute, parent index_L1, child index_L2, origin xyz=38.472723e-3 3.257695e-3 0.000000e-3 rpy=0 0 0.084474, axis 0 0 1, limit lower=0.766 upper=2.61 effort=6.0 velocity=8.0677777442, mimic joint=index_q1 multiplier=1.05851325 offset=0.72349796
- added joint index_q2_right: type revolute, parent index_L1_right, child index_L2_right, origin xyz=38.472723e-3 3.257695e-3 0.000000e-3 rpy=0 0 0.084474, axis 0 0 1, limit lower=0.766 upper=2.61 effort=6.0 velocity=8.0677777442, mimic joint=index_q1_right multiplier=1.05851325 offset=0.72349796
- added joint mid_anchor: type fixed, parent middle_L2, child middle_anchor, origin xyz=31.5541e-3  -10.44e-3 0.14e-3 rpy=0 0 0
- added joint mid_anchor_right: type fixed, parent middle_L2_right, child middle_anchor_right, origin xyz=31.5541e-3  -10.44e-3 0.14e-3 rpy=0 0 0
- added joint middle_q1: type revolute, parent base, child middle_L1, origin xyz=0.008 -0.012 0.099 rpy=1.629 -1.322 -1.583, axis 0 0 1, limit lower=0 upper=1.74 effort=6.0 velocity=8.0677777442
- added joint middle_q1_right: type revolute, parent base_right, child middle_L1_right, origin xyz= -0.008 -0.012 0.099  rpy= 1.513 -1.322 -1.558 , axis 0 0 1, limit lower=0 upper=1.74 effort=6.0 velocity=8.0677777442
- added joint middle_q2: type revolute, parent middle_L1, child middle_L2, origin xyz=38.472723e-3 3.257695e-3 0.000000 rpy=0 0 0.084474, axis 0 0 1, limit lower=0.766 upper=2.61 effort=6.0 velocity=8.0677777442, mimic joint=middle_q1 multiplier=1.05851325 offset=0.72349796
- added joint middle_q2_right: type revolute, parent middle_L1_right, child middle_L2_right, origin xyz=38.472723e-3 3.257695e-3 0.000000 rpy=0 0 0.084474, axis 0 0 1, limit lower=0.766 upper=2.61 effort=6.0 velocity=8.0677777442, mimic joint=middle_q1_right multiplier=1.05851325 offset=0.72349796
- added joint pinky_q1: type revolute, parent base, child pinky_L1, origin xyz=-0.031 -0.007 0.091 rpy=1.731 -1.315 -1.828, axis 0 0 1, limit lower=0 upper=1.74 effort=6.0 velocity=8.0677777442
- added joint pinky_q1_right: type revolute, parent base_right, child pinky_L1_right, origin xyz= 0.031 -0.007 0.091  rpy= 1.410 -1.315 -1.313 , axis 0 0 1, limit lower=0 upper=1.74 effort=6.0 velocity=8.0677777442
- added joint pinky_q2: type revolute, parent pinky_L1, child pinky_L2, origin xyz=38.472723e-3 3.257695e-3 0.000000 rpy=0 0 0.084474, axis 0 0 1, limit lower=0.766 upper=2.61 effort=6.0 velocity=8.0677777442, mimic joint=pinky_q1 multiplier=1.05851325 offset=0.72349796
- added joint pinky_q2_right: type revolute, parent pinky_L1_right, child pinky_L2_right, origin xyz=38.472723e-3 3.257695e-3 0.000000 rpy=0 0 0.084474, axis 0 0 1, limit lower=0.766 upper=2.61 effort=6.0 velocity=8.0677777442, mimic joint=pinky_q1_right multiplier=1.05851325 offset=0.72349796
- added joint pnky_anchor: type fixed, parent pinky_L2, child pinky_anchor, origin xyz=31.5541e-3  -10.44e-3 0.14e-3 rpy=0 0 0
- added joint pnky_anchor_right: type fixed, parent pinky_L2_right, child pinky_anchor_right, origin xyz=31.5541e-3  -10.44e-3 0.14e-3 rpy=0 0 0
- added joint ring_q1: type revolute, parent base, child ring_L1, origin xyz=-0.012 -0.010 0.097 rpy=1.780 -1.315 -1.811, axis 0 0 1, limit lower=0 upper=1.74 effort=6.0 velocity=8.0677777442
- added joint ring_q1_right: type revolute, parent base_right, child ring_L1_right, origin xyz= 0.012 -0.010 0.097  rpy= 1.361 -1.315 -1.330 , axis 0 0 1, limit lower=0 upper=1.74 effort=6.0 velocity=8.0677777442
- added joint ring_q2: type revolute, parent ring_L1, child ring_L2, origin xyz=38.472723e-3 3.257695e-3 0.000000 rpy=0 0 0.084474, axis 0 0 1, limit lower=0.766 upper=2.61 effort=6.0 velocity=8.0677777442, mimic joint=ring_q1 multiplier=1.05851325 offset=0.72349796
- added joint ring_q2_right: type revolute, parent ring_L1_right, child ring_L2_right, origin xyz=38.472723e-3 3.257695e-3 0.000000 rpy=0 0 0.084474, axis 0 0 1, limit lower=0.766 upper=2.61 effort=6.0 velocity=8.0677777442, mimic joint=ring_q1_right multiplier=1.05851325 offset=0.72349796
- added joint rng_anchor: type fixed, parent ring_L2, child ring_anchor, origin xyz=31.5541e-3  -10.44e-3 0.14e-3 rpy=0 0 0
- added joint rng_anchor_right: type fixed, parent ring_L2_right, child ring_anchor_right, origin xyz=31.5541e-3  -10.44e-3 0.14e-3 rpy=0 0 0
- added joint thmb_anchor: type fixed, parent thumb_L2, child thumb_anchor, origin xyz=52.0012259e-3  28.0086971e-3 -.884835778e-3 rpy=0 0 0
- added joint thmb_anchor_right: type fixed, parent thumb_L2_right, child thumb_anchor_right, origin xyz=52.00122724e-3 28.00869333e-3 6.98483578e-3 rpy=0 0 0
- added joint thumb_q1: type revolute, parent base, child thumb_L1, origin xyz=24.0476665e-3 3.78124745e-3 32.32964923e-3 rpy=-3.1250458 -0.08693131 -0.1883423, axis 0 0 1, limit lower=-1.74 upper=0 effort=1.2 velocity=40.338888721
- added joint thumb_q1_right: type revolute, parent base_right, child thumb_L1_right, origin xyz=-24.0476665e-3 3.78124745e-3 32.32964923e-3 rpy=-0.01675973 -0.08689062 -2.95079797, axis 0 0 1, limit lower=-1.74 upper=0 effort=1.2 velocity=40.338888721
- added joint thumb_q2: type revolute, parent thumb_L1, child thumb_L2, origin xyz=27.8283501e-3 0 -14.7507000e-3 rpy=4.450589592585541 0 0, axis 0 0 1, limit lower=0 upper=1.74 effort=6.0 velocity=8.0677777442
- added joint thumb_q2_right: type revolute, parent thumb_L1_right, child thumb_L2_right, origin xyz= 27.8283501e-3 1.7436510745838653e-19 14.7507e-3  rpy= 1.832595714594045 -0.0 5.366520605522463e-18 , axis 0 0 1, limit lower=0 upper=1.74 effort=6.0 velocity=8.0677777442
- joint LEFT_GRIPPER_Z: child LEFT_GRIPPER_Z_LINK -> base; origin xyz=0.0 0.013 -0.031 rpy=0.0 0.0 0.0 -> xyz=0.0 0.013 -0.031 rpy=3.14 0.0 0.0
- joint RIGHT_GRIPPER_Z: child RIGHT_GRIPPER_Z_LINK -> base_right; origin xyz=0.0 -0.013 -0.031 rpy=0.0 0.0 0.0 -> xyz=0.0 -0.013 -0.031 rpy=3.14 0.0 3.14
