Commit message: Fixed names for IMU links and joints to match standard

File: alexander-models/alexander_V1_description/urdf/alexander_v1_cad_accurate_total.urdf (robot description, URDF)
Before this commit: robot Alexander, 43 links, 44 joints
Links:
- removed link LEFT_SHOULDER_PITCH_IMU_LINK
- removed link LEFT_SHOULDER_YAW_IMU_LINK
- removed link RIGHT_SHOULDER_PITCH_IMU_LINK
- removed link RIGHT_SHOULDER_YAW_IMU_LINK
- added link LEFT_SHOULDER_Y_IMU_LINK, mass 0
- added link LEFT_SHOULDER_Z_IMU_LINK, mass 0
- added link RIGHT_SHOULDER_Y_IMU_LINK, mass 0
- added link RIGHT_SHOULDER_Z_IMU_LINK, mass 0
Joints:
- removed joint LEFT_SHOULDER_PITCH_IMU_JOINT
- removed joint LEFT_SHOULDER_YAW_IMU_JOINT
- removed joint RIGHT_HIP_ROLL_IMU_JOINT
- removed joint RIGHT_SHOULDER_PITCH_IMU_JOINT
- removed joint RIGHT_SHOULDER_YAW_IMU_JOINT
- added joint LEFT_SHOULDER_Y_IMU_JOINT: type fixed, parent LEFT_SHOULDER_Y_LINK, child LEFT_SHOULDER_Y_IMU_LINK, origin xyz=0.0174 0.06944 -0.03025 rpy=-1.570796 1.570796 0, axis 0 0 1
- added joint LEFT_SHOULDER_Z_IMU_JOINT: type fixed, parent LEFT_SHOULDER_Z_LINK, child LEFT_SHOULDER_Z_IMU_LINK, origin xyz=-0.00763459 -0.0123324 -0.318 rpy=-1.570796 3.1415926 -0.314159, axis 0 0 1
- added joint RIGHT_HIP_X_IMU_JOINT: type fixed, parent RIGHT_HIP_X_LINK, child RIGHT_HIP_X_IMU_LINK, origin xyz=-0.01922309 -0.07694987 -0.01488788 rpy=-1.570796 0 1.570796, axis 0 0 1
- added joint RIGHT_SHOULDER_Y_IMU_JOINT: type fixed, parent RIGHT_SHOULDER_Y_LINK, child RIGHT_SHOULDER_Y_IMU_LINK, origin xyz=0.0175 -0.0704 -0.00778 rpy=1.570796 -1.570796 0, axis 0 0 1
- added joint RIGHT_SHOULDER_Z_IMU_JOINT: type fixed, parent RIGHT_SHOULDER_Z_LINK, child RIGHT_SHOULDER_Z_IMU_LINK, origin xyz=0.002 0.016 -0.318 rpy=1.570796 0 0.314159, axis 0 0 1

File: alexander-models/alexander_V1_description/urdf/alexander_v1_realLife_accurate_total.urdf (robot description, URDF)
Before this commit: robot Alexander, 45 links, 44 joints
Links:
- removed link LEFT_SHOULDER_PITCH_IMU_LINK
- removed link LEFT_SHOULDER_YAW_IMU_LINK
- removed link RIGHT_SHOULDER_PITCH_IMU_LINK
- removed link RIGHT_SHOULDER_YAW_IMU_LINK
- added link LEFT_SHOULDER_Y_IMU_LINK, mass 0
- added link LEFT_SHOULDER_Z_IMU_LINK, mass 0
- added link RIGHT_SHOULDER_Y_IMU_LINK, mass 0
- added link RIGHT_SHOULDER_Z_IMU_LINK, mass 0
Joints:
- removed joint LEFT_SHOULDER_PITCH_IMU_JOINT
- removed joint LEFT_SHOULDER_YAW_IMU_JOINT
- removed joint RIGHT_HIP_ROLL_IMU_JOINT
- removed joint RIGHT_SHOULDER_PITCH_IMU_JOINT
- removed joint RIGHT_SHOULDER_YAW_IMU_JOINT
- added joint LEFT_SHOULDER_Y_IMU_JOINT: type fixed, parent LEFT_SHOULDER_Y_LINK, child LEFT_SHOULDER_Y_IMU_LINK, origin xyz=0.0174 0.06944 -0.03025 rpy=-1.570796 1.570796 0, axis 0 0 1
- added joint LEFT_SHOULDER_Z_IMU_JOINT: type fixed, parent LEFT_SHOULDER_Z_LINK, child LEFT_SHOULDER_Z_IMU_LINK, origin xyz=-0.00763459 -0.0123324 -0.318 rpy=-1.570796 3.1415926 -0.314159, axis 0 0 1
- added joint RIGHT_HIP_X_IMU_JOINT: type fixed, parent RIGHT_HIP_X_LINK, child RIGHT_HIP_X_IMU_LINK, origin xyz=-0.01922309 -0.07694987 -0.01488788 rpy=-1.570796 0 1.570796, axis 0 0 1
- added joint RIGHT_SHOULDER_Y_IMU_JOINT: type fixed, parent RIGHT_SHOULDER_Y_LINK, child RIGHT_SHOULDER_Y_IMU_LINK, origin xyz=0.0175 -0.0704 -0.00778 rpy=1.570796 -1.570796 0, axis 0 0 1
- added joint RIGHT_SHOULDER_Z_IMU_JOINT: type fixed, parent RIGHT_SHOULDER_Z_LINK, child RIGHT_SHOULDER_Z_IMU_LINK, origin xyz=0.002 0.016 -0.318 rpy=1.570796 0 0.314159, axis 0 0 1

File: alexander-models/alexander_V1_description/urdf/alexander_v1_realLife_accurate_total_hands.urdf (robot description, URDF)
Before this commit: robot Alexander, 135 links, 134 joints
Links:
- removed link LEFT_SHOULDER_PITCH_IMU_LINK
- removed link LEFT_SHOULDER_YAW_IMU_LINK
- removed link RIGHT_SHOULDER_PITCH_IMU_LINK
- removed link RIGHT_SHOULDER_YAW_IMU_LINK
- added link LEFT_SHOULDER_Y_IMU_LINK, mass 0
- added link LEFT_SHOULDER_Z_IMU_LINK, mass 0
- added link RIGHT_SHOULDER_Y_IMU_LINK, mass 0
- added link RIGHT_SHOULDER_Z_IMU_LINK, mass 0
Joints:
- removed joint LEFT_SHOULDER_PITCH_IMU_JOINT
- removed joint LEFT_SHOULDER_YAW_IMU_JOINT
- removed joint RIGHT_HIP_ROLL_IMU_JOINT
- removed joint RIGHT_SHOULDER_PITCH_IMU_JOINT
- removed joint RIGHT_SHOULDER_YAW_IMU_JOINT
- added joint LEFT_SHOULDER_Y_IMU_JOINT: type fixed, parent LEFT_SHOULDER_Y_LINK, child LEFT_SHOULDER_Y_IMU_LINK, origin xyz=0.0174 0.06944 -0.03025 rpy=-1.570796 1.570796 0, axis 0 0 1
- added joint LEFT_SHOULDER_Z_IMU_JOINT: type fixed, parent LEFT_SHOULDER_Z_LINK, child LEFT_SHOULDER_Z_IMU_LINK, origin xyz=-0.00763459 -0.0123324 -0.318 rpy=-1.570796 3.1415926 -0.314159, axis 0 0 1
- added joint RIGHT_HIP_X_IMU_JOINT: type fixed, parent RIGHT_HIP_X_LINK, child RIGHT_HIP_X_IMU_LINK, origin xyz=-0.01922309 -0.07694987 -0.01488788 rpy=-1.570796 0 1.570796, axis 0 0 1
- added joint RIGHT_SHOULDER_Y_IMU_JOINT: type fixed, parent RIGHT_SHOULDER_Y_LINK, child RIGHT_SHOULDER_Y_IMU_LINK, origin xyz=0.0175 -0.0704 -0.00778 rpy=1.570796 -1.570796 0, axis 0 0 1
- added joint RIGHT_SHOULDER_Z_IMU_JOINT: type fixed, parent RIGHT_SHOULDER_Z_LINK, child RIGHT_SHOULDER_Z_IMU_LINK, origin xyz=0.002 0.016 -0.318 rpy=1.570796 0 0.314159, axis 0 0 1
