Commit message: Add right ability hand adapter

File: alexander-models/alexander_V1_description/urdf/alexander_v1.leftAbilityHandAdapter.urdf (robot description, URDF)
Before this commit: robot Alexander, 0 links, 1 joints
Joints:
- joint LEFT_ABILITY_HAND_ADAPTER: child base -> left_ability_hand_base

Commit message: added yaw offset for hand adapter urdf

File: alexander-models/alexander_V1_description/urdf/alexander_v1.leftAbilityHandAdapter.urdf (robot description, URDF)
Before this commit: robot Alexander, 0 links, 1 joints
Joints:
- joint LEFT_ABILITY_HAND_ADAPTER: origin xyz=0 0 -0.022 rpy=3.141592 0 0 -> xyz=0 0 -0.022 rpy=3.141592 0 -1.570796

File: alexander-models/alexander_V1_description/urdf/alexander_v1.leftEZGripperAdapter.urdf (robot description, URDF)
Before this commit: robot Alexander, 0 links, 1 joints
Joints:
- joint LEFT_EZGRIPPER_ADAPTER: origin xyz=0 0 -0.022 rpy=3.141592 1.5708 0 -> xyz=0 0 -0.022 rpy=3.141592 1.570796 0

File: alexander-models/alexander_V1_description/urdf/alexander_v1.rightAbilityHandAdapter.urdf (robot description, URDF)
Before this commit: robot Alexander, 0 links, 1 joints
Joints:
- joint RIGHT_ABILITY_HAND_ADAPTER: origin xyz=0 0 -0.022 rpy=3.141592 0 3.141592 -> xyz=0 0 -0.022 rpy=3.141592 0 -1.570796

File: alexander-models/alexander_V1_description/urdf/alexander_v1.rightEZGripperAdapter.urdf (robot description, URDF)
Before this commit: robot Alexander, 0 links, 1 joints
Joints:
- joint RIGHT_EZGRIPPER_ADAPTER: origin xyz=0 0 -0.022 rpy=3.141592 1.5708 0 -> xyz=0 0 -0.022 rpy=3.141592 1.570796 0

Commit message: reversed left J7 motor direction and re-did zero. fixed some offsets in hand adapter urdfs

File: alexander-models/alexander_V1_description/urdf/alexander_v1.leftAbilityHandAdapter.urdf (robot description, URDF)
Before this commit: robot Alexander, 0 links, 1 joints
Joints:
- joint LEFT_ABILITY_HAND_ADAPTER: origin xyz=0 0 -0.022 rpy=3.141592 0 -1.570796 -> xyz=-0.0175 0 -0.022 rpy=3.141592 0 -1.570796

File: alexander-models/alexander_V1_description/urdf/alexander_v1.leftEZGripperAdapter.urdf (robot description, URDF)
Before this commit: robot Alexander, 0 links, 1 joints
Joints:
- joint LEFT_EZGRIPPER_ADAPTER: origin xyz=0 0 -0.022 rpy=3.141592 1.570796 0 -> xyz=0 0 -0.02 rpy=3.141592 1.570796 0

File: alexander-models/alexander_V1_description/urdf/alexander_v1.rightAbilityHandAdapter.urdf (robot description, URDF)
Before this commit: robot Alexander, 0 links, 1 joints
Joints:
- joint RIGHT_ABILITY_HAND_ADAPTER: origin xyz=0 0 -0.022 rpy=3.141592 0 -1.570796 -> xyz=-0.0175 0 -0.02 rpy=3.141592 0 -1.570796

File: alexander-models/alexander_V1_description/urdf/alexander_v1.rightEZGripperAdapter.urdf (robot description, URDF)
Before this commit: robot Alexander, 0 links, 1 joints
Joints:
- joint RIGHT_EZGRIPPER_ADAPTER: origin xyz=0 0 -0.022 rpy=3.141592 1.570796 0 -> xyz=0 0 -0.02 rpy=3.141592 1.570796 0
