Commit message: Swapping in retopologized meshes and increasing diffuse of mtl's.

File: alexander-models/alexander_V1_description/urdf/alexander_v1.fullBody.urdf (robot description, URDF)
Before this commit: robot Alexander, 41 links, 40 joints
Links:
- link LEFT_ANKLE_Y_LINK: geometry visual mesh filename=package://alexander_V1_description/meshes/legs/AnklePitchLi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
- link LEFT_FOOT: geometry visual mesh filename=package://alexander_V1_description/meshes/legs/Foot.obj
- link LEFT_HIP_X_LINK: geometry visual mesh filename=package://alexander_V1_description/meshes/legs/LeftHipRollL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
- link LEFT_HIP_Z_LINK: geometry visual mesh filename=package://alexander_V1_description/meshes/legs/LeftHipYawLi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
- link LEFT_SHIN: geometry visual mesh filename=package://alexander_V1_description/meshes/legs/LeftShin.obj
- link LEFT_THIGH: geometry visual mesh filename=package://alexander_V1_description/meshes/legs/LeftThigh.obj
- link PELVIS_LINK: geometry visual mesh filename=package://alexander_V1_description/meshes/legs/Pelvis.obj
- link RIGHT_ANKLE_Y_LINK: geometry visual mesh filename=package://alexander_V1_description/meshes/legs/AnklePitchLi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
- link RIGHT_FOOT: geometry visual mesh filename=package://alexander_V1_description/meshes/legs/Foot.obj
- link RIGHT_HIP_X_LINK: geometry visual mesh filename=package://alexander_V1_description/meshes/legs/RightHipRoll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
- link RIGHT_HIP_Z_LINK: geometry visual mesh filename=package://alexander_V1_description/meshes/legs/RightHipYawL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
- link RIGHT_SHIN: geometry visual mesh filename=package://alexander_V1_description/meshes/legs/RightShin.obj
- link RIGHT_THIGH: geometry visual mesh filename=package://alexander_V1_description/meshes/legs/RightThigh.o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

File: alexander-models/alexander_V1_description/urdf/alexander_v1.lowerBody.urdf (robot description, URDF)
Before this commit: robot Alexander, 24 links, 23 joints
Links:
- link LEFT_ANKLE_Y_LINK: geometry visual mesh filename=package://alexander_V1_description/meshes/legs/AnklePitchLi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
- link LEFT_FOOT: geometry visual mesh filename=package://alexander_V1_description/meshes/legs/Foot.obj
- link LEFT_HIP_X_LINK: geometry visual mesh filename=package://alexander_V1_description/meshes/legs/LeftHipRollL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
- link LEFT_HIP_Z_LINK: geometry visual mesh filename=package://alexander_V1_description/meshes/legs/LeftHipYawLi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
- link LEFT_SHIN: geometry visual mesh filename=package://alexander_V1_description/meshes/legs/LeftShin.obj
- link LEFT_THIGH: geometry visual mesh filename=package://alexander_V1_description/meshes/legs/LeftThigh.obj
- link PELVIS_LINK: geometry visual mesh filename=package://alexander_V1_description/meshes/legs/Pelvis.obj
- link RIGHT_ANKLE_Y_LINK: geometry visual mesh filename=package://alexander_V1_description/meshes/legs/AnklePitchLi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
- link RIGHT_FOOT: geometry visual mesh filename=package://alexander_V1_description/meshes/legs/Foot.obj
- link RIGHT_HIP_X_LINK: geometry visual mesh filename=package://alexander_V1_description/meshes/legs/RightHipRoll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
- link RIGHT_HIP_Z_LINK: geometry visual mesh filename=package://alexander_V1_description/meshes/legs/RightHipYawL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
- link RIGHT_SHIN: geometry visual mesh filename=package://alexander_V1_description/meshes/legs/RightShin.obj
- link RIGHT_THIGH: geometry visual mesh filename=package://alexander_V1_description/meshes/legs/RightThigh.o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

File: alexander-models/alexander_V1_description/urdf/alexander_v1.lowerBodyOnly.urdf (robot description, URDF)
Before this commit: robot Alexander, 23 links, 22 joints
Links:
- link LEFT_ANKLE_Y_LINK: geometry visual mesh filename=package://alexander_V1_description/meshes/legs/AnklePitchLi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
- link LEFT_FOOT: geometry visual mesh filename=package://alexander_V1_description/meshes/legs/Foot.obj
- link LEFT_HIP_X_LINK: geometry visual mesh filename=package://alexander_V1_description/meshes/legs/LeftHipRollL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
- link LEFT_HIP_Z_LINK: geometry visual mesh filename=package://alexander_V1_description/meshes/legs/LeftHipYawLi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
- link LEFT_SHIN: geometry visual mesh filename=package://alexander_V1_description/meshes/legs/LeftShin.obj
- link LEFT_THIGH: geometry visual mesh filename=package://alexander_V1_description/meshes/legs/LeftThigh.obj
- link PELVIS_LINK: geometry visual mesh filename=package://alexander_V1_description/meshes/legs/Pelvis.obj
- link RIGHT_ANKLE_Y_LINK: geometry visual mesh filename=package://alexander_V1_description/meshes/legs/AnklePitchLi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
- link RIGHT_FOOT: geometry visual mesh filename=package://alexander_V1_description/meshes/legs/Foot.obj
- link RIGHT_HIP_X_LINK: geometry visual mesh filename=package://alexander_V1_description/meshes/legs/RightHipRoll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
- link RIGHT_HIP_Z_LINK: geometry visual mesh filename=package://alexander_V1_description/meshes/legs/RightHipYawL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
- link RIGHT_SHIN: geometry visual mesh filename=package://alexander_V1_description/meshes/legs/RightShin.obj
- link RIGHT_THIGH: geometry visual mesh filename=package://alexander_V1_description/meshes/legs/RightThigh.o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

Commit message: Added imus to arms, switched to nadia ethersnacks boards

File: alexander-models/alexander_V1_description/urdf/alexander_v1.fullBody.urdf (robot description, URDF)
Before this commit: robot Alexander, 41 links, 40 joints
Links:
- added link LEFT_SHOULDER_PITCH_IMU_LINK, mass 0
- added link LEFT_SHOULDER_YAW_IMU_LINK, mass 0
- added link RIGHT_SHOULDER_PITCH_IMU_LINK, mass 0
- added link RIGHT_SHOULDER_YAW_IMU_LINK, mass 0
Joints:
- added joint LEFT_SHOULDER_PITCH_IMU_JOINT: type fixed, parent LEFT_SHOULDER_Y_LINK, child LEFT_SHOULDER_PITCH_IMU_LINK, origin xyz=0.0174 0.06944 -0.03025 rpy=-1.570796 1.570796 0, axis 0 0 1
- added joint LEFT_SHOULDER_YAW_IMU_JOINT: type fixed, parent LEFT_SHOULDER_Z_LINK, child LEFT_SHOULDER_YAW_IMU_LINK, origin xyz=-0.00763459 -0.0123324 -0.318 rpy=-1.570796 3.1415926 -0.314159, axis 0 0 1
- added joint RIGHT_SHOULDER_PITCH_IMU_JOINT: type fixed, parent RIGHT_SHOULDER_Y_LINK, child RIGHT_SHOULDER_PITCH_IMU_LINK, origin xyz=0.0175 -0.0704 -0.00778 rpy=1.570796 -1.570796 0, axis 0 0 1
- added joint RIGHT_SHOULDER_YAW_IMU_JOINT: type fixed, parent RIGHT_SHOULDER_Z_LINK, child RIGHT_SHOULDER_YAW_IMU_LINK, origin xyz=0.002 0.016 -0.318 rpy=1.570796 0 0.314159, axis 0 0 1

Commit message: added some imu definitions into urdf. added missing things into xml. reversed motor directions for right J1 and J4

File: alexander-models/alexander_V1_description/urdf/alexander_v1.fullBody.urdf (robot description, URDF)
Before this commit: robot Alexander, 45 links, 44 joints
Links:
- added link HEAD_IMU_LINK, mass 0
- added link TORSO_IMU_LINK, mass 0
Joints:
- added joint HEAD_IMU_JOINT: type fixed, parent HEAD_LINK, child HEAD_IMU_LINK, origin xyz=0.0 0.0 0.0 rpy=0.0 0 0.0, axis 0 0 1
- added joint TORSO_IMU_JOINT: type fixed, parent TORSO_LINK, child TORSO_IMU_LINK, origin xyz=0.0 0.0 0.0 rpy=0.0 0 0.0, axis 0 0 1

Commit message: Feature/adding arms (#36)
* Added information for arms and split arms into fore and aft

* Updated all the joint limits and added new cycloid configs

* Modified xmls to check if using latest codes for twitters, formatting for ethersnacks

* Added imus to arms, switched to nadia ethersnacks boards

* added some imu definitions into urdf. added missing things into xml. reversed motor directions for right J1 and J4

* updated individual body part urdfs to include IMU information

* added raw zero offsets to xmls for arms and neck actuators

* updated torso mass to include delta between expected and measured whole robot mass. scaled inertias too

* Fixed xml names for upper arm

---------

Co-authored-by: Biomech OCU <jli@ihmc.org>
Co-authored-by: Alexander OCU <rpeterson@ihmc.org>

File: alexander-models/alexander_V1_description/urdf/alexander_v1.fullBody.urdf (robot description, URDF)
Before this commit: robot Alexander, 41 links, 40 joints
Links:
- added link HEAD_IMU_LINK, mass 0
- added link LEFT_SHOULDER_PITCH_IMU_LINK, mass 0
- added link LEFT_SHOULDER_YAW_IMU_LINK, mass 0
- added link RIGHT_SHOULDER_PITCH_IMU_LINK, mass 0
- added link RIGHT_SHOULDER_YAW_IMU_LINK, mass 0
- added link TORSO_IMU_LINK, mass 0
Joints:
- added joint HEAD_IMU_JOINT: type fixed, parent HEAD_LINK, child HEAD_IMU_LINK, origin xyz=0.0 0.0 0.0 rpy=0.0 0 0.0, axis 0 0 1
- added joint LEFT_SHOULDER_PITCH_IMU_JOINT: type fixed, parent LEFT_SHOULDER_Y_LINK, child LEFT_SHOULDER_PITCH_IMU_LINK, origin xyz=0.0174 0.06944 -0.03025 rpy=-1.570796 1.570796 0, axis 0 0 1
- added joint LEFT_SHOULDER_YAW_IMU_JOINT: type fixed, parent LEFT_SHOULDER_Z_LINK, child LEFT_SHOULDER_YAW_IMU_LINK, origin xyz=-0.00763459 -0.0123324 -0.318 rpy=-1.570796 3.1415926 -0.314159, axis 0 0 1
- added joint RIGHT_SHOULDER_PITCH_IMU_JOINT: type fixed, parent RIGHT_SHOULDER_Y_LINK, child RIGHT_SHOULDER_PITCH_IMU_LINK, origin xyz=0.0175 -0.0704 -0.00778 rpy=1.570796 -1.570796 0, axis 0 0 1
- added joint RIGHT_SHOULDER_YAW_IMU_JOINT: type fixed, parent RIGHT_SHOULDER_Z_LINK, child RIGHT_SHOULDER_YAW_IMU_LINK, origin xyz=0.002 0.016 -0.318 rpy=1.570796 0 0.314159, axis 0 0 1
- added joint TORSO_IMU_JOINT: type fixed, parent TORSO_LINK, child TORSO_IMU_LINK, origin xyz=0.0 0.0 0.0 rpy=0.0 0 0.0, axis 0 0 1

File: alexander-models/alexander_V1_description/urdf/alexander_v1.head.urdf (robot description, URDF)
Before this commit: robot Alexander, 2 links, 2 joints
Links:
- added link HEAD_IMU_LINK, mass 0
Joints:
- added joint HEAD_IMU_JOINT: type fixed, parent HEAD_LINK, child HEAD_IMU_LINK, origin xyz=0.0 0.0 0.0 rpy=0.0 0 0.0, axis 0 0 1

File: alexander-models/alexander_V1_description/urdf/alexander_v1.lowerBodyOnly.urdf (robot description, URDF)
Before this commit: robot Alexander, 23 links, 22 joints
Links:
- added link TORSO_IMU_LINK, mass 0
- link TORSO_LINK: mass 4.806 -> 7.0081
Joints:
- added joint TORSO_IMU_JOINT: type fixed, parent TORSO_LINK, child TORSO_IMU_LINK, origin xyz=0.0 0.0 0.0 rpy=0.0 0 0.0, axis 0 0 1

Commit message: Feature/adding arms (#36)
* Added information for arms and split arms into fore and aft

* Updated all the joint limits and added new cycloid configs

* Modified xmls to check if using latest codes for twitters, formatting for ethersnacks

* Added imus to arms, switched to nadia ethersnacks boards

* added some imu definitions into urdf. added missing things into xml. reversed motor directions for right J1 and J4

* updated individual body part urdfs to include IMU information

* added raw zero offsets to xmls for arms and neck actuators

* updated torso mass to include delta between expected and measured whole robot mass. scaled inertias too

* Fixed xml names for upper arm

---------

Co-authored-by: Biomech OCU <jli@ihmc.org>
Co-authored-by: Alexander OCU <rpeterson@ihmc.org>

File: alexander-models/alexander_V1_description/urdf/alexander_v1.fullBody.urdf (robot description, URDF)
Before this commit: robot Alexander, 41 links, 40 joints
Links:
- added link HEAD_IMU_LINK, mass 0
- added link LEFT_SHOULDER_PITCH_IMU_LINK, mass 0
- added link LEFT_SHOULDER_YAW_IMU_LINK, mass 0
- added link RIGHT_SHOULDER_PITCH_IMU_LINK, mass 0
- added link RIGHT_SHOULDER_YAW_IMU_LINK, mass 0
- added link TORSO_IMU_LINK, mass 0
Joints:
- added joint HEAD_IMU_JOINT: type fixed, parent HEAD_LINK, child HEAD_IMU_LINK, origin xyz=0.0 0.0 0.0 rpy=0.0 0 0.0, axis 0 0 1
- added joint LEFT_SHOULDER_PITCH_IMU_JOINT: type fixed, parent LEFT_SHOULDER_Y_LINK, child LEFT_SHOULDER_PITCH_IMU_LINK, origin xyz=0.0174 0.06944 -0.03025 rpy=-1.570796 1.570796 0, axis 0 0 1
- added joint LEFT_SHOULDER_YAW_IMU_JOINT: type fixed, parent LEFT_SHOULDER_Z_LINK, child LEFT_SHOULDER_YAW_IMU_LINK, origin xyz=-0.00763459 -0.0123324 -0.318 rpy=-1.570796 3.1415926 -0.314159, axis 0 0 1
- added joint RIGHT_SHOULDER_PITCH_IMU_JOINT: type fixed, parent RIGHT_SHOULDER_Y_LINK, child RIGHT_SHOULDER_PITCH_IMU_LINK, origin xyz=0.0175 -0.0704 -0.00778 rpy=1.570796 -1.570796 0, axis 0 0 1
- added joint RIGHT_SHOULDER_YAW_IMU_JOINT: type fixed, parent RIGHT_SHOULDER_Z_LINK, child RIGHT_SHOULDER_YAW_IMU_LINK, origin xyz=0.002 0.016 -0.318 rpy=1.570796 0 0.314159, axis 0 0 1
- added joint TORSO_IMU_JOINT: type fixed, parent TORSO_LINK, child TORSO_IMU_LINK, origin xyz=0.0 0.0 0.0 rpy=0.0 0 0.0, axis 0 0 1

File: alexander-models/alexander_V1_description/urdf/alexander_v1.lowerBodyOnly.urdf (robot description, URDF)
Before this commit: robot Alexander, 23 links, 22 joints
Links:
- added link TORSO_IMU_LINK, mass 0
- link TORSO_LINK: mass 4.806 -> 7.0081
Joints:
- added joint TORSO_IMU_JOINT: type fixed, parent TORSO_LINK, child TORSO_IMU_LINK, origin xyz=0.0 0.0 0.0 rpy=0.0 0 0.0, axis 0 0 1

Commit message: Adding pelvis imu orientation offset to fullbody urdf

File: alexander-models/alexander_V1_description/urdf/alexander_v1.fullBody.urdf (robot description, URDF)
Before this commit: robot Alexander, 47 links, 46 joints
Joints:
- joint PELVIS_STIM_IMU_JOINT: origin xyz=-0.08687724 0.01225028 -0.08051472 rpy=0.0 0.0 1.570796 -> xyz=-0.08687724 0.01225028 -0.08051472 rpy=-0.01399 -0.013054 1.570796

Commit message: Added imus for forearm to full body urdf

File: alexander-models/alexander_V1_description/urdf/alexander_v1.fullBody.urdf (robot description, URDF)
Before this commit: robot Alexander, 47 links, 46 joints
Links:
- added link LEFT_GRIPPER_YAW_IMU_LINK, mass 0
- added link LEFT_WRIST_YAW_IMU_LINK, mass 0
- added link RIGHT_GRIPPER_YAW_IMU_LINK, mass 0
- added link RIGHT_WRIST_YAW_IMU_LINK, mass 0
Joints:
- added joint LEFT_GRIPPER_YAW_IMU_JOINT: type fixed, parent LEFT_GRIPPER_YAW_LINK, child LEFT_GRIPPER_YAW_IMU_LINK, origin xyz=0 0 0 rpy=0 0 0, axis 0 0 1
- added joint LEFT_WRIST_YAW_IMU_JOINT: type fixed, parent LEFT_WRIST_YAW_LINK, child LEFT_WRIST_YAW_IMU_LINK, origin xyz=-0.033554 0.010450 -0.148527 rpy=1.571  0.0 1.571, axis 0 0 1
- added joint RIGHT_GRIPPER_YAW_IMU_JOINT: type fixed, parent RIGHT_GRIPPER_YAW_LINK, child RIGHT_GRIPPER_YAW_IMU_LINK, origin xyz=0 0 0 rpy=0 0 0, axis 0 0 1
- added joint RIGHT_WRIST_YAW_IMU_JOINT: type fixed, parent RIGHT_WRIST_YAW_LINK, child RIGHT_WRIST_YAW_IMU_LINK, origin xyz=-0.033554 0.010450 -0.148527 rpy=1.571  0.0 1.571, axis 0 0 1

Commit message: Altered masses of full body urdf to match edits in lower body

File: alexander-models/alexander_V1_description/urdf/alexander_v1.fullBody.urdf (robot description, URDF)
Before this commit: robot Alexander, 51 links, 50 joints
Links:
- link LEFT_SHIN: mass 5.5 -> 6.31087157
- link RIGHT_SHIN: mass 5.5 -> 6.31087157
- link TORSO_LINK: mass 4.208 -> 7.0081

Commit message: Merge/develop to ahs 08132025 (#37)
* Retopologized meshes (#35)

* Swapping in retopologized meshes and increasing diffuse of mtl's.

* Replace .g3djs with new .glbs from Louis.

* Capitalizing Pelvis obj

---------

Co-authored-by: Duncan Calvert <dcalvert@ihmc.org>

* Added imus for forearm to full body urdf

* Altered masses of full body urdf to match edits in lower body

* Feature/alexander long (#38)

* did some general URDF cleanup

* set up a long bicep version

---------

Co-authored-by: Stephen McCrory <smccrory@ihmc.us>
Co-authored-by: Duncan Calvert <dcalvert@ihmc.org>
Co-authored-by: Robert Griffin <rjgriffin42@gmail.com>

File: alexander-models/alexander_V1_description/urdf/alexander_v1.fullBody.urdf (robot description, URDF)
Before this commit: robot Alexander, 47 links, 46 joints
Links:
- added link LEFT_GRIPPER_YAW_IMU_LINK, mass 0
- added link LEFT_WRIST_YAW_IMU_LINK, mass 0
- added link RIGHT_GRIPPER_YAW_IMU_LINK, mass 0
- added link RIGHT_WRIST_YAW_IMU_LINK, mass 0
- link LEFT_SHIN: mass 5.5 -> 6.31087157
- link RIGHT_SHIN: mass 5.5 -> 6.31087157
- link TORSO_LINK: mass 4.208 -> 7.0081
Joints:
- added joint LEFT_GRIPPER_YAW_IMU_JOINT: type fixed, parent LEFT_GRIPPER_YAW_LINK, child LEFT_GRIPPER_YAW_IMU_LINK, origin xyz=0 0 0 rpy=0 0 0, axis 0 0 1
- added joint LEFT_WRIST_YAW_IMU_JOINT: type fixed, parent LEFT_WRIST_YAW_LINK, child LEFT_WRIST_YAW_IMU_LINK, origin xyz=-0.033554 0.010450 -0.148527 rpy=1.571  0.0 1.571, axis 0 0 1
- added joint RIGHT_GRIPPER_YAW_IMU_JOINT: type fixed, parent RIGHT_GRIPPER_YAW_LINK, child RIGHT_GRIPPER_YAW_IMU_LINK, origin xyz=0 0 0 rpy=0 0 0, axis 0 0 1
- added joint RIGHT_WRIST_YAW_IMU_JOINT: type fixed, parent RIGHT_WRIST_YAW_LINK, child RIGHT_WRIST_YAW_IMU_LINK, origin xyz=-0.033554 0.010450 -0.148527 rpy=1.571  0.0 1.571, axis 0 0 1

Commit message: Merge/develop to ahs 08132025 (#37)
* Retopologized meshes (#35)

* Swapping in retopologized meshes and increasing diffuse of mtl's.

* Replace .g3djs with new .glbs from Louis.

* Capitalizing Pelvis obj

---------

Co-authored-by: Duncan Calvert <dcalvert@ihmc.org>

* Added imus for forearm to full body urdf

* Altered masses of full body urdf to match edits in lower body

* Feature/alexander long (#38)

* did some general URDF cleanup

* set up a long bicep version

---------

Co-authored-by: Stephen McCrory <smccrory@ihmc.us>
Co-authored-by: Duncan Calvert <dcalvert@ihmc.org>
Co-authored-by: Robert Griffin <rjgriffin42@gmail.com>

File: alexander-models/alexander_V1_description/urdf/alexander_v1.fullBody.urdf (robot description, URDF)
Before this commit: robot Alexander, 47 links, 46 joints
Links:
- added link LEFT_GRIPPER_YAW_IMU_LINK, mass 0
- added link LEFT_WRIST_YAW_IMU_LINK, mass 0
- added link RIGHT_GRIPPER_YAW_IMU_LINK, mass 0
- added link RIGHT_WRIST_YAW_IMU_LINK, mass 0
- link LEFT_ANKLE_Y_LINK: geometry visual mesh filename=package://alexander_V1_description/meshes/legs/AnklePitchLi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
- link LEFT_FOOT: geometry visual mesh filename=package://alexander_V1_description/meshes/legs/Foot.obj
- link LEFT_HIP_X_LINK: geometry visual mesh filename=package://alexander_V1_description/meshes/legs/LeftHipRollL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
- link LEFT_HIP_Z_LINK: geometry visual mesh filename=package://alexander_V1_description/meshes/legs/LeftHipYawLi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
- link LEFT_SHIN: mass 5.5 -> 6.31087157; geometry visual mesh filename=package://alexander_V1_description/meshes/legs/LeftShin.obj
- link LEFT_THIGH: geometry visual mesh filename=package://alexander_V1_description/meshes/legs/LeftThigh.obj
- link PELVIS_LINK: geometry visual mesh filename=package://alexander_V1_description/meshes/legs/Pelvis.obj
- link RIGHT_ANKLE_Y_LINK: geometry visual mesh filename=package://alexander_V1_description/meshes/legs/AnklePitchLi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
- link RIGHT_FOOT: geometry visual mesh filename=package://alexander_V1_description/meshes/legs/Foot.obj
- link RIGHT_HIP_X_LINK: geometry visual mesh filename=package://alexander_V1_description/meshes/legs/RightHipRoll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
- link RIGHT_HIP_Z_LINK: geometry visual mesh filename=package://alexander_V1_description/meshes/legs/RightHipYawL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
- link RIGHT_SHIN: mass 5.5 -> 6.31087157; geometry visual mesh filename=package://alexander_V1_description/meshes/legs/RightShin.obj
- link RIGHT_THIGH: geometry visual mesh filename=package://alexander_V1_description/meshes/legs/RightThigh.o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
- link TORSO_LINK: mass 4.208 -> 7.0081
Joints:
- added joint LEFT_GRIPPER_YAW_IMU_JOINT: type fixed, parent LEFT_GRIPPER_YAW_LINK, child LEFT_GRIPPER_YAW_IMU_LINK, origin xyz=0 0 0 rpy=0 0 0, axis 0 0 1
- added joint LEFT_WRIST_YAW_IMU_JOINT: type fixed, parent LEFT_WRIST_YAW_LINK, child LEFT_WRIST_YAW_IMU_LINK, origin xyz=-0.033554 0.010450 -0.148527 rpy=1.571  0.0 1.571, axis 0 0 1
- added joint RIGHT_GRIPPER_YAW_IMU_JOINT: type fixed, parent RIGHT_GRIPPER_YAW_LINK, child RIGHT_GRIPPER_YAW_IMU_LINK, origin xyz=0 0 0 rpy=0 0 0, axis 0 0 1
- added joint RIGHT_WRIST_YAW_IMU_JOINT: type fixed, parent RIGHT_WRIST_YAW_LINK, child RIGHT_WRIST_YAW_IMU_LINK, origin xyz=-0.033554 0.010450 -0.148527 rpy=1.571  0.0 1.571, axis 0 0 1

File: alexander-models/alexander_V1_description/urdf/alexander_v1.lowerBody.urdf (robot description, URDF)
Before this commit: robot Alexander, 24 links, 23 joints
Links:
- link LEFT_ANKLE_Y_LINK: geometry visual mesh filename=package://alexander_V1_description/meshes/legs/AnklePitchLi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
- link LEFT_FOOT: geometry visual mesh filename=package://alexander_V1_description/meshes/legs/Foot.obj
- link LEFT_HIP_X_LINK: geometry visual mesh filename=package://alexander_V1_description/meshes/legs/LeftHipRollL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
- link LEFT_HIP_Z_LINK: geometry visual mesh filename=package://alexander_V1_description/meshes/legs/LeftHipYawLi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
- link LEFT_SHIN: geometry visual mesh filename=package://alexander_V1_description/meshes/legs/LeftShin.obj
- link LEFT_THIGH: geometry visual mesh filename=package://alexander_V1_description/meshes/legs/LeftThigh.obj
- link PELVIS_LINK: geometry visual mesh filename=package://alexander_V1_description/meshes/legs/Pelvis.obj
- link RIGHT_ANKLE_Y_LINK: geometry visual mesh filename=package://alexander_V1_description/meshes/legs/AnklePitchLi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
- link RIGHT_FOOT: geometry visual mesh filename=package://alexander_V1_description/meshes/legs/Foot.obj
- link RIGHT_HIP_X_LINK: geometry visual mesh filename=package://alexander_V1_description/meshes/legs/RightHipRoll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
- link RIGHT_HIP_Z_LINK: geometry visual mesh filename=package://alexander_V1_description/meshes/legs/RightHipYawL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
- link RIGHT_SHIN: geometry visual mesh filename=package://alexander_V1_description/meshes/legs/RightShin.obj
- link RIGHT_THIGH: geometry visual mesh filename=package://alexander_V1_description/meshes/legs/RightThigh.o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
- link TORSO_IMU_LINK: mass 0.0 -> 0
- link TORSO_LINK: mass 4.806 -> 7.0081
Joints:
- joint TORSO_IMU_JOINT: axis (none) -> 0 0 1; origin xyz=0.04529 -0.02427 0.33757 rpy=3.141592 0 0 -> xyz=0.0 0.0 0.0 rpy=0.0 0 0.0

Commit message: resetting ankle motor kt to spreadsheet

File: alexander-models/alexander_V1_description/urdf/alexander_v1.fullBody.urdf (robot description, URDF)
Before this commit: robot Alexander, 51 links, 50 joints
Links:
- link LEFT_FOOT: geometry collision box size=0.22 0.1 0.02; visual mesh filename=package://alexander_V1_description/meshes/legs/Foot.obj
- link LEFT_HIP_X_LINK: geometry collision box size=0.02 0.12 0.10; visual mesh filename=package://alexander_V1_description/meshes/legs/LeftHipRollL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
- link LEFT_SHIN: geometry collision cylinder length=0.3 radius=0.08; visual mesh filename=package://alexander_V1_description/meshes/legs/LeftShin.obj
- link LEFT_THIGH: geometry collision box size=0.16 0.13 0.29; visual mesh filename=package://alexander_V1_description/meshes/legs/LeftThigh.obj
- link PELVIS_LINK: geometry collision box size=0.15 0.10 0.12; visual mesh filename=package://alexander_V1_description/meshes/legs/Pelvis.obj
- link RIGHT_FOOT: geometry collision box size=0.22 0.1 0.02; visual mesh filename=package://alexander_V1_description/meshes/legs/Foot.obj
- link RIGHT_HIP_X_LINK: geometry collision box size=0.02 0.12 0.10; visual mesh filename=package://alexander_V1_description/meshes/legs/RightHipRoll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
- link RIGHT_SHIN: geometry collision cylinder length=0.3 radius=0.08; visual mesh filename=package://alexander_V1_description/meshes/legs/RightShin.obj
- link RIGHT_THIGH: geometry collision box size=0.16 0.13 0.29; visual mesh filename=package://alexander_V1_description/meshes/legs/RightThigh.o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
