Commit message: Finally fixed naming convention from ROLL PITCH YAW links, IMUs, to X Y Z links, IMUs

File: alexander-models/alexander_V1_description/urdf/alexander_v1.fullBody.urdf (robot description, URDF)
Before this commit: robot Alexander, 51 links, 50 joints
Links:
- removed link LEFT_SHOULDER_PITCH_IMU_LINK
- removed link RIGHT_SHOULDER_PITCH_IMU_LINK
- added link LEFT_SHOULDER_Y_IMU_LINK, mass 0
- added link RIGHT_SHOULDER_Y_IMU_LINK, mass 0
Joints:
- removed joint LEFT_SHOULDER_PITCH_IMU_JOINT
- removed joint RIGHT_HIP_ROLL_IMU_JOINT
- removed joint RIGHT_SHOULDER_PITCH_IMU_JOINT
- added joint LEFT_SHOULDER_Y_IMU_JOINT: type fixed, parent LEFT_SHOULDER_Y_LINK, child LEFT_SHOULDER_Y_IMU_LINK, origin xyz=0.0174 0.06944 -0.03025 rpy=-1.570796 1.570796 0, axis 0 0 1
- added joint RIGHT_HIP_X_IMU_JOINT: type fixed, parent RIGHT_HIP_X_LINK, child RIGHT_HIP_X_IMU_LINK, origin xyz=-0.01922309 -0.07694987 -0.01488788 rpy=-1.570796 0 1.570796, axis 0 0 1
- added joint RIGHT_SHOULDER_Y_IMU_JOINT: type fixed, parent RIGHT_SHOULDER_Y_LINK, child RIGHT_SHOULDER_Y_IMU_LINK, origin xyz=0.0175 -0.0704 -0.00778 rpy=1.570796 -1.570796 0, axis 0 0 1

File: alexander-models/alexander_V1_description/urdf/alexander_v1.fullBodyNubForearms.urdf (robot description, URDF)
Before this commit: robot Alexander, 39 links, 38 joints
Links:
- removed link LEFT_SHOULDER_PITCH_IMU_LINK
- removed link LEFT_SHOULDER_YAW_IMU_LINK
- removed link RIGHT_SHOULDER_PITCH_IMU_LINK
- removed link RIGHT_SHOULDER_YAW_IMU_LINK
- added link LEFT_SHOULDER_Y_IMU_LINK, mass 0
- added link LEFT_SHOULDER_Z_IMU_LINK, mass 0
- added link RIGHT_SHOULDER_Y_IMU_LINK, mass 0
- added link RIGHT_SHOULDER_Z_IMU_LINK, mass 0
Joints:
- removed joint LEFT_SHOULDER_PITCH_IMU_JOINT
- removed joint LEFT_SHOULDER_YAW_IMU_JOINT
- removed joint RIGHT_SHOULDER_PITCH_IMU_JOINT
- removed joint RIGHT_SHOULDER_YAW_IMU_JOINT
- added joint LEFT_SHOULDER_Y_IMU_JOINT: type fixed, parent LEFT_SHOULDER_Y_LINK, child LEFT_SHOULDER_Y_IMU_LINK, origin xyz=0.0174 0.06944 -0.03025 rpy=-1.570796 1.570796 0, axis 0 0 1
- added joint LEFT_SHOULDER_Z_IMU_JOINT: type fixed, parent LEFT_SHOULDER_Z_LINK, child LEFT_SHOULDER_Z_IMU_LINK, origin xyz=-0.00763459 -0.0123324 -0.318 rpy=-1.570796 3.1415926 -0.314159, axis 0 0 1
- added joint RIGHT_SHOULDER_Y_IMU_JOINT: type fixed, parent RIGHT_SHOULDER_Y_LINK, child RIGHT_SHOULDER_Y_IMU_LINK, origin xyz=0.0175 -0.0704 -0.00778 rpy=1.570796 -1.570796 0, axis 0 0 1
- added joint RIGHT_SHOULDER_Z_IMU_JOINT: type fixed, parent RIGHT_SHOULDER_Z_LINK, child RIGHT_SHOULDER_Z_IMU_LINK, origin xyz=0.002 0.016 -0.318 rpy=1.570796 0 0.314159, axis 0 0 1

File: alexander-models/alexander_V1_description/urdf/alexander_v1.leftForearm.urdf (robot description, URDF)
Before this commit: robot Alexander, 4 links, 4 joints
Links:
- added link LEFT_GRIPPER_Z_IMU_LINK, mass 0
- added link LEFT_WRIST_Z_IMU_LINK, mass 0
Joints:
- added joint LEFT_GRIPPER_Z_IMU_JOINT: type fixed, parent LEFT_GRIPPER_Z_LINK, child LEFT_GRIPPER_Z_IMU_LINK, origin xyz=0 0 0 rpy=0 0 0, axis 0 0 1
- added joint LEFT_WRIST_Z_IMU_JOINT: type fixed, parent LEFT_WRIST_Z_LINK, child LEFT_WRIST_Z_IMU_LINK, origin xyz=-0.033554 0.010450 -0.148527 rpy=1.571 0.0 1.571, axis 0 0 1

File: alexander-models/alexander_V1_description/urdf/alexander_v1.leftLongUpperArm.urdf (robot description, URDF)
Before this commit: robot Alexander, 5 links, 5 joints
Links:
- removed link LEFT_SHOULDER_PITCH_IMU_LINK
- removed link LEFT_SHOULDER_YAW_IMU_LINK
- added link LEFT_SHOULDER_Y_IMU_LINK, mass 0
- added link LEFT_SHOULDER_Z_IMU_LINK, mass 0
Joints:
- removed joint LEFT_SHOULDER_PITCH_IMU_JOINT
- removed joint LEFT_SHOULDER_YAW_IMU_JOINT
- added joint LEFT_SHOULDER_Y_IMU_JOINT: type fixed, parent LEFT_SHOULDER_Y_LINK, child LEFT_SHOULDER_Y_IMU_LINK, origin xyz=0.0174 0.06944 -0.03025 rpy=-1.570796 1.570796 0, axis 0 0 1
- added joint LEFT_SHOULDER_Z_IMU_JOINT: type fixed, parent LEFT_SHOULDER_Z_LINK, child LEFT_SHOULDER_Z_IMU_LINK, origin xyz=-0.00763459 -0.0123324 -0.318 rpy=-1.570796 3.1415926 -0.314159, axis 0 0 1

File: alexander-models/alexander_V1_description/urdf/alexander_v1.leftUpperArm.urdf (robot description, URDF)
Before this commit: robot Alexander, 5 links, 5 joints
Links:
- removed link LEFT_SHOULDER_PITCH_IMU_LINK
- removed link LEFT_SHOULDER_YAW_IMU_LINK
- added link LEFT_SHOULDER_Y_IMU_LINK, mass 0
- added link LEFT_SHOULDER_Z_IMU_LINK, mass 0
Joints:
- removed joint LEFT_SHOULDER_PITCH_IMU_JOINT
- removed joint LEFT_SHOULDER_YAW_IMU_JOINT
- added joint LEFT_SHOULDER_Y_IMU_JOINT: type fixed, parent LEFT_SHOULDER_Y_LINK, child LEFT_SHOULDER_Y_IMU_LINK, origin xyz=0.0174 0.06944 -0.03025 rpy=-1.570796 1.570796 0, axis 0 0 1
- added joint LEFT_SHOULDER_Z_IMU_JOINT: type fixed, parent LEFT_SHOULDER_Z_LINK, child LEFT_SHOULDER_Z_IMU_LINK, origin xyz=-0.00763459 -0.0123324 -0.318 rpy=-1.570796 3.1415926 -0.314159, axis 0 0 1

File: alexander-models/alexander_V1_description/urdf/alexander_v1.lowerBody.urdf (robot description, URDF)
Before this commit: robot Alexander, 24 links, 23 joints
Joints:
- removed joint RIGHT_HIP_ROLL_IMU_JOINT
- added joint RIGHT_HIP_X_IMU_JOINT: type fixed, parent RIGHT_HIP_X_LINK, child RIGHT_HIP_X_IMU_LINK, origin xyz=-0.01922309 -0.07694987 -0.01488788 rpy=-1.570796 0 1.570796, axis 0 0 1

File: alexander-models/alexander_V1_description/urdf/alexander_v1.rightForearm.urdf (robot description, URDF)
Before this commit: robot Alexander, 4 links, 4 joints
Links:
- added link RIGHT_GRIPPER_Z_IMU_LINK, mass 0
- added link RIGHT_WRIST_Z_IMU_LINK, mass 0
Joints:
- added joint RIGHT_GRIPPER_Z_IMU_JOINT: type fixed, parent RIGHT_GRIPPER_Z_LINK, child RIGHT_GRIPPER_Z_IMU_LINK, origin xyz=0 0 0 rpy=0 0 0, axis 0 0 1
- added joint RIGHT_WRIST_Z_IMU_JOINT: type fixed, parent RIGHT_WRIST_Z_LINK, child RIGHT_WRIST_Z_IMU_LINK, origin xyz=-0.033554 0.010450 -0.148527 rpy=1.571  0.0 1.571, axis 0 0 1

File: alexander-models/alexander_V1_description/urdf/alexander_v1.rightLongUpperArm.urdf (robot description, URDF)
Before this commit: robot Alexander, 5 links, 5 joints
Links:
- removed link RIGHT_SHOULDER_PITCH_IMU_LINK
- removed link RIGHT_SHOULDER_YAW_IMU_LINK
- added link RIGHT_SHOULDER_Y_IMU_LINK, mass 0
- added link RIGHT_SHOULDER_Z_IMU_LINK, mass 0
Joints:
- removed joint RIGHT_SHOULDER_PITCH_IMU_JOINT
- removed joint RIGHT_SHOULDER_YAW_IMU_JOINT
- added joint RIGHT_SHOULDER_Y_IMU_JOINT: type fixed, parent RIGHT_SHOULDER_Y_LINK, child RIGHT_SHOULDER_Y_IMU_LINK, origin xyz=0.0175 -0.0704 -0.00778 rpy=1.570796 -1.570796 0, axis 0 0 1
- added joint RIGHT_SHOULDER_Z_IMU_JOINT: type fixed, parent RIGHT_SHOULDER_Z_LINK, child RIGHT_SHOULDER_Z_IMU_LINK, origin xyz=0.002 0.016 -0.318 rpy=1.570796 0 0.314159, axis 0 0 1

File: alexander-models/alexander_V1_description/urdf/alexander_v1.rightUpperArm.urdf (robot description, URDF)
Before this commit: robot Alexander, 5 links, 5 joints
Links:
- removed link RIGHT_SHOULDER_PITCH_IMU_LINK
- removed link RIGHT_SHOULDER_YAW_IMU_LINK
- added link RIGHT_SHOULDER_Y_IMU_LINK, mass 0
- added link RIGHT_SHOULDER_Z_IMU_LINK, mass 0
Joints:
- removed joint RIGHT_SHOULDER_PITCH_IMU_JOINT
- removed joint RIGHT_SHOULDER_YAW_IMU_JOINT
- added joint RIGHT_SHOULDER_Y_IMU_JOINT: type fixed, parent RIGHT_SHOULDER_Y_LINK, child RIGHT_SHOULDER_Y_IMU_LINK, origin xyz=0.0175 -0.0704 -0.00778 rpy=1.570796 -1.570796 0, axis 0 0 1
- added joint RIGHT_SHOULDER_Z_IMU_JOINT: type fixed, parent RIGHT_SHOULDER_Z_LINK, child RIGHT_SHOULDER_Z_IMU_LINK, origin xyz=0.002 0.016 -0.318 rpy=1.570796 0 0.314159, axis 0 0 1

Commit message: Fixed IMU names to match x y z link convention

File: alexander-models/alexander_V1_description/urdf/alexander_v1.fullBody.urdf (robot description, URDF)
Before this commit: robot Alexander, 51 links, 50 joints
Links:
- removed link PELVIS_STIM_IMU_LINK
- added link PELVIS_IMU_LINK, mass 0.0
Joints:
- removed joint PELVIS_STIM_IMU_JOINT
- added joint PELVIS_IMU_JOINT: type fixed, parent PELVIS_LINK, child PELVIS_IMU_LINK, origin xyz=-0.08687724 0.01225028 -0.08051472 rpy=-0.01399 -0.013054 1.570796

File: alexander-models/alexander_V1_description/urdf/alexander_v1.fullBodyNubForearms.urdf (robot description, URDF)
Before this commit: robot Alexander, 39 links, 38 joints
Links:
- removed link PELVIS_STIM_IMU_LINK
- added link PELVIS_IMU_LINK, mass 0.0
Joints:
- removed joint PELVIS_STIM_IMU_JOINT
- added joint PELVIS_IMU_JOINT: type fixed, parent PELVIS_LINK, child PELVIS_IMU_LINK, origin xyz=-0.08687724 0.01225028 -0.08051472 rpy=-0.01399 -0.013054 1.570796

File: alexander-models/alexander_V1_description/urdf/alexander_v1.lowerBody.urdf (robot description, URDF)
Before this commit: robot Alexander, 24 links, 23 joints
Links:
- removed link PELVIS_STIM_IMU_LINK
- added link PELVIS_IMU_LINK, mass 0.0
Joints:
- removed joint PELVIS_STIM_IMU_JOINT
- added joint PELVIS_IMU_JOINT: type fixed, parent PELVIS_LINK, child PELVIS_IMU_LINK, origin xyz=-0.08687724 0.01225028 -0.08051472 rpy=-0.01399 -0.013054 1.570796

Commit message: added toe and hand objects for retargeting

File: alexander-models/alexander_V1_description/urdf/alexander_v1.fullBody.urdf (robot description, URDF)
Before this commit: robot Alexander, 51 links, 50 joints
Links:
- added link LEFT_TOE_LINK, mass 0
- added link RIGHT_TOE_LINK, mass 0
Joints:
- added joint LEFT_TOE_JOINT: type fixed, parent LEFT_FOOT, child LEFT_TOE_LINK, origin xyz=0.11 0.0 -0.04 rpy=0 0 0, axis 0 0 1
- added joint RIGHT_TOE_JOINT: type fixed, parent RIGHT_FOOT, child RIGHT_TOE_LINK, origin xyz=0.11 0.0 -0.04 rpy=0 0 0, axis 0 0 1

File: alexander-models/alexander_V1_description/urdf/alexander_v1.fullBodyNubForearms.urdf (robot description, URDF)
Before this commit: robot Alexander, 39 links, 38 joints
Links:
- added link LEFT_HAND, mass 0
- added link LEFT_TOE, mass 0
- added link RIGHT_HAND, mass 0
- added link RIGHT_TOE, mass 0
Joints:
- added joint LEFT_HAND_JOINT: type fixed, parent LEFT_ELBOW_Y_LINK, child LEFT_HAND, origin xyz=0.0 0.0 -0.3 rpy=0 0 0, axis 0 0 1
- added joint LEFT_TOE_JOINT: type fixed, parent LEFT_FOOT, child LEFT_TOE, origin xyz=0.11 0.0 -0.04 rpy=0 0 0, axis 0 0 1
- added joint RIGHT_HAND_JOINT: type fixed, parent RIGHT_ELBOW_Y_LINK, child RIGHT_HAND, origin xyz=0.0 0.0 -0.3 rpy=0 0 0, axis 0 0 1
- added joint RIGHT_TOE_JOINT: type fixed, parent RIGHT_FOOT, child RIGHT_TOE, origin xyz=0.11 0.0 -0.04 rpy=0 0 0, axis 0 0 1
