Commit message: updated collisions and added numb forearms urdf's

File: alexander-models/alexander_V1_description/urdf/alexander_v1_cad_accurate_nubforarms.urdf (robot description, URDF)
Before this commit: robot Alexander, 43 links, 44 joints
Links:
- removed link LEFT_WRIST_X_LINK
- removed link LEFT_WRIST_Z_LINK
- removed link RIGHT_WRIST_X_LINK
- removed link RIGHT_WRIST_Z_LINK
- link LEFT_ELBOW_Y_LINK: mass 0.579  -> 0.69372585; geometry collision cylinder length=0.30 radius=0.04; visual mesh filename=package://alexander_V1_description/meshes/cycloidal_arm/LEF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
- link RIGHT_ELBOW_Y_LINK: mass 0.579  -> 0.69372166 ; geometry collision cylinder length=0.30 radius=0.04; visual mesh filename=package://alexander_V1_description/meshes/cycloidal_arm/RIG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
Joints:
- removed joint LEFT_GRIPPER_Z
- removed joint LEFT_WRIST_X
- removed joint LEFT_WRIST_Z
- removed joint RIGHT_GRIPPER_Z
- removed joint RIGHT_WRIST_X
- removed joint RIGHT_WRIST_Z

File: alexander-models/alexander_V1_description/urdf/alexander_v1_realLife_accurate_nubforarms.urdf (robot description, URDF)
Before this commit: robot Alexander, 43 links, 44 joints
Links:
- removed link LEFT_WRIST_X_LINK
- removed link LEFT_WRIST_Z_LINK
- removed link RIGHT_WRIST_X_LINK
- removed link RIGHT_WRIST_Z_LINK
- link LEFT_ELBOW_Y_LINK: mass 0.579  -> 0.69372585; geometry collision cylinder length=0.30 radius=0.04; visual mesh filename=package://alexander_V1_description/meshes/cycloidal_arm/LEF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
- link PELVIS_LINK: mass 9.161 -> 7.161
- link RIGHT_ELBOW_Y_LINK: mass 0.579  -> 0.69372166 ; geometry collision cylinder length=0.30 radius=0.04; visual mesh filename=package://alexander_V1_description/meshes/cycloidal_arm/RIG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
- link TORSO_LINK: mass 11.478322779 -> 10.878322779
Joints:
- removed joint LEFT_GRIPPER_Z
- removed joint LEFT_WRIST_X
- removed joint LEFT_WRIST_Z
- removed joint RIGHT_GRIPPER_Z
- removed joint RIGHT_WRIST_X
- removed joint RIGHT_WRIST_Z

File: alexander-models/alexander_V1_description/urdf/alexander_v1_realLife_accurate_total.urdf (robot description, URDF)
Before this commit: robot Alexander, 45 links, 44 joints
Links:
- link LEFT_SHIN: geometry collision cylinder length=0.3 radius=0.06; visual mesh filename=package://alexander_V1_description/meshes/legs/LeftShin.obj
- link LEFT_SHOULDER_Z_LINK: geometry collision cylinder length=0.22 radius=0.05; visual mesh filename=package://alexander_V1_description/meshes/cycloidal_arm/Lef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
- link LEFT_THIGH: geometry collision box size=0.13 0.13 0.29; visual mesh filename=package://alexander_V1_description/meshes/legs/LeftThigh.obj
- link RIGHT_SHIN: geometry collision cylinder length=0.3 radius=0.06; visual mesh filename=package://alexander_V1_description/meshes/legs/RightShin.obj
- link RIGHT_SHOULDER_Z_LINK: geometry collision cylinder length=0.22 radius=0.05; visual mesh filename=package://alexander_V1_description/meshes/cycloidal_arm/Rig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
- link RIGHT_THIGH: geometry collision box size=0.13 0.13 0.29; visual mesh filename=package://alexander_V1_description/meshes/legs/RightThigh.o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
- link TORSO_LINK: geometry collision box size=0.27 0.24 0.3; visual mesh filename=package://alexander_V1_description/meshes/torso.obj

Commit message: Also fixed the cad-accurate urdf shoulder z offsets

File: alexander-models/alexander_V1_description/urdf/alexander_v1_cad_accurate_nubforarms.urdf (robot description, URDF)
Before this commit: robot Alexander, 39 links, 38 joints
Joints:
- joint LEFT_SHOULDER_Z: origin xyz=0.0 0.035 -0.08 rpy=0.0 0.0 0.0 -> xyz=0.0 0.035 0.0 rpy=0.0 0.0 0.0
- joint RIGHT_SHOULDER_Z: origin xyz=0.0 -0.035 -0.08 rpy=0.0 0.0 0.0 -> xyz=0.0 -0.035 0.0 rpy=0.0 0.0 0.0

File: alexander-models/alexander_V1_description/urdf/alexander_v1_cad_accurate_total.urdf (robot description, URDF)
Before this commit: robot Alexander, 43 links, 44 joints
Joints:
- joint LEFT_SHOULDER_Z: origin xyz=0.0 0.035 -0.08 rpy=0.0 0.0 0.0 -> xyz=0.0 0.035 0.0 rpy=0.0 0.0 0.0
- joint RIGHT_SHOULDER_Z: origin xyz=0.0 -0.035 -0.08 rpy=0.0 0.0 0.0 -> xyz=0.0 -0.035 0.0 rpy=0.0 0.0 0.0
