Commit message: updated the urdf model a bit

File: alexander-models/alexander_V1_description/urdf/alexander_v1.lowerBody.urdf (robot description, URDF)
Before this commit: robot Alexander, 24 links, 23 joints
Links:
- link LEFT_ANKLE_Y_LINK: mass 0.04972436486 -> 0.05045632
- link LEFT_FOOT: mass 1.264275635 -> 1.28288609
- link LEFT_HIP_X_LINK: mass 1.933 -> 2.32977961
- link LEFT_HIP_Z_LINK: mass 0.777 -> 0.77281362
- link LEFT_SHIN: mass 7.400 -> 6.31087157
- link LEFT_THIGH: mass 8.200 -> 7.75
- link PELVIS_LINK: mass 7.700 -> 9.50083635
- link RIGHT_ANKLE_Y_LINK: mass 0.04972436486 -> 0.05045632
- link RIGHT_FOOT: mass 1.264275635 -> 1.28288609
- link RIGHT_HIP_X_LINK: mass 1.933 -> 2.32977248
- link RIGHT_HIP_Z_LINK: mass 0.777 -> 0.77281055
- link RIGHT_SHIN: mass 7.400 -> 6.31087157
- link RIGHT_THIGH: mass 8.200 -> 7.75
- link TORSO_LINK: mass 2.13269743 -> 4.806

File: alexander-models/alexander_V1_description/urdf/alexander_v1.lowerBodyOnly.urdf (robot description, URDF)
Before this commit: robot Alexander, 23 links, 22 joints
Links:
- link LEFT_ANKLE_Y_LINK: mass 0.04972436486 -> 0.05045632
- link LEFT_FOOT: mass 1.264275635 -> 1.28288609
- link LEFT_HIP_X_LINK: mass 1.933 -> 2.32977961
- link LEFT_HIP_Z_LINK: mass 0.777 -> 0.77281362
- link LEFT_SHIN: mass 7.400 -> 6.31087157
- link LEFT_THIGH: mass 8.200 -> 7.75
- link PELVIS_LINK: mass 7.700 -> 9.50083635
- link RIGHT_ANKLE_Y_LINK: mass 0.04972436486 -> 0.05045632
- link RIGHT_FOOT: mass 1.264275635 -> 1.28288609
- link RIGHT_HIP_X_LINK: mass 1.933 -> 2.32977248
- link RIGHT_HIP_Z_LINK: mass 0.777 -> 0.77281055
- link RIGHT_SHIN: mass 7.400 -> 6.31087157
- link RIGHT_THIGH: mass 8.200 -> 7.75
- link TORSO_LINK: mass 4.352 -> 4.806

Commit message: Feature/urdf update (#33)
* updated the urdf model a bit

* moved torso CoM offset

* modified pelvis IMU rpy

* Modified imu origins in lowerBody

---------

Co-authored-by: Robert <rgriffin@ihmc.org>
Co-authored-by: Stefan Fasano <sfasano@ihmc.org>
Co-authored-by: Biomech OCU <jli@ihmc.org>

File: alexander-models/alexander_V1_description/urdf/alexander_v1.lowerBody.urdf (robot description, URDF)
Before this commit: robot Alexander, 24 links, 23 joints
Links:
- link LEFT_ANKLE_Y_LINK: mass 0.04972436486 -> 0.05045632
- link LEFT_FOOT: mass 1.264275635 -> 1.28288609
- link LEFT_HIP_X_LINK: mass 1.933 -> 2.32977961
- link LEFT_HIP_Z_LINK: mass 0.777 -> 0.77281362
- link LEFT_SHIN: mass 7.400 -> 6.31087157
- link LEFT_THIGH: mass 8.200 -> 7.75
- link PELVIS_LINK: mass 7.700 -> 9.50083635
- link RIGHT_ANKLE_Y_LINK: mass 0.04972436486 -> 0.05045632
- link RIGHT_FOOT: mass 1.264275635 -> 1.28288609
- link RIGHT_HIP_X_LINK: mass 1.933 -> 2.32977248
- link RIGHT_HIP_Z_LINK: mass 0.777 -> 0.77281055
- link RIGHT_SHIN: mass 7.400 -> 6.31087157
- link RIGHT_THIGH: mass 8.200 -> 7.75
- link TORSO_LINK: mass 2.13269743 -> 4.806
Joints:
- joint LEFT_THIGH_IMU_JOINT: origin xyz=0.10004 0.03746 -0.21194 rpy=1.6947717585 0 1.570796 -> xyz=0.10004 0.03746 -0.21194 rpy=1.437982 0 1.570796
- joint PELVIS_STIM_IMU_JOINT: origin xyz=-0.08687724 0.01225028 -0.08051472 rpy=0.0 0.0 1.570796 -> xyz=-0.08687724 0.01225028 -0.08051472 rpy=-0.01399 -0.013054 1.570796

File: alexander-models/alexander_V1_description/urdf/alexander_v1.lowerBodyOnly.urdf (robot description, URDF)
Before this commit: robot Alexander, 23 links, 22 joints
Links:
- link LEFT_ANKLE_Y_LINK: mass 0.04972436486 -> 0.05045632
- link LEFT_FOOT: mass 1.264275635 -> 1.28288609
- link LEFT_HIP_X_LINK: mass 1.933 -> 2.32977961
- link LEFT_HIP_Z_LINK: mass 0.777 -> 0.77281362
- link LEFT_SHIN: mass 7.400 -> 6.31087157
- link LEFT_THIGH: mass 8.200 -> 7.75
- link PELVIS_LINK: mass 7.700 -> 9.50083635
- link RIGHT_ANKLE_Y_LINK: mass 0.04972436486 -> 0.05045632
- link RIGHT_FOOT: mass 1.264275635 -> 1.28288609
- link RIGHT_HIP_X_LINK: mass 1.933 -> 2.32977248
- link RIGHT_HIP_Z_LINK: mass 0.777 -> 0.77281055
- link RIGHT_SHIN: mass 7.400 -> 6.31087157
- link RIGHT_THIGH: mass 8.200 -> 7.75
- link TORSO_LINK: mass 4.352 -> 4.806
Joints:
- joint LEFT_THIGH_IMU_JOINT: origin xyz=0.10004 0.03746 -0.21194 rpy=1.6947717585 0 1.570796 -> xyz=0.10004 0.03746 -0.21194 rpy=1.437982 0 1.570796
- joint PELVIS_STIM_IMU_JOINT: origin xyz=-0.08687724 0.01225028 -0.08051472 rpy=0.0 0.0 1.570796 -> xyz=-0.08687724 0.01225028 -0.08051472 rpy=-0.01399 -0.013054 1.570796

Commit message: Fixed some incorrect link names, fixed formatting

File: alexander-models/alexander_V1_description/urdf/alexander_v1.lowerBody.urdf (robot description, URDF)
Before this commit: robot Alexander, 24 links, 23 joints
Links:
- link LEFT_FOOT: geometry collision box size=0.22 0.1 0.02; visual mesh filename=package://alexander_V1_description/meshes/legs/Foot.obj
- link LEFT_HIP_X_LINK: geometry collision box size=0.02 0.12 0.10; visual mesh filename=package://alexander_V1_description/meshes/legs/LeftHipRollL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
- link LEFT_SHIN: geometry collision cylinder length=0.3 radius=0.08; visual mesh filename=package://alexander_V1_description/meshes/legs/LeftShin.obj
- link LEFT_THIGH: geometry collision box size=0.16 0.13 0.29; visual mesh filename=package://alexander_V1_description/meshes/legs/LeftThigh.obj
- link PELVIS_LINK: geometry collision box size=0.15 0.10 0.12; visual mesh filename=package://alexander_V1_description/meshes/legs/Pelvis.obj
- link RIGHT_FOOT: geometry collision box size=0.22 0.1 0.02; visual mesh filename=package://alexander_V1_description/meshes/legs/Foot.obj
- link RIGHT_HIP_X_LINK: geometry collision box size=0.02 0.12 0.10; visual mesh filename=package://alexander_V1_description/meshes/legs/RightHipRoll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
- link RIGHT_SHIN: geometry collision cylinder length=0.3 radius=0.08; visual mesh filename=package://alexander_V1_description/meshes/legs/RightShin.obj
- link RIGHT_THIGH: geometry collision box size=0.16 0.13 0.29; visual mesh filename=package://alexander_V1_description/meshes/legs/RightThigh.o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
- link TORSO_LINK: geometry collision box size=0.275 0.33 0.43; visual mesh filename=package://alexander_V1_description/meshes/torso.obj

Commit message: temp removal of right FT and foot imu from xml and urdf (cad accurate urdf)

File: alexander-models/alexander_V1_description/urdf/alexander_v1.lowerBody.urdf (robot description, URDF)
Before this commit: robot Alexander, 24 links, 23 joints
Links:
- removed link RIGHT_FOOT_IMU_LINK
Joints:
- removed joint RIGHT_FOOT_IMU_JOINT

Commit message: removed left foot sensors from urdf and xml

File: alexander-models/alexander_V1_description/urdf/alexander_v1.lowerBody.urdf (robot description, URDF)
Before this commit: robot Alexander, 23 links, 22 joints
Links:
- removed link LEFT_FOOT_IMU_LINK
Joints:
- removed joint LEFT_FOOT_IMU_JOINT
