Commit message: fixed naming

File: alexander-models/alexander_V1_description/rl_urdf/alex_v1.rlModel_fullBody_robotAccurate_torsoFootCollisions.urdf (robot description, URDF)
Before this commit: robot Alexander, 39 links, 38 joints
Links:
- added link LEFT_GRIPPER_Z_LINK, mass 0.251; visual mesh filename=package://alexander_V1_description/meshes/cycloidal_arm/nub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
- added link LEFT_WRIST_X_LINK, mass 0.909; visual mesh filename=package://alexander_V1_description/meshes/cycloidal_arm/Lef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
- added link LEFT_WRIST_Z_LINK, mass 1.547; visual mesh filename=package://alexander_V1_description/meshes/cycloidal_arm/Lef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
- added link RIGHT_GRIPPER_Z_LINK, mass 0.251; visual mesh filename=package://alexander_V1_description/meshes/cycloidal_arm/nub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
- added link RIGHT_WRIST_X_LINK, mass 0.909; visual mesh filename=package://alexander_V1_description/meshes/cycloidal_arm/Rig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
- added link RIGHT_WRIST_Z_LINK, mass 1.547; visual mesh filename=package://alexander_V1_description/meshes/cycloidal_arm/Rig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
- link LEFT_ELBOW_Y_LINK: mass 0.69372585 -> 0.45; geometry visual mesh filename=package://alexander_V1_description/meshes/cycloidal_arm/Lef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
- link RIGHT_ELBOW_Y_LINK: mass 0.69372166  -> 0.45; geometry visual mesh filename=package://alexander_V1_description/meshes/cycloidal_arm/Rig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
- link TORSO_LINK: mass 10.878322779 -> 11.478322779
Joints:
- added joint LEFT_GRIPPER_Z: type revolute, parent LEFT_WRIST_X_LINK, child LEFT_GRIPPER_Z_LINK, origin xyz=0.0 0.013 -0.031 rpy=0.0 0.0 0.0, axis 0.0 0.0 1.0, limit lower=-2.61799 upper=2.61799 effort=20.0 velocity=25.0
- added joint LEFT_WRIST_X: type revolute, parent LEFT_WRIST_Z_LINK, child LEFT_WRIST_X_LINK, origin xyz=0.0 -0.013 -0.25 rpy=0.0 0.0 0.0, axis 1 0 0, limit lower=-1.8326 upper=0.610865 effort=20.0 velocity=25.0
- added joint LEFT_WRIST_Z: type revolute, parent LEFT_ELBOW_Y_LINK, child LEFT_WRIST_Z_LINK, origin xyz=-0.015 0.0 0.0 rpy=0.0 0.0 0.0, axis 0.0 0.0 1.0, limit lower=-2.61799 upper=2.61799 effort=20.0 velocity=25.0
- added joint RIGHT_GRIPPER_Z: type revolute, parent RIGHT_WRIST_X_LINK, child RIGHT_GRIPPER_Z_LINK, origin xyz=0.0 -0.013 -0.031 rpy=0.0 0.0 0.0, axis 0.0 0.0 1.0, limit lower=-2.61799 upper=2.61799 effort=20.0 velocity=25.0
- added joint RIGHT_WRIST_X: type revolute, parent RIGHT_WRIST_Z_LINK, child RIGHT_WRIST_X_LINK, origin xyz=0.0 0.013 -0.25 rpy=0.0 0.0 0.0, axis 1 0 0, limit lower=-0.610865 upper=1.8326 effort=20.0 velocity=25.0
- added joint RIGHT_WRIST_Z: type revolute, parent RIGHT_ELBOW_Y_LINK, child RIGHT_WRIST_Z_LINK, origin xyz=-0.015 0.0 0.0 rpy=0.0 0.0 0.0, axis 0.0 0.0 1.0, limit lower=-2.61799 upper=2.61799 effort=20.0 velocity=25.0

File: alexander-models/alexander_V1_description/rl_urdf/alex_v1.rlModel_nubForearms_robotAccurate_torsoFootCollisions.urdf (robot description, URDF)
Before this commit: robot Alexander, 45 links, 44 joints
Links:
- removed link LEFT_GRIPPER_Z_LINK
- removed link LEFT_WRIST_X_LINK
- removed link LEFT_WRIST_Z_LINK
- removed link RIGHT_GRIPPER_Z_LINK
- removed link RIGHT_WRIST_X_LINK
- removed link RIGHT_WRIST_Z_LINK
- link LEFT_ELBOW_Y_LINK: mass 0.45 -> 0.69372585; geometry visual mesh filename=package://alexander_V1_description/meshes/cycloidal_arm/LEF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
- link RIGHT_ELBOW_Y_LINK: mass 0.45 -> 0.69372166 ; geometry visual mesh filename=package://alexander_V1_description/meshes/cycloidal_arm/RIG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
- link TORSO_LINK: mass 11.478322779 -> 10.878322779
Joints:
- removed joint LEFT_GRIPPER_Z
- removed joint LEFT_WRIST_X
- removed joint LEFT_WRIST_Z
- removed joint RIGHT_GRIPPER_Z
- removed joint RIGHT_WRIST_X
- removed joint RIGHT_WRIST_Z
