Commit message: Changed hanging urdf files

File: alexander-models/alexander_V1_description/rl_urdf/alex_v1.rlModel_nubForearms_robotAccurate_fullCollisions_hanging.urdf (robot description, URDF)
Before this commit: robot Alexander, 45 links, 44 joints
Links:
- removed link temp_link2
Joints:
- removed joint joint3
- joint joint2: child temp_link2 -> rod
- joint joint4: child robot_body -> temp_link3; limit lower=-3.14 upper=3.14 effort=100 velocity=1.0 -> lower=-3.14 upper=3.14 effort=0 velocity=100.0
- joint joint5: child robot_body -> temp_link4; limit lower=-3.14 upper=3.14 effort=100 velocity=1.0 -> lower=-3.14 upper=3.14 effort=0 velocity=100.0; origin xyz=0 0 -10 rpy=0 1.57 0 -> xyz=0 0 -0.0 rpy=0 0 0; parent rod -> temp_link3
- joint joint6: child robot_body -> PELVIS_LINK; limit lower=-3.14 upper=3.14 effort=100 velocity=1.0 -> lower=-3.14 upper=3.14 effort=0 velocity=100.0; origin xyz=0 0 -10 rpy=1.57 0 0 -> xyz=0 0 -0.75 rpy=0 0 0; parent rod -> temp_link4

File: alexander-models/alexander_V1_description/rl_urdf/alex_v1.rlModel_nubForearms_robotAccurate_torsoFootCollisions_hanging.urdf (robot description, URDF)
Before this commit: robot Alexander, 45 links, 44 joints
Joints:
- joint joint4: child robot_body -> temp_link3; limit lower=-3.14 upper=3.14 effort=100 velocity=1.0 -> lower=-3.14 upper=3.14 effort=0 velocity=100.0
- joint joint5: child robot_body -> temp_link4; limit lower=-3.14 upper=3.14 effort=100 velocity=1.0 -> lower=-3.14 upper=3.14 effort=0 velocity=100.0; origin xyz=0 0 -10 rpy=0 1.57 0 -> xyz=0 0 0 rpy=0 0 0; parent rod -> temp_link3
- joint joint6: child robot_body -> PELVIS_LINK; limit lower=-3.14 upper=3.14 effort=100 velocity=1.0 -> lower=-3.14 upper=3.14 effort=0 velocity=100.0; origin xyz=0 0 -10 rpy=1.57 0 0 -> xyz=0 0 -0.75 rpy=0 0 0; parent rod -> temp_link4
