Commit message: Updated mjx masses and inertias

File: alexander-models/alexander_V1_description/rl_urdf/alex_v1.rlModel_fullBody_robotAccurate_fullCollisions.urdf (robot description, URDF)
Before this commit: robot Alexander, 45 links, 44 joints
Links:
- link LEFT_FOOT: mass 1.28831268  -> 1.28831268
- link LEFT_HIP_Z_LINK: mass 0.74972192  -> 0.74972192
- link LEFT_SHIN: mass 6.3405718  -> 6.3405718
- link LEFT_SHOULDER_X_LINK: mass 1.16160776  -> 1.16160776
- link LEFT_SHOULDER_Y_LINK: mass 3.0331992  -> 3.0331992
- link LEFT_SHOULDER_Z_LINK: mass 3.134  -> 3.134
- link RIGHT_HIP_X_LINK: mass 2.33123426  -> 2.33123426
- link RIGHT_HIP_Z_LINK: mass 0.77280715  -> 0.77280715
- link RIGHT_SHIN: mass 6.33633928  -> 6.33633928
- link RIGHT_SHOULDER_X_LINK: mass 1.1615873  -> 1.1615873
- link RIGHT_SHOULDER_Y_LINK: mass 3.00752318  -> 3.00752318
- link RIGHT_SHOULDER_Z_LINK: mass 3.10111287  -> 3.10111287
- link RIGHT_THIGH: mass 8.27617423  -> 8.27617423

Commit message: Found 8 cm offset relic from old Nadia arms

File: alexander-models/alexander_V1_description/rl_urdf/alex_v1.rlModel_fullBody_robotAccurate_fullCollisions.urdf (robot description, URDF)
Before this commit: robot Alexander, 45 links, 44 joints
Joints:
- joint LEFT_SHOULDER_Z: origin xyz=0.0 0.035 -0.08 rpy=0.0 0.0 0.0 -> xyz=0.0 0.035 0.0 rpy=0.0 0.0 0.0
- joint RIGHT_SHOULDER_Z: origin xyz=0.0 -0.035 -0.08 rpy=0.0 0.0 0.0 -> xyz=0.0 -0.035 0.0 rpy=0.0 0.0 0.0

File: alexander-models/alexander_V1_description/rl_urdf/alex_v1.rlModel_fullBody_robotAccurate_torsoFootCollisions.urdf (robot description, URDF)
Before this commit: robot Alexander, 45 links, 44 joints
Joints:
- joint LEFT_SHOULDER_Z: origin xyz=0.0 0.035 -0.08 rpy=0.0 0.0 0.0 -> xyz=0.0 0.035 0.0 rpy=0.0 0.0 0.0
- joint RIGHT_SHOULDER_Z: origin xyz=0.0 -0.035 -0.08 rpy=0.0 0.0 0.0 -> xyz=0.0 -0.035 0.0 rpy=0.0 0.0 0.0

File: alexander-models/alexander_V1_description/rl_urdf/alex_v1.rlModel_nubForearms_robotAccurate_fullCollisions.urdf (robot description, URDF)
Before this commit: robot Alexander, 39 links, 38 joints
Joints:
- joint LEFT_SHOULDER_Z: origin xyz=0.0 0.035 -0.08 rpy=0.0 0.0 0.0 -> xyz=0.0 0.035 0.0 rpy=0.0 0.0 0.0
- joint RIGHT_SHOULDER_Z: origin xyz=0.0 -0.035 -0.08 rpy=0.0 0.0 0.0 -> xyz=0.0 -0.035 0.0 rpy=0.0 0.0 0.0

File: alexander-models/alexander_V1_description/rl_urdf/alex_v1.rlModel_nubForearms_robotAccurate_torsoFootCollisions.urdf (robot description, URDF)
Before this commit: robot Alexander, 39 links, 38 joints
Joints:
- joint LEFT_SHOULDER_Z: origin xyz=0.0 0.035 -0.08 rpy=0.0 0.0 0.0 -> xyz=0.0 0.035 0.0 rpy=0.0 0.0 0.0
- joint RIGHT_SHOULDER_Z: origin xyz=0.0 -0.035 -0.08 rpy=0.0 0.0 0.0 -> xyz=0.0 -0.035 -0.0 rpy=0.0 0.0 0.0

Commit message: Fixed hip roll limits

File: alexander-models/alexander_V1_description/rl_urdf/alex_v1.rlModel_fullBody_robotAccurate_fullCollisions.urdf (robot description, URDF)
Before this commit: robot Alexander, 45 links, 44 joints
Joints:
- joint LEFT_HIP_X: limit lower=-0.3490658504 upper=0.872664626 effort=150 velocity=9 -> lower=-0.368 upper=0.872664626 effort=150 velocity=9
- joint RIGHT_HIP_X: limit lower=-0.872664626 upper=0.3490658504 effort=150 velocity=9 -> lower=-0.872664626 upper=0.368 effort=150 velocity=9

File: alexander-models/alexander_V1_description/rl_urdf/alex_v1.rlModel_fullBody_robotAccurate_torsoFootCollisions.urdf (robot description, URDF)
Before this commit: robot Alexander, 45 links, 44 joints
Joints:
- joint LEFT_HIP_X: limit lower=-0.3490658504 upper=0.872664626 effort=150 velocity=9 -> lower=-0.368 upper=0.872664626 effort=150 velocity=9
- joint RIGHT_HIP_X: limit lower=-0.872664626 upper=0.3490658504 effort=150 velocity=9 -> lower=-0.872664626 upper=0.368 effort=150 velocity=9

File: alexander-models/alexander_V1_description/rl_urdf/alex_v1.rlModel_nubForearms_robotAccurate_fullCollisions.urdf (robot description, URDF)
Before this commit: robot Alexander, 39 links, 38 joints
Joints:
- joint LEFT_HIP_X: limit lower=-0.3490658504 upper=0.872664626 effort=150 velocity=9 -> lower=-0.368 upper=0.872664626 effort=150 velocity=9
- joint RIGHT_HIP_X: limit lower=-0.872664626 upper=0.3490658504 effort=150 velocity=9 -> lower=-0.872664626 upper=0.368 effort=150 velocity=9

File: alexander-models/alexander_V1_description/rl_urdf/alex_v1.rlModel_nubForearms_robotAccurate_torsoFootCollisions.urdf (robot description, URDF)
Before this commit: robot Alexander, 39 links, 38 joints
Joints:
- joint LEFT_HIP_X: limit lower=-0.3490658504 upper=0.872664626 effort=150 velocity=9 -> lower=-0.368 upper=0.872664626 effort=150 velocity=9
- joint RIGHT_HIP_X: limit lower=-0.872664626 upper=0.3490658504 effort=150 velocity=9 -> lower=-0.872664626 upper=0.368 effort=150 velocity=9

File: alexander-models/alexander_V1_description/urdf/alexander_v1.lowerBody.urdf (robot description, URDF)
Before this commit: robot Alexander, 23 links, 22 joints
Joints:
- joint LEFT_HIP_X: limit lower=-0.3490658504 upper=0.872664626 effort=150 velocity=9 -> lower=-0.368 upper=0.872664626 effort=150 velocity=9
- joint RIGHT_HIP_X: limit lower=-0.872664626 upper=0.3490658504 effort=150 velocity=9 -> lower=-0.872664626 upper=0.368 effort=150 velocity=9

File: alexander-models/alexander_V1_description/urdf/alexander_v1_cad_accurate_nubforarms.urdf (robot description, URDF)
Before this commit: robot Alexander, 39 links, 38 joints
Joints:
- joint LEFT_HIP_X: limit lower=-0.3490658504 upper=0.872664626 effort=150 velocity=9 -> lower=-0.368 upper=0.872664626 effort=150 velocity=9
- joint RIGHT_HIP_X: limit lower=-0.872664626 upper=0.3490658504 effort=150 velocity=9 -> lower=-0.872664626 upper=0.368 effort=150 velocity=9

File: alexander-models/alexander_V1_description/urdf/alexander_v1_cad_accurate_total.urdf (robot description, URDF)
Before this commit: robot Alexander, 43 links, 44 joints
Joints:
- joint LEFT_HIP_X: limit lower=-0.3490658504 upper=0.872664626 effort=150 velocity=9 -> lower=-0.368 upper=0.872664626 effort=150 velocity=9
- joint RIGHT_HIP_X: limit lower=-0.872664626 upper=0.3490658504 effort=150 velocity=9 -> lower=-0.872664626 upper=0.368 effort=150 velocity=9
