Commit message: added new urdfs and changed knee limits on old

File: alexander-models/alexander_V1_description/rl_urdf/alex_v1.rlModel_nubForearms_robotAccurate_fullCollisions.urdf (robot description, URDF)
Before this commit: robot Alexander, 39 links, 38 joints
Joints:
- joint LEFT_KNEE_Y: limit lower=0 upper=2.445206282 effort=200 velocity=8 -> lower=0.15 upper=2.445206282 effort=200 velocity=8
- joint RIGHT_KNEE_Y: limit lower=0 upper=2.445206282 effort=200 velocity=8 -> lower=0.15 upper=2.445206282 effort=200 velocity=8

File: alexander-models/alexander_V1_description/rl_urdf/alex_v1.rlModel_nubForearms_robotAccurate_fullSphereCollisions.urdf (robot description, URDF)
Before this commit: robot Alexander, 39 links, 38 joints
Links:
- added link LEFT_FOOT_CONTACT_1, mass 0.00; collision sphere radius=0.013
- added link LEFT_FOOT_CONTACT_2, mass 0.00; collision sphere radius=0.013
- added link LEFT_FOOT_CONTACT_3, mass 0.00; collision sphere radius=0.013
- added link LEFT_FOOT_CONTACT_4, mass 0.00; collision sphere radius=0.013
- added link RIGHT_FOOT_CONTACT_1, mass 0.00; collision sphere radius=0.013
- added link RIGHT_FOOT_CONTACT_2, mass 0.00; collision sphere radius=0.013
- added link RIGHT_FOOT_CONTACT_3, mass 0.00; collision sphere radius=0.013
- added link RIGHT_FOOT_CONTACT_4, mass 0.00; collision sphere radius=0.013
- link HEAD_LINK: geometry collision sphere radius=0.14; visual mesh filename=package://alexander_V1_description/meshes/ALX02_01_A02_Head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
- link LEFT_ELBOW_Y_LINK: geometry collision cylinder length=0.30 radius=0.04; visual mesh filename=package://alexander_V1_description/meshes/cycloidal_arm/LEF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
- link LEFT_FOOT: geometry visual mesh filename=package://alexander_V1_description/meshes/legs/Foot.obj
- link LEFT_HIP_X_LINK: geometry collision box size=0.02 0.12 0.10; visual mesh filename=package://alexander_V1_description/meshes/legs/LeftHipRollL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
- link LEFT_SHIN: geometry collision cylinder length=0.3 radius=0.06; visual mesh filename=package://alexander_V1_description/meshes/legs/LeftShin.obj
- link LEFT_SHOULDER_Z_LINK: geometry collision cylinder length=0.22 radius=0.05; visual mesh filename=package://alexander_V1_description/meshes/cycloidal_arm/Lef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
- link LEFT_THIGH: geometry collision box size=0.13 0.13 0.29; visual mesh filename=package://alexander_V1_description/meshes/legs/LeftThigh.obj
- link PELVIS_LINK: geometry collision box size=0.15 0.10 0.12; visual mesh filename=package://alexander_V1_description/meshes/legs/Pelvis.obj
- link RIGHT_ELBOW_Y_LINK: geometry collision cylinder length=0.30 radius=0.04; visual mesh filename=package://alexander_V1_description/meshes/cycloidal_arm/RIG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
- link RIGHT_FOOT: geometry visual mesh filename=package://alexander_V1_description/meshes/legs/Foot.obj
- link RIGHT_HIP_X_LINK: geometry collision box size=0.02 0.12 0.10; visual mesh filename=package://alexander_V1_description/meshes/legs/RightHipRoll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
- link RIGHT_SHIN: geometry collision cylinder length=0.3 radius=0.06; visual mesh filename=package://alexander_V1_description/meshes/legs/RightShin.obj
- link RIGHT_SHOULDER_Z_LINK: geometry collision cylinder length=0.22 radius=0.05; visual mesh filename=package://alexander_V1_description/meshes/cycloidal_arm/Rig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
- link RIGHT_THIGH: geometry collision box size=0.13 0.13 0.29; visual mesh filename=package://alexander_V1_description/meshes/legs/RightThigh.o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
- link TORSO_LINK: geometry collision box size=0.27 0.24 0.3; visual mesh filename=package://alexander_V1_description/meshes/torso.obj
Joints:
- added joint LEFT_FOOT_C1_JOINT: type fixed, parent LEFT_FOOT, child LEFT_FOOT_CONTACT_1, origin xyz=0.0 0.0 0.0 rpy=0 0 0, axis 0 0 1
- added joint LEFT_FOOT_C2_JOINT: type fixed, parent LEFT_FOOT, child LEFT_FOOT_CONTACT_2, origin xyz=0.0 0.0 0.0 rpy=0 0 0, axis 0 0 1
- added joint LEFT_FOOT_C3_JOINT: type fixed, parent LEFT_FOOT, child LEFT_FOOT_CONTACT_3, origin xyz=0.0 0.0 0.0 rpy=0 0 0, axis 0 0 1
- added joint LEFT_FOOT_C4_JOINT: type fixed, parent LEFT_FOOT, child LEFT_FOOT_CONTACT_4, origin xyz=0.0 0.0 0.0 rpy=0 0 0, axis 0 0 1
- added joint RIGHT_FOOT_C1_JOINT: type fixed, parent RIGHT_FOOT, child RIGHT_FOOT_CONTACT_1, origin xyz=0.0 0.0 0.0 rpy=0 0 0, axis 0 0 1
- added joint RIGHT_FOOT_C2_JOINT: type fixed, parent RIGHT_FOOT, child RIGHT_FOOT_CONTACT_2, origin xyz=0.0 0.0 0.0 rpy=0 0 0, axis 0 0 1
- added joint RIGHT_FOOT_C3_JOINT: type fixed, parent RIGHT_FOOT, child RIGHT_FOOT_CONTACT_3, origin xyz=0.0 0.0 0.0 rpy=0 0 0, axis 0 0 1
- added joint RIGHT_FOOT_C4_JOINT: type fixed, parent RIGHT_FOOT, child RIGHT_FOOT_CONTACT_4, origin xyz=0.0 0.0 0.0 rpy=0 0 0, axis 0 0 1
- joint LEFT_KNEE_Y: limit lower=0.15 upper=2.445206282 effort=200 velocity=8 -> lower=0 upper=2.445206282 effort=200 velocity=8
- joint RIGHT_KNEE_Y: limit lower=0.15 upper=2.445206282 effort=200 velocity=8 -> lower=0 upper=2.445206282 effort=200 velocity=8
- joint RIGHT_SHOULDER_Z: origin xyz=0.0 -0.035 -0.0 rpy=0.0 0.0 0.0 -> xyz=0.0 -0.035 0.0 rpy=0.0 0.0 0.0

File: alexander-models/alexander_V1_description/rl_urdf/alex_v1.rlModel_nubForearms_robotAccurate_torsoFootCollisionsmeshes.urdf (robot description, URDF)
Before this commit: robot Alexander, 39 links, 38 joints
Links:
- link LEFT_FOOT: geometry collision mesh filename=package://alexander_V1_description/meshes/legs/Foot.obj; visual mesh filename=package://alexander_V1_description/meshes/legs/Foot.obj
- link PELVIS_LINK: geometry collision mesh filename=package://alexander_V1_description/meshes/legs/Pelvis.obj; visual mesh filename=package://alexander_V1_description/meshes/legs/Pelvis.obj
- link RIGHT_FOOT: geometry collision mesh filename=package://alexander_V1_description/meshes/legs/Foot.obj; visual mesh filename=package://alexander_V1_description/meshes/legs/Foot.obj
Joints:
- joint LEFT_KNEE_Y: limit lower=0.15 upper=2.445206282 effort=200 velocity=8 -> lower=0 upper=2.445206282 effort=200 velocity=8
- joint LEFT_SHOULDER_Z: origin xyz=0.0 0.035 0.0 rpy=0.0 0.0 0.0 -> xyz=0.0 0.035 -0.08 rpy=0.0 0.0 0.0
- joint RIGHT_KNEE_Y: limit lower=0.15 upper=2.445206282 effort=200 velocity=8 -> lower=0 upper=2.445206282 effort=200 velocity=8
- joint RIGHT_SHOULDER_Z: origin xyz=0.0 -0.035 -0.0 rpy=0.0 0.0 0.0 -> xyz=0.0 -0.035 -0.08 rpy=0.0 0.0 0.0

File: alexander-models/alexander_V1_description/rl_urdf/alex_v1.rlModel_nubForearms_robotAccurate_torsoFootSphereCollisions.urdf (robot description, URDF)
Before this commit: robot Alexander, 39 links, 38 joints
Links:
- added link LEFT_FOOT_CONTACT_1, mass 0.00; collision sphere radius=0.013
- added link LEFT_FOOT_CONTACT_2, mass 0.00; collision sphere radius=0.013
- added link LEFT_FOOT_CONTACT_3, mass 0.00; collision sphere radius=0.013
- added link LEFT_FOOT_CONTACT_4, mass 0.00; collision sphere radius=0.013
- added link RIGHT_FOOT_CONTACT_1, mass 0.00; collision sphere radius=0.013
- added link RIGHT_FOOT_CONTACT_2, mass 0.00; collision sphere radius=0.013
- added link RIGHT_FOOT_CONTACT_3, mass 0.00; collision sphere radius=0.013
- added link RIGHT_FOOT_CONTACT_4, mass 0.00; collision sphere radius=0.013
- link LEFT_FOOT: geometry visual mesh filename=package://alexander_V1_description/meshes/legs/Foot.obj
- link RIGHT_FOOT: geometry visual mesh filename=package://alexander_V1_description/meshes/legs/Foot.obj
Joints:
- added joint LEFT_FOOT_C1_JOINT: type fixed, parent LEFT_FOOT, child LEFT_FOOT_CONTACT_1, origin xyz=0.0 0.0 0.0 rpy=0 0 0, axis 0 0 1
- added joint LEFT_FOOT_C2_JOINT: type fixed, parent LEFT_FOOT, child LEFT_FOOT_CONTACT_2, origin xyz=0.0 0.0 0.0 rpy=0 0 0, axis 0 0 1
- added joint LEFT_FOOT_C3_JOINT: type fixed, parent LEFT_FOOT, child LEFT_FOOT_CONTACT_3, origin xyz=0.0 0.0 0.0 rpy=0 0 0, axis 0 0 1
- added joint LEFT_FOOT_C4_JOINT: type fixed, parent LEFT_FOOT, child LEFT_FOOT_CONTACT_4, origin xyz=0.0 0.0 0.0 rpy=0 0 0, axis 0 0 1
- added joint RIGHT_FOOT_C1_JOINT: type fixed, parent RIGHT_FOOT, child RIGHT_FOOT_CONTACT_1, origin xyz=0.0 0.0 0.0 rpy=0 0 0, axis 0 0 1
- added joint RIGHT_FOOT_C2_JOINT: type fixed, parent RIGHT_FOOT, child RIGHT_FOOT_CONTACT_2, origin xyz=0.0 0.0 0.0 rpy=0 0 0, axis 0 0 1
- added joint RIGHT_FOOT_C3_JOINT: type fixed, parent RIGHT_FOOT, child RIGHT_FOOT_CONTACT_3, origin xyz=0.0 0.0 0.0 rpy=0 0 0, axis 0 0 1
- added joint RIGHT_FOOT_C4_JOINT: type fixed, parent RIGHT_FOOT, child RIGHT_FOOT_CONTACT_4, origin xyz=0.0 0.0 0.0 rpy=0 0 0, axis 0 0 1
- joint LEFT_KNEE_Y: limit lower=0.15 upper=2.445206282 effort=200 velocity=8 -> lower=0 upper=2.445206282 effort=200 velocity=8
- joint RIGHT_KNEE_Y: limit lower=0.15 upper=2.445206282 effort=200 velocity=8 -> lower=0 upper=2.445206282 effort=200 velocity=8

Commit message: reverted joint limits on full collision

File: alexander-models/alexander_V1_description/rl_urdf/alex_v1.rlModel_nubForearms_robotAccurate_fullCollisions.urdf (robot description, URDF)
Before this commit: robot Alexander, 39 links, 38 joints
Joints:
- joint LEFT_KNEE_Y: limit lower=0.15 upper=2.445206282 effort=200 velocity=8 -> lower=0.00 upper=2.445206282 effort=200 velocity=8
- joint RIGHT_KNEE_Y: limit lower=0.15 upper=2.445206282 effort=200 velocity=8 -> lower=0.00 upper=2.445206282 effort=200 velocity=8
