Commit message: Change joint type to revolute to separate hand link from wrist link.

File: alex-models/alex_V1_description/urdf/alex_v1.leftAbilityHandAdapter.urdf (robot description, URDF)
Before this commit: robot Alex, 0 links, 1 joints
Joints:
- joint LEFT_ABILITY_HAND_ADAPTER: type fixed -> revolute

File: alex-models/alex_V1_description/urdf/alex_v1.rightAbilityHandAdapter.urdf (robot description, URDF)
Before this commit: robot Alex, 0 links, 1 joints
Joints:
- joint RIGHT_ABILITY_HAND_ADAPTER: type fixed -> revolute

Commit message: Switch back to fixed adapter joints and get the visual working.

File: alex-models/alex_V1_description/urdf/alex_v1.leftAbilityHandAdapter.urdf (robot description, URDF)
Before this commit: robot Alex, 0 links, 1 joints
Joints:
- joint LEFT_ABILITY_HAND_ADAPTER: type revolute -> fixed

File: alex-models/alex_V1_description/urdf/alex_v1.rightAbilityHandAdapter.urdf (robot description, URDF)
Before this commit: robot Alex, 0 links, 1 joints
Joints:
- joint RIGHT_ABILITY_HAND_ADAPTER: type revolute -> fixed

Commit message: Update Ability Hand Adapter URDF

File: alex-models/alex_V1_description/urdf/alex_v1.leftAbilityHandAdapter.urdf (robot description, URDF)
Before this commit: robot Alex, 0 links, 1 joints
Joints:
- joint LEFT_ABILITY_HAND_ADAPTER: origin xyz=-0.0175 0 -0.022 rpy=3.141592 0 -1.570796 -> xyz=0 -0.0175 -0.02 rpy=3.141592 0 0

File: alex-models/alex_V1_description/urdf/alex_v1.rightAbilityHandAdapter.urdf (robot description, URDF)
Before this commit: robot Alex, 0 links, 1 joints
Joints:
- joint RIGHT_ABILITY_HAND_ADAPTER: origin xyz=-0.0175 0 -0.02 rpy=3.141592 0 -1.570796 -> xyz=0 0.0175 -0.02 rpy=3.141592 0 3.141592
