Commit message: Updated arm collisions

File: alex-models/alex_V1_description/urdf/alex_v1.leftFixedForearm.urdf (robot description, URDF)
Before this commit: robot Alex, 1 links, 1 joints
Links:
- link LEFT_ELBOW_Y_LINK: geometry collision cylinder length=0.30 radius=0.04; visual mesh filename=package://alex_V1_description/meshes/cycloidal_arm/LEFT_ELB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

File: alex-models/alex_V1_description/urdf/alex_v1.leftForearm.urdf (robot description, URDF)
Before this commit: robot Alex, 6 links, 6 joints
Links:
- link LEFT_ELBOW_Y_LINK: geometry visual mesh filename=package://alex_V1_description/meshes/cycloidal_arm/LeftElbo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

File: alex-models/alex_V1_description/urdf/alex_v1.leftUpperArm.urdf (robot description, URDF)
Before this commit: robot Alex, 5 links, 5 joints
Links:
- link LEFT_SHOULDER_Z_LINK: geometry collision cylinder length=0.22 radius=0.05; visual mesh filename=package://alex_V1_description/meshes/cycloidal_arm/LeftShou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

File: alex-models/alex_V1_description/urdf/alex_v1.rightFixedForearm.urdf (robot description, URDF)
Before this commit: robot Alex, 1 links, 1 joints
Links:
- link RIGHT_ELBOW_Y_LINK: geometry collision cylinder length=0.30 radius=0.04; visual mesh filename=package://alex_V1_description/meshes/cycloidal_arm/RIGHT_EL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

File: alex-models/alex_V1_description/urdf/alex_v1.rightUpperArm.urdf (robot description, URDF)
Before this commit: robot Alex, 5 links, 5 joints
Links:
- link RIGHT_SHOULDER_Z_LINK: geometry collision cylinder length=0.22 radius=0.05; visual mesh filename=package://alex_V1_description/meshes/cycloidal_arm/RightSho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
