Commit message: Switching to mass accurate URDFs

File: alex-models/alex_V1_description/urdf/alex_v1.head.urdf (robot description, URDF)
Before this commit: robot Alex, 3 links, 3 joints
Links:
- link HEAD_LINK: mass 1.677 -> 1.27065932
- link NECK_Z_LINK: mass 1.141 -> 1.03172573

File: alex-models/alex_V1_description/urdf/alex_v1.leftForearm.urdf (robot description, URDF)
Before this commit: robot Alex, 6 links, 6 joints
Links:
- link LEFT_GRIPPER_Z_LINK: mass 0.144 -> 0.251; geometry visual mesh filename=package://alex_V1_description/meshes/cycloidal_arm/nub.obj

File: alex-models/alex_V1_description/urdf/alex_v1.leftUpperArm.urdf (robot description, URDF)
Before this commit: robot Alex, 5 links, 5 joints
Links:
- link LEFT_SHOULDER_X_LINK: mass 0.972 -> 1.16160776 
- link LEFT_SHOULDER_Y_LINK: mass 2.99 -> 3.0331992
- link LEFT_SHOULDER_Z_LINK: mass 2.91 -> 3.134 

File: alex-models/alex_V1_description/urdf/alex_v1.lowerBody.urdf (robot description, URDF)
Before this commit: robot Alex, 22 links, 21 joints
Links:
- link LEFT_FOOT: mass 1.28288609 -> 1.28831268
- link LEFT_HIP_X_LINK: mass 2.32977961 -> 2.332078
- link LEFT_HIP_Z_LINK: mass 0.77281362 -> 0.74972192 
- link LEFT_SHIN: mass 6.31087157 -> 6.3405718 
- link LEFT_THIGH: mass 7.75 -> 8.286
- link PELVIS_LINK: mass 9.50083635 -> 7.161
- link RIGHT_FOOT: mass 1.28288609 -> 1.28831268
- link RIGHT_HIP_X_LINK: mass 2.32977248 -> 2.33123426 
- link RIGHT_HIP_Z_LINK: mass 0.77281055 -> 0.77280715
- link RIGHT_SHIN: mass 6.31087157 -> 6.33633928 
- link RIGHT_THIGH: mass 7.75 -> 8.27617423 
- link TORSO_LINK: mass 7.0081 -> 11.478322779

File: alex-models/alex_V1_description/urdf/alex_v1.rightForearm.urdf (robot description, URDF)
Before this commit: robot Alex, 6 links, 6 joints
Links:
- link RIGHT_GRIPPER_Z_LINK: mass 0.144 -> 0.251; geometry visual mesh filename=package://alex_V1_description/meshes/cycloidal_arm/nub.obj

File: alex-models/alex_V1_description/urdf/alex_v1.rightUpperArm.urdf (robot description, URDF)
Before this commit: robot Alex, 5 links, 5 joints
Links:
- link RIGHT_SHOULDER_X_LINK: mass 0.972 -> 1.1615873 
- link RIGHT_SHOULDER_Y_LINK: mass 2.99 -> 3.00752318
- link RIGHT_SHOULDER_Z_LINK: mass 2.91 -> 3.10111287

File: alex-models/alex_V1_description/urdf/old/alex_v1.head.urdf (robot description, URDF)
Before this commit: robot Alex, 3 links, 3 joints
Links:
- link HEAD_LINK: mass 1.27065932 -> 1.677
- link NECK_Z_LINK: mass 1.03172573 -> 1.141

File: alex-models/alex_V1_description/urdf/old/alex_v1.leftForearm.urdf (robot description, URDF)
Before this commit: robot Alex, 6 links, 6 joints
Links:
- link LEFT_GRIPPER_Z_LINK: mass 0.251 -> 0.144; geometry visual mesh filename=package://alex_V1_description/meshes/cycloidal_arm/LeftGrip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

File: alex-models/alex_V1_description/urdf/old/alex_v1.leftUpperArm.urdf (robot description, URDF)
Before this commit: robot Alex, 5 links, 5 joints
Links:
- link LEFT_SHOULDER_X_LINK: mass 1.16160776  -> 0.972
- link LEFT_SHOULDER_Y_LINK: mass 3.0331992 -> 2.99
- link LEFT_SHOULDER_Z_LINK: mass 3.134  -> 2.91

File: alex-models/alex_V1_description/urdf/old/alex_v1.lowerBody.urdf (robot description, URDF)
Before this commit: robot Alex, 24 links, 23 joints
Links:
- removed link LEFT_FOOT_IMU_LINK
- removed link RIGHT_FOOT_IMU_LINK
- link LEFT_FOOT: mass 1.28831268 -> 1.28288609
- link LEFT_HIP_X_LINK: mass 2.332078 -> 2.32977961
- link LEFT_HIP_Z_LINK: mass 0.74972192  -> 0.77281362
- link LEFT_SHIN: mass 6.3405718  -> 6.31087157
- link LEFT_THIGH: mass 8.286 -> 7.75
- link PELVIS_LINK: mass 7.161 -> 9.50083635
- link RIGHT_FOOT: mass 1.28831268 -> 1.28288609
- link RIGHT_HIP_X_LINK: mass 2.33123426  -> 2.32977248
- link RIGHT_HIP_Z_LINK: mass 0.77280715 -> 0.77281055
- link RIGHT_SHIN: mass 6.33633928  -> 6.31087157
- link RIGHT_THIGH: mass 8.27617423  -> 7.75
- link TORSO_LINK: mass 11.478322779 -> 7.0081
Joints:
- removed joint LEFT_FOOT_IMU_JOINT
- removed joint RIGHT_FOOT_IMU_JOINT

File: alex-models/alex_V1_description/urdf/old/alex_v1.rightForearm.urdf (robot description, URDF)
Before this commit: robot Alex, 6 links, 6 joints
Links:
- link RIGHT_GRIPPER_Z_LINK: mass 0.251 -> 0.144; geometry visual mesh filename=package://alex_V1_description/meshes/cycloidal_arm/RightGri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

File: alex-models/alex_V1_description/urdf/old/alex_v1.rightUpperArm.urdf (robot description, URDF)
Before this commit: robot Alex, 5 links, 5 joints
Links:
- link RIGHT_SHOULDER_X_LINK: mass 1.1615873  -> 0.972
- link RIGHT_SHOULDER_Y_LINK: mass 3.00752318 -> 2.99
- link RIGHT_SHOULDER_Z_LINK: mass 3.10111287 -> 2.91

Commit message: Fixed some collisions, added hanging chain for hanging urdfs

File: alex-models/alex_V1_description/urdf/alex_v1.head.urdf (robot description, URDF)
Before this commit: robot Alex, 3 links, 3 joints
Links:
- link HEAD_LINK: geometry collision sphere radius=0.14; visual mesh filename=package://alex_V1_description/meshes/ALX02_01_A02_HeadLink.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

File: alex-models/alex_V1_description/urdf/alex_v1.lowerBody.urdf (robot description, URDF)
Before this commit: robot Alex, 22 links, 21 joints
Links:
- link LEFT_SHIN: geometry collision cylinder length=0.3 radius=0.06; visual mesh filename=package://alex_V1_description/meshes/legs/LeftShin.obj
- link LEFT_THIGH: geometry collision box size=0.13 0.13 0.29; visual mesh filename=package://alex_V1_description/meshes/legs/LeftThigh.obj
- link RIGHT_SHIN: geometry collision cylinder length=0.3 radius=0.06; visual mesh filename=package://alex_V1_description/meshes/legs/RightShin.obj
- link RIGHT_THIGH: geometry collision box size=0.13 0.13 0.29; visual mesh filename=package://alex_V1_description/meshes/legs/RightThigh.obj
- link TORSO_LINK: geometry collision box size=0.27 0.24 0.3; visual mesh filename=package://alex_V1_description/meshes/torso.obj
