Commit message: Revert "Merge branch 'develop' into feature/alex-full-convex"
This reverts commit 8cedf7465d66bde9361a63a2e6d48d65778df130, reversing
changes made to 8d03a7ce682bee1433ddec977266ea8b61e3980d.

File: alex-models/alex_V1_description/urdf/alex_v1.head.urdf (robot description, URDF)
Before this commit: robot Alex, 4 links, 4 joints
Links:
- removed link HEAD_ZED_X_MINI_LINK
Joints:
- removed joint HEAD_ZED_X_MINI_JOINT

File: alex-models/alex_V1_description/urdf/alex_v1.lowerBody.urdf (robot description, URDF)
Before this commit: robot Alex, 23 links, 22 joints
Links:
- removed link TORSO_ZED_X_MINI_LINK
Joints:
- removed joint TORSO_ZED_X_MINI_JOINT
