Commit message: Averaged left and right upper arm masses and inertias

File: alex-models/alex_V1_description/urdf/alex_v1.leftUpperArm.urdf (robot description, URDF)
Before this commit: robot Alex, 5 links, 5 joints
Links:
- link LEFT_SHOULDER_X_LINK: mass 1.16160776  -> 1.16159753
- link LEFT_SHOULDER_Y_LINK: mass 3.0331992 -> 3.02036119
- link LEFT_SHOULDER_Z_LINK: mass 3.134  -> 3.117556435

File: alex-models/alex_V1_description/urdf/alex_v1.rightUpperArm.urdf (robot description, URDF)
Before this commit: robot Alex, 5 links, 5 joints
Links:
- link RIGHT_SHOULDER_X_LINK: mass 1.1615873  -> 1.16159753
- link RIGHT_SHOULDER_Y_LINK: mass 3.00752318 -> 3.02036119
- link RIGHT_SHOULDER_Z_LINK: mass 3.10111287 -> 3.117556435
