Commit message: finished modifying the urdf directory

File: alex-models/alex_V1_description/urdf/alex_v1.fullBody.urdf (robot description, URDF)
Before this commit: robot Alex, 47 links, 46 joints
Links:
- added link LEFT_SHOULDER_Y_IMU_LINK, mass 0
Joints:
- added joint LEFT_SHOULDER_Y_IMU_JOINT: type fixed, parent LEFT_SHOULDER_Y_LINK, child LEFT_SHOULDER_Y_IMU_LINK, origin xyz=0.0174 0.06944 -0.03025 rpy=-1.570796 1.570796 0, axis 0 0 1

File: alex-models/alex_V1_description/urdf/alex_v1.fullBodyNubForearms.urdf (robot description, URDF)
Before this commit: robot Alex, 37 links, 36 joints
Links:
- link LEFT_SHOULDER_X_LINK: mass 1.17068 -> 1.16160776 
- link LEFT_SHOULDER_Y_LINK: mass 2.99 -> 3.0331992
- link LEFT_SHOULDER_Z_LINK: mass 2.91 -> 3.134 ; geometry collision cylinder length=0.15 radius=0.05; visual mesh filename=package://alex_V1_description/meshes/cycloidal_arm/LeftShou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
- link RIGHT_SHOULDER_X_LINK: mass 1.17068 -> 1.1615873 
- link RIGHT_SHOULDER_Y_LINK: mass 2.99 -> 3.00752318
- link RIGHT_SHOULDER_Z_LINK: mass 2.91 -> 3.10111287; geometry collision cylinder length=0.15 radius=0.05; visual mesh filename=package://alex_V1_description/meshes/cycloidal_arm/RightSho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

File: alex-models/alex_V1_description/urdf/alex_v1.leftFixedForearm.urdf (robot description, URDF)
Before this commit: robot Alex, 1 links, 1 joints
Links:
- link LEFT_ELBOW_Y_LINK: geometry collision cylinder length=0.34 radius=0.033; visual mesh filename=package://alex_V1_description/meshes/cycloidal_arm/LEFT_ELB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

File: alex-models/alex_V1_description/urdf/alex_v1.rightFixedForearm.urdf (robot description, URDF)
Before this commit: robot Alex, 1 links, 1 joints
Links:
- link RIGHT_ELBOW_Y_LINK: geometry collision cylinder length=0.34 radius=0.033; visual mesh filename=package://alex_V1_description/meshes/cycloidal_arm/RIGHT_EL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

Commit message: full body feet update

File: alex-models/alex_V1_description/urdf/alex_v1.fullBody.urdf (robot description, URDF)
Before this commit: robot Alex, 49 links, 48 joints
Links:
- link LEFT_FOOT: mass 1.28831268  -> 1.28831268
