Commit message: extra frames for toes and nub tips

File: alex-models/alex_V1_description/urdf/alex_v1.leftNub.urdf (robot description, URDF)
Before this commit: robot Alex, 1 links, 1 joints
Links:
- added link LEFT_NUB_TIP, mass 0.0; visual sphere radius=0.001
Joints:
- added joint LEFT_NUB_TIP_FIXED: type fixed, parent LEFT_NUB, child LEFT_NUB_TIP, origin xyz=-0.01 0.0 -0.4 rpy=0 0 0

File: alex-models/alex_V1_description/urdf/alex_v1.lowerBody.urdf (robot description, URDF)
Before this commit: robot Alex, 22 links, 21 joints
Links:
- added link LEFT_TOE_LINK, mass 0.0; visual sphere radius=0.001
- added link RIGHT_TOE_LINK, mass 0.0; visual sphere radius=0.001
Joints:
- added joint LEFT_TOE_FIXED: type fixed, parent LEFT_FOOT, child LEFT_TOE_LINK, origin xyz=0.11 0 -0.06 rpy=0 0 0
- added joint RIGHT_TOE_FIXED: type fixed, parent RIGHT_FOOT, child RIGHT_TOE_LINK, origin xyz=0.11 0 -0.06 rpy=0 0 0

File: alex-models/alex_V1_description/urdf/alex_v1.rightNub.urdf (robot description, URDF)
Before this commit: robot Alex, 1 links, 1 joints
Links:
- added link RIGHT_NUB_TIP, mass 0.0; visual sphere radius=0.001
Joints:
- added joint RIGHT_NUB_TIP_FIXED: type fixed, parent RIGHT_NUB, child RIGHT_NUB_TIP, origin xyz=-0.01 0.0 -0.4 rpy=0 0 0
