Commit message: Reverted forearm to use hands instead of nubs

File: alex-models/alex_V1_description/urdf/alex_v1.leftForearm.urdf (robot description, URDF)
Before this commit: robot Alex, 6 links, 6 joints
Links:
- link LEFT_GRIPPER_Z_LINK: mass 0.251 -> 0.144; geometry visual mesh filename=package://alex_V1_description/meshes/cycloidal_arm/LeftGrip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

File: alex-models/alex_V1_description/urdf/alex_v1.rightForearm.urdf (robot description, URDF)
Before this commit: robot Alex, 6 links, 6 joints
Links:
- link RIGHT_GRIPPER_Z_LINK: mass 0.251 -> 0.144; geometry visual mesh filename=package://alex_V1_description/meshes/cycloidal_arm/RightGri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

Commit message: Fixed some very messed up inertias in forearms

File: alex-models/alex_V1_description/urdf/alex_v1.leftForearm.urdf (robot description, URDF)
Before this commit: robot Alex, 6 links, 6 joints
Links:
- link LEFT_GRIPPER_Z_LINK: mass 0.144 -> 0.287

File: alex-models/alex_V1_description/urdf/alex_v1.rightForearm.urdf (robot description, URDF)
Before this commit: robot Alex, 6 links, 6 joints
Links:
- link RIGHT_GRIPPER_Z_LINK: mass 0.144 -> 0.287

Commit message: Revert "Fix mass and inertia assymetry (#82)"
This reverts commit cb217fd040fe13abd19c655a650513a6220ff69a.

File: alex-models/alex_V1_description/urdf/alex_v1.leftForearm.urdf (robot description, URDF)
Before this commit: robot Alex, 6 links, 6 joints
Links:
- link LEFT_GRIPPER_Z_LINK: mass 0.287 -> 0.144

File: alex-models/alex_V1_description/urdf/alex_v1.leftUpperArm.urdf (robot description, URDF)
Before this commit: robot Alex, 5 links, 5 joints
Links:
- link LEFT_SHOULDER_X_LINK: mass 1.16159753 -> 1.16160776 
- link LEFT_SHOULDER_Y_LINK: mass 3.02036119 -> 3.0331992
- link LEFT_SHOULDER_Z_LINK: mass 3.117556435 -> 3.134 

File: alex-models/alex_V1_description/urdf/alex_v1.lowerBody.urdf (robot description, URDF)
Before this commit: robot Alex, 22 links, 21 joints
Links:
- link LEFT_HIP_X_LINK: mass 2.33165613 -> 2.332078
- link LEFT_HIP_Z_LINK: mass 0.761264535 -> 0.74972192 
- link LEFT_SHIN: mass 6.33845554 -> 6.3405718 
- link LEFT_THIGH: mass 8.281087115 -> 8.286
- link RIGHT_HIP_X_LINK: mass 2.33165613 -> 2.33123426 
- link RIGHT_HIP_Z_LINK: mass 0.761264535 -> 0.77280715
- link RIGHT_SHIN: mass 6.33845554 -> 6.33633928 
- link RIGHT_THIGH: mass 8.281087115 -> 8.27617423 

File: alex-models/alex_V1_description/urdf/alex_v1.rightForearm.urdf (robot description, URDF)
Before this commit: robot Alex, 6 links, 6 joints
Links:
- link RIGHT_GRIPPER_Z_LINK: mass 0.287 -> 0.144

File: alex-models/alex_V1_description/urdf/alex_v1.rightUpperArm.urdf (robot description, URDF)
Before this commit: robot Alex, 5 links, 5 joints
Links:
- link RIGHT_SHOULDER_X_LINK: mass 1.16159753 -> 1.1615873 
- link RIGHT_SHOULDER_Y_LINK: mass 3.02036119 -> 3.00752318
- link RIGHT_SHOULDER_Z_LINK: mass 3.117556435 -> 3.10111287

File: alex-models/alex_V2_description/urdf/alex_v2.leftUpperArm.urdf (robot description, URDF)
Before this commit: robot Alex, 5 links, 5 joints
Links:
- link LEFT_SHOULDER_X_LINK: mass 1.16159753 -> 0.972
- link LEFT_SHOULDER_Y_LINK: mass 3.02036119 -> 2.99
- link LEFT_SHOULDER_Z_LINK: mass 3.117556435 -> 2.91
Joints:
- joint LEFT_SHOULDER_X: limit lower=-0.349066 upper=2.79253 effort=160.7 velocity=10.38 -> lower=-0.349066 upper=2.79253 effort=150.0 velocity=9.0
- joint LEFT_SHOULDER_Y: limit lower=-3.141592 upper=1.22173 effort=160.7 velocity=10.38 -> lower=-3.141592 upper=1.22173 effort=150.0 velocity=9.0
- joint LEFT_SHOULDER_Z: limit lower=-1.91986 upper=1.22173 effort=71.28 velocity=4.47 -> lower=-1.91986 upper=1.22173 effort=80.0 velocity=11.5

File: alex-models/alex_V2_description/urdf/alex_v2.lowerBody.urdf (robot description, URDF)
Before this commit: robot Alex, 21 links, 20 joints
Links:
- link LEFT_FOOT: mass 1.28831268 -> 1.28288609
- link LEFT_HIP_X_LINK: mass 2.33165613 -> 2.32977961
- link LEFT_HIP_Z_LINK: mass 0.761264535 -> 0.77281362
- link LEFT_SHIN: mass 6.33845554 -> 6.31087157
- link LEFT_THIGH: mass 8.281087115 -> 7.75
- link PELVIS_LINK: mass 7.161 -> 9.50083635
- link RIGHT_FOOT: mass 1.28831268 -> 1.28288609
- link RIGHT_HIP_X_LINK: mass 2.33165613 -> 2.32977248
- link RIGHT_HIP_Z_LINK: mass 0.761264535 -> 0.77281055
- link RIGHT_SHIN: mass 6.33845554 -> 6.31087157
- link RIGHT_THIGH: mass 8.281087115 -> 7.75
Joints:
- joint LEFT_ANKLE_X: limit lower=-0.436332 upper=0.436332 effort=145.2 velocity=9.72 -> lower=-0.436332 upper=0.436332 effort=90 velocity=8
- joint LEFT_ANKLE_Y: limit lower=-1.0472 upper=0.523599 effort=193.6 velocity=9.72 -> lower=-1.0472 upper=0.523599 effort=180 velocity=8
- joint LEFT_HIP_X: limit lower=-0.488692 upper=0.872665 effort=160.7 velocity=10.38 -> lower=-0.3490658504 upper=0.872664626 effort=150 velocity=9
- joint LEFT_HIP_Y: limit lower=-2.61799 upper=0.785398 effort=217.2 velocity=9.3 -> lower=-2.61799 upper=0.785398 effort=200 velocity=8
- joint LEFT_HIP_Z: limit lower=-0.349066 upper=1.0472 effort=70.5 velocity=10.59 -> lower=-0.3490658504 upper=1.0472 effort=60 velocity=11
- joint LEFT_KNEE_Y: limit lower=0 upper=2.44346 effort=217.2 velocity=9.3 -> lower=0 upper=2.445206282 effort=200 velocity=8
- joint RIGHT_ANKLE_X: limit lower=-0.436332 upper=0.436332 effort=145.2 velocity=9.72 -> lower=-0.436332 upper=0.436332 effort=90 velocity=8
- joint RIGHT_ANKLE_Y: limit lower=-1.0472 upper=0.523599 effort=193.6 velocity=9.72 -> lower=-1.0472 upper=0.523599 effort=180 velocity=8
- joint RIGHT_HIP_X: limit lower=-0.872665 upper=0.488692 effort=160.7 velocity=10.38 -> lower=-0.872664626 upper=0.3490658504 effort=150 velocity=9
- joint RIGHT_HIP_Y: limit lower=-2.61799 upper=0.785398 effort=217.2 velocity=9.3 -> lower=-2.61799 upper=0.785398 effort=200 velocity=8
- joint RIGHT_HIP_Z: limit lower=-1.0472 upper=0.349066 effort=70.5 velocity=10.59 -> lower=-1.0472 upper=0.3490658504 effort=60 velocity=11
- joint RIGHT_KNEE_Y: limit lower=0 upper=2.44346 effort=217.2 velocity=9.3 -> lower=0 upper=2.445206282 effort=200 velocity=8
- joint SPINE_Z: limit lower=-0.523599 upper=0.523599 effort=160.7 velocity=10.38 -> lower=-0.5235987756 upper=0.5235987756 effort=150 velocity=9.0

File: alex-models/alex_V2_description/urdf/alex_v2.rightUpperArm.urdf (robot description, URDF)
Before this commit: robot Alex, 5 links, 5 joints
Links:
- link RIGHT_SHOULDER_X_LINK: mass 1.16159753 -> 0.972
- link RIGHT_SHOULDER_Y_LINK: mass 3.02036119 -> 2.99
- link RIGHT_SHOULDER_Z_LINK: mass 3.117556435 -> 2.91
Joints:
- joint RIGHT_SHOULDER_X: limit lower=-2.79253 upper=0.349066 effort=160.7 velocity=10.38 -> lower=-2.79253 upper=0.349066 effort=1000 velocity=100
- joint RIGHT_SHOULDER_Y: limit lower=-3.141592 upper=1.22173 effort=160.7 velocity=10.38 -> lower=-3.141592 upper=1.22173 effort=1000 velocity=100
- joint RIGHT_SHOULDER_Z: limit lower=-1.22173 upper=1.91986 effort=71.28 velocity=4.47 -> lower=-1.22173 upper=1.91986 effort=1000 velocity=100

Commit message: Added hand collisions on wrist for RL

File: alex-models/alex_V1_description/urdf/alex_v1.leftForearm.urdf (robot description, URDF)
Before this commit: robot Alex, 6 links, 6 joints
Links:
- link LEFT_GRIPPER_Z_LINK: geometry collision box size=0.08 0.025 0.075; collision cylinder length=0.06 radius=0.047

File: alex-models/alex_V1_description/urdf/alex_v1.rightForearm.urdf (robot description, URDF)
Before this commit: robot Alex, 6 links, 6 joints
Links:
- link RIGHT_GRIPPER_Z_LINK: geometry collision box size=0.08 0.025 0.075; collision cylinder length=0.06 radius=0.047

Commit message: updated the collisions for the forearms, thighs, and shins

File: alex-models/alex_V1_description/urdf/alex_v1.leftForearm.urdf (robot description, URDF)
Before this commit: robot Alex, 6 links, 6 joints
Links:
- link LEFT_ELBOW_Y_LINK: geometry collision capsule length=0.18 radius=0.05; visual mesh filename=package://alex_V1_description/meshes/cycloidal_arm/LeftElbo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
- link LEFT_GRIPPER_Z_LINK: geometry collision box size=0.08 0.025 0.075; collision capsule length=0.1 radius=0.04

File: alex-models/alex_V1_description/urdf/alex_v1.lowerBody.urdf (robot description, URDF)
Before this commit: robot Alex, 22 links, 21 joints
Links:
- link LEFT_SHIN: geometry collision capsule length=0.11 radius=0.065; collision capsule length=0.3 radius=0.06
- link LEFT_THIGH: geometry collision capsule length=0.26 radius=0.08; collision cylinder length=0.155 radius=0.03
- link RIGHT_SHIN: geometry collision capsule length=0.11 radius=0.065; collision capsule length=0.3 radius=0.06
- link RIGHT_THIGH: geometry collision capsule length=0.26 radius=0.08; collision cylinder length=0.155 radius=0.03

File: alex-models/alex_V1_description/urdf/alex_v1.rightForearm.urdf (robot description, URDF)
Before this commit: robot Alex, 6 links, 6 joints
Links:
- link RIGHT_ELBOW_Y_LINK: geometry collision capsule length=0.18 radius=0.05; visual mesh filename=package://alex_V1_description/meshes/cycloidal_arm/RightElb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
- link RIGHT_GRIPPER_Z_LINK: geometry collision box size=0.08 0.025 0.075; collision capsule length=0.1 radius=0.04
