Commit message: Averaged the lower body masses and inertias

File: alex-models/alex_V1_description/urdf/alex_v1.lowerBody.urdf (robot description, URDF)
Before this commit: robot Alex, 22 links, 21 joints
Links:
- link LEFT_HIP_X_LINK: mass 2.332078 -> 2.33165613
- link LEFT_HIP_Z_LINK: mass 0.74972192  -> 0.761264535
- link LEFT_SHIN: mass 6.3405718  -> 6.33845554
- link LEFT_THIGH: mass 8.286 -> 8.281087115
- link RIGHT_HIP_X_LINK: mass 2.33123426  -> 2.33165613
- link RIGHT_HIP_Z_LINK: mass 0.77280715 -> 0.761264535
- link RIGHT_SHIN: mass 6.33633928  -> 6.33845554
- link RIGHT_THIGH: mass 8.27617423  -> 8.281087115

Commit message: avatar alex

File: alex-models/alex_V1_description/urdf/alex_v1.lowerBody.urdf (robot description, URDF)
Before this commit: robot Alex, 22 links, 21 joints
Links:
- link LEFT_FOOT: mass 0.810 -> 1.28831268
- link LEFT_HIP_X_LINK: mass 2.33165613 -> 2.332078
- link LEFT_HIP_Z_LINK: mass 0.761264535 -> 0.74972192 
- link LEFT_SHIN: mass 6.33845554 -> 6.3405718 
- link LEFT_THIGH: mass 8.281087115 -> 8.286
- link RIGHT_FOOT: mass 0.810 -> 1.28831268
- link RIGHT_HIP_X_LINK: mass 2.33165613 -> 2.33123426 
- link RIGHT_HIP_Z_LINK: mass 0.761264535 -> 0.77280715
- link RIGHT_SHIN: mass 6.33845554 -> 6.33633928 
- link RIGHT_THIGH: mass 8.281087115 -> 8.27617423 

Commit message: updated feet mass, inertia and com

File: alex-models/alex_V1_description/urdf/alex_v1.lowerBody.urdf (robot description, URDF)
Before this commit: robot Alex, 22 links, 21 joints
Links:
- link LEFT_FOOT: mass 0.810 -> 0.799
- link RIGHT_FOOT: mass 0.810 -> 0.799

Commit message: Fixed the limit of hip roll for both, updated some joint zeros for V2

File: alex-models/alex_V1_description/urdf/alex_v1.lowerBody.urdf (robot description, URDF)
Before this commit: robot Alex, 22 links, 21 joints
Joints:
- joint LEFT_HIP_X: limit lower=-0.488692 upper=0.872665 effort=160.7 velocity=10.38 -> lower=-0.36792 upper=0.872665 effort=160.7 velocity=10.38
- joint RIGHT_HIP_X: limit lower=-0.872665 upper=0.488692 effort=160.7 velocity=10.38 -> lower=-0.872665 upper=0.36792 effort=160.7 velocity=10.38

File: alex-models/alex_V2_description/urdf/alex_v2.lowerBody.urdf (robot description, URDF)
Before this commit: robot Alex, 22 links, 21 joints
Joints:
- joint LEFT_HIP_X: limit lower=-0.488692 upper=0.872665 effort=160.7 velocity=10.38 -> lower=-0.36792 upper=0.872665 effort=160.7 velocity=10.38
- joint RIGHT_HIP_X: limit lower=-0.872665 upper=0.488692 effort=160.7 velocity=10.38 -> lower=-0.872665 upper=0.36792 effort=160.7 velocity=10.38

Commit message: Rolled back v1 changes, added robot specific roll changes to v2

File: alex-models/alex_V1_description/urdf/alex_v1.lowerBody.urdf (robot description, URDF)
Before this commit: robot Alex, 22 links, 21 joints
Joints:
- joint LEFT_HIP_X: limit lower=-0.36792 upper=0.872665 effort=160.7 velocity=10.38 -> lower=-0.488692 upper=0.872665 effort=160.7 velocity=10.38
- joint RIGHT_HIP_X: limit lower=-0.872665 upper=0.36792 effort=160.7 velocity=10.38 -> lower=-0.872665 upper=0.488692 effort=160.7 velocity=10.38

File: alex-models/alex_V2_description/urdf/alex_v2.lowerBody.urdf (robot description, URDF)
Before this commit: robot Alex, 22 links, 21 joints
Joints:
- joint LEFT_HIP_X: limit lower=-0.36792 upper=0.872665 effort=160.7 velocity=10.38 -> lower=-0.349066 upper=0.872665 effort=160.7 velocity=10.38
- joint RIGHT_HIP_X: limit lower=-0.872665 upper=0.36792 effort=160.7 velocity=10.38 -> lower=-0.872665 upper=0.349066 effort=160.7 velocity=10.38

Commit message: WIP - adding ZEDs to URDF

File: alex-models/alex_V1_description/urdf/alex_v1.lowerBody.urdf (robot description, URDF)
Before this commit: robot Alex, 22 links, 21 joints
Links:
- added link TORSO_ZED_X_MINI_LINK, mass 0; visual mesh filename=package://alex_V1_description/meshes/ZEDXMini.obj
Joints:
- added joint TORSO_ZED_X_MINI_JOINT: type fixed, parent TORSO_LINK, child TORSO_ZED_X_MINI_LINK, origin xyz=0.1 0.0 0.05 rpy=0.0 0.907571 0.0

File: alex-models/alex_V2_description/urdf/alex_v2.head.urdf (robot description, URDF)
Before this commit: robot Alex, 3 links, 3 joints
Links:
- added link HEAD_ZED_X_MINI_LINK, mass 0; visual mesh filename=package://alex_V1_description/meshes/ZEDXMini.obj
Joints:
- added joint HEAD_ZED_X_MINI_JOINT: type fixed, parent HEAD_LINK, child HEAD_ZED_X_MINI_LINK, origin xyz=0.13041 -0.01079 0.02381 rpy=0.0 0.3633 0.0

File: alex-models/alex_V2_description/urdf/alex_v2.lowerBody.urdf (robot description, URDF)
Before this commit: robot Alex, 22 links, 21 joints
Links:
- added link TORSO_ZED_X_MINI_LINK, mass 0; visual mesh filename=package://alex_V1_description/meshes/ZEDXMini.obj
Joints:
- added joint TORSO_ZED_X_MINI_JOINT: type fixed, parent TORSO_LINK, child TORSO_ZED_X_MINI_LINK, origin xyz=0.1 0.0 0.05 rpy=0.0 0.907571 0.0
