Commit message: started updating all the different model parameters

File: alex-models/alex_V1_description/rl_urdf/alex_v1.rlModel_fullBody_robotAccurate_fullCollisions.urdf (robot description, URDF)
Before this commit: robot Alex, 45 links, 44 joints
Joints:
- joint LEFT_ANKLE_X: limit lower=-0.436332 upper=0.436332 effort=90 velocity=8 -> lower=-0.436332 upper=0.436332 effort=145.2 velocity=9.75
- joint LEFT_ANKLE_Y: limit lower=-1.0472 upper=0.523599 effort=180 velocity=8 -> lower=-1.0472 upper=0.523599 effort=193.6 velocity=9.72
- joint LEFT_ELBOW_Y: limit lower=-2.35619 upper=0.174532925 effort=80.0 velocity=11.5 -> lower=-2.35619 upper=0.174532925 effort=67.72 velocity=5.29
- joint LEFT_GRIPPER_Z: limit lower=-2.61799 upper=2.61799 effort=20.0 velocity=25.0 -> lower=-2.61799 upper=2.61799 effort=25.0 velocity=17.3
- joint LEFT_HIP_X: limit lower=-0.3490658504 upper=0.872664626 effort=150 velocity=9 -> lower=-0.3490658504 upper=0.872664626 effort=160.7 velocity=10.38
- joint LEFT_HIP_Y: limit lower=-2.61799 upper=0.785398 effort=200 velocity=8 -> lower=-2.61799 upper=0.785398 effort=217.2 velocity=9.3
- joint LEFT_HIP_Z: limit lower=-0.3490658504 upper=1.0472 effort=60 velocity=11 -> lower=-0.3490658504 upper=1.0472 effort=70.5 velocity=10.59
- joint LEFT_KNEE_Y: limit lower=0 upper=2.445206282 effort=200 velocity=8 -> lower=0 upper=2.445206282 effort=217.2 velocity=9.3
- joint LEFT_SHOULDER_X: limit lower=-0.349066 upper=2.79253 effort=150.0 velocity=9.0 -> lower=-0.349066 upper=2.79253 effort=160.7 velocity=10.38
- joint LEFT_SHOULDER_Y: limit lower=-3.141592 upper=1.22173 effort=150.0 velocity=9.0 -> lower=-3.141592 upper=1.22173 effort=160.7 velocity=10.38
- joint LEFT_SHOULDER_Z: limit lower=-1.91986 upper=1.22173 effort=80.0 velocity=11.5 -> lower=-1.91986 upper=1.22173 effort=67.72 velocity=5.29
- joint LEFT_WRIST_X: limit lower=-1.8326 upper=0.610865 effort=20.0 velocity=25.0 -> lower=-1.8326 upper=0.610865 effort=25.0 velocity=17.3
- joint LEFT_WRIST_Z: limit lower=-2.61799 upper=2.61799 effort=20.0 velocity=25.0 -> lower=-2.61799 upper=2.61799 effort=25.0 velocity=17.3
- joint NECK_Y: limit lower=-1.0472 upper=1.0472 effort=20 velocity=20 -> lower=-1.0472 upper=1.0472 effort=25.0 velocity=17.3
- joint NECK_Z: limit lower=-1.5708 upper=1.5708 effort=20 velocity=20 -> lower=-1.5708 upper=1.5708 effort=25.0 velocity=17.3
- joint RIGHT_ANKLE_X: limit lower=-0.436332 upper=0.436332 effort=90 velocity=8 -> lower=-0.436332 upper=0.436332 effort=145.2 velocity=9.72
- joint RIGHT_ANKLE_Y: limit lower=-1.0472 upper=0.523599 effort=180 velocity=8 -> lower=-1.0472 upper=0.523599 effort=193.6 velocity=9.72
- joint RIGHT_ELBOW_Y: limit lower=-2.35619 upper=0.174532925 effort=1000 velocity=100 -> lower=-2.35619 upper=0.174532925 effort=67.72 velocity=5.29
- joint RIGHT_GRIPPER_Z: limit lower=-2.61799 upper=2.61799 effort=20.0 velocity=25.0 -> lower=-2.61799 upper=2.61799 effort=25.0 velocity=17.3
- joint RIGHT_HIP_X: limit lower=-0.872664626 upper=0.3490658504 effort=150 velocity=9 -> lower=-0.3490658504 upper=0.872664626 effort=160.7 velocity=10.38
- joint RIGHT_HIP_Y: limit lower=-2.61799 upper=0.785398 effort=200 velocity=8 -> lower=-2.61799 upper=0.785398 effort=217.2 velocity=9.3
- joint RIGHT_HIP_Z: limit lower=-1.0472 upper=0.3490658504 effort=60 velocity=11 -> lower=-0.3490658504 upper=1.0472 effort=70.5 velocity=10.59
- joint RIGHT_KNEE_Y: limit lower=0 upper=2.445206282 effort=200 velocity=8 -> lower=0 upper=2.445206282 effort=217.2 velocity=9.3
- joint RIGHT_SHOULDER_X: limit lower=-2.79253 upper=0.349066 effort=1000 velocity=100 -> lower=-2.79253 upper=0.349066 effort=160.7 velocity=10.38
- joint RIGHT_SHOULDER_Y: limit lower=-3.141592 upper=1.22173 effort=1000 velocity=100 -> lower=-3.141592 upper=1.22173 effort=160.7 velocity=10.38
- joint RIGHT_SHOULDER_Z: limit lower=-1.22173 upper=1.91986 effort=1000 velocity=100 -> lower=-1.22173 upper=1.91986 effort=67.7 velocity=5.29
- joint RIGHT_WRIST_X: limit lower=-0.610865 upper=1.8326 effort=20.0 velocity=25.0 -> lower=-0.610865 upper=1.8326 effort=25.0 velocity=17.3
- joint RIGHT_WRIST_Z: limit lower=-2.61799 upper=2.61799 effort=20.0 velocity=25.0 -> lower=-2.61799 upper=2.61799 effort=25.0 velocity=17.3
- joint SPINE_Z: limit lower=-0.5235987756 upper=0.5235987756 effort=150 velocity=9.0 -> lower=-0.5235987756 upper=0.5235987756 effort=179 velocity=9.2

File: alex-models/alex_V1_description/rl_urdf/alex_v1.rlModel_fullBody_robotAccurate_torsoFootCollisions.urdf (robot description, URDF)
Before this commit: robot Alex, 45 links, 44 joints
Joints:
- joint LEFT_HIP_X: limit lower=-0.3490658504 upper=0.872664626 effort=150 velocity=9 -> lower=-0.3490658504 upper=0.872664626 effort=160.7 velocity=10.38
- joint LEFT_HIP_Y: limit lower=-2.61799 upper=0.785398 effort=200 velocity=8 -> lower=-2.61799 upper=0.785398 effort=217.2 velocity=9.3
- joint LEFT_HIP_Z: limit lower=-0.3490658504 upper=1.0472 effort=60 velocity=11 -> lower=-0.3490658504 upper=1.0472 effort=70.5 velocity=10.59

File: alex-models/alex_V1_description/urdf/alex_v1.lowerBody.urdf (robot description, URDF)
Before this commit: robot Alex, 22 links, 21 joints
Joints:
- joint LEFT_ANKLE_X: limit lower=-0.436332 upper=0.436332 effort=90 velocity=8 -> lower=-0.436332 upper=0.436332 effort=145.2 velocity=9.72
- joint LEFT_ANKLE_Y: limit lower=-1.0472 upper=0.523599 effort=180 velocity=8 -> lower=-1.0472 upper=0.523599 effort=193.6 velocity=9.72
- joint LEFT_HIP_X: limit lower=-0.3490658504 upper=0.872664626 effort=150 velocity=9 -> lower=-0.3490658504 upper=0.872664626 effort=160.7 velocity=10.38
- joint LEFT_HIP_Y: limit lower=-2.61799 upper=0.785398 effort=200 velocity=8 -> lower=-2.61799 upper=0.785398 effort=217.2 velocity=9.3
- joint LEFT_HIP_Z: limit lower=-0.3490658504 upper=1.0472 effort=60 velocity=11 -> lower=-0.3490658504 upper=1.0472 effort=70.5 velocity=10.59
- joint LEFT_KNEE_Y: limit lower=0 upper=2.445206282 effort=200 velocity=8 -> lower=0 upper=2.445206282 effort=217.2 velocity=9.3
- joint RIGHT_ANKLE_X: limit lower=-0.436332 upper=0.436332 effort=90 velocity=8 -> lower=-0.436332 upper=0.436332 effort=145.2 velocity=9.72
- joint RIGHT_ANKLE_Y: limit lower=-1.0472 upper=0.523599 effort=180 velocity=8 -> lower=-1.0472 upper=0.523599 effort=193.6 velocity=9.72
- joint RIGHT_HIP_X: limit lower=-0.872664626 upper=0.3490658504 effort=150 velocity=9 -> lower=-0.3490658504 upper=0.872664626 effort=160.7 velocity=10.38
- joint RIGHT_HIP_Y: limit lower=-2.61799 upper=0.785398 effort=200 velocity=8 -> lower=-2.61799 upper=0.785398 effort=217.2 velocity=9.3
- joint RIGHT_HIP_Z: limit lower=-1.0472 upper=0.3490658504 effort=60 velocity=11 -> lower=-0.3490658504 upper=1.0472 effort=70.5 velocity=10.59
- joint RIGHT_KNEE_Y: limit lower=0 upper=2.445206282 effort=200 velocity=8 -> lower=0 upper=2.445206282 effort=217.2 velocity=9.3
- joint SPINE_Z: limit lower=-0.5235987756 upper=0.5235987756 effort=150 velocity=9.0 -> lower=-0.5235987756 upper=0.5235987756 effort=160.7 velocity=10.38

Commit message: finished fixing all the models

File: alex-models/alex_V1_description/rl_urdf/alex_v1.rlModel_fullBody_robotAccurate_fullCollisions.urdf (robot description, URDF)
Before this commit: robot Alex, 45 links, 44 joints
Links:
- removed link LEFT_FOOT_IMU_LINK
- removed link PELVIS_STIM_IMU_LINK
- removed link RIGHT_FOOT_IMU_LINK
- added link LEFT_GRIPPER_Z_IMU_LINK, mass 0
- added link LEFT_WRIST_Z_IMU_LINK, mass 0
- added link PELVIS_IMU_LINK, mass 0.0
- added link RIGHT_GRIPPER_Z_IMU_LINK, mass 0
- added link RIGHT_WRIST_Z_IMU_LINK, mass 0
- link LEFT_GRIPPER_Z_LINK: mass 0.251 -> 0.144
- link RIGHT_GRIPPER_Z_LINK: mass 0.251 -> 0.144
Joints:
- removed joint LEFT_FOOT_IMU_JOINT
- removed joint PELVIS_STIM_IMU_JOINT
- removed joint RIGHT_FOOT_IMU_JOINT
- added joint LEFT_GRIPPER_Z_IMU_JOINT: type fixed, parent LEFT_GRIPPER_Z_LINK, child LEFT_GRIPPER_Z_IMU_LINK, origin xyz=0 0 0 rpy=0 0 0, axis 0 0 1
- added joint LEFT_WRIST_Z_IMU_JOINT: type fixed, parent LEFT_WRIST_Z_LINK, child LEFT_WRIST_Z_IMU_LINK, origin xyz=-0.033554 0.010450 -0.148527 rpy=1.571 0.0 1.571, axis 0 0 1
- added joint PELVIS_IMU_JOINT: type fixed, parent PELVIS_LINK, child PELVIS_IMU_LINK, origin xyz=-0.08687724 0.01225028 -0.08051472 rpy=-0.01399 -0.013054 1.570796
- added joint RIGHT_GRIPPER_Z_IMU_JOINT: type fixed, parent RIGHT_GRIPPER_Z_LINK, child RIGHT_GRIPPER_Z_IMU_LINK, origin xyz=0 0 0 rpy=0 0 0, axis 0 0 1
- added joint RIGHT_WRIST_Z_IMU_JOINT: type fixed, parent RIGHT_WRIST_Z_LINK, child RIGHT_WRIST_Z_IMU_LINK, origin xyz=-0.033554 0.010450 -0.148527 rpy=1.571  0.0 1.571, axis 0 0 1
- joint LEFT_ELBOW_Y: limit lower=-2.35619 upper=0.174532925 effort=71.28 velocity=4.47 -> lower=-2.35619 upper=0.174533 effort=71.28 velocity=4.47
- joint LEFT_HIP_X: limit lower=-0.3490658504 upper=0.872664626 effort=160.7 velocity=10.38 -> lower=-0.349066 upper=0.872664626 effort=160.7 velocity=10.38
- joint LEFT_HIP_Z: limit lower=-0.3490658504 upper=1.0472 effort=70.5 velocity=10.59 -> lower=-0.349066 upper=1.0472 effort=70.5 velocity=10.59
- joint LEFT_KNEE_Y: limit lower=0 upper=2.445206282 effort=217.2 velocity=9.3 -> lower=0 upper=2.44346 effort=217.2 velocity=9.3
- joint NECK_Y: limit lower=-0.49 upper=0.49 effort=20.86 velocity=17.3 -> lower=-0.488692 upper=0.488692 effort=20.86 velocity=17.3
- joint RIGHT_HIP_X: limit lower=-0.3490658504 upper=0.872664626 effort=160.7 velocity=10.38 -> lower=-1.0472 upper=0.349066 effort=70.5 velocity=10.59
- joint RIGHT_HIP_Z: limit lower=-0.3490658504 upper=1.0472 effort=70.5 velocity=10.59 -> lower=-2.61799 upper=0.785398 effort=217.2 velocity=9.3
- joint RIGHT_KNEE_Y: limit lower=0 upper=2.445206282 effort=217.2 velocity=9.3 -> lower=0 upper=2.44346 effort=217.2 velocity=9.3
- joint SPINE_Z: limit lower=-0.5235987756 upper=0.5235987756 effort=160.7 velocity=10.38 -> lower=-0.523599 upper=0.523599 effort=160.7 velocity=10.38

File: alex-models/alex_V1_description/rl_urdf/alex_v1.rlModel_fullBody_robotAccurate_torsoFootCollisions.urdf (robot description, URDF)
Before this commit: robot Alex, 45 links, 44 joints
Links:
- removed link LEFT_FOOT_IMU_LINK
- removed link PELVIS_STIM_IMU_LINK
- removed link RIGHT_FOOT_IMU_LINK
- added link LEFT_GRIPPER_Z_IMU_LINK, mass 0
- added link LEFT_WRIST_Z_IMU_LINK, mass 0
- added link PELVIS_IMU_LINK, mass 0.0
- added link RIGHT_GRIPPER_Z_IMU_LINK, mass 0
- added link RIGHT_WRIST_Z_IMU_LINK, mass 0
- link LEFT_GRIPPER_Z_LINK: mass 0.251 -> 0.144
- link RIGHT_GRIPPER_Z_LINK: mass 0.251 -> 0.144
Joints:
- removed joint LEFT_FOOT_IMU_JOINT
- removed joint PELVIS_STIM_IMU_JOINT
- removed joint RIGHT_FOOT_IMU_JOINT
- added joint LEFT_GRIPPER_Z_IMU_JOINT: type fixed, parent LEFT_GRIPPER_Z_LINK, child LEFT_GRIPPER_Z_IMU_LINK, origin xyz=0 0 0 rpy=0 0 0, axis 0 0 1
- added joint LEFT_WRIST_Z_IMU_JOINT: type fixed, parent LEFT_WRIST_Z_LINK, child LEFT_WRIST_Z_IMU_LINK, origin xyz=-0.033554 0.010450 -0.148527 rpy=1.571 0.0 1.571, axis 0 0 1
- added joint PELVIS_IMU_JOINT: type fixed, parent PELVIS_LINK, child PELVIS_IMU_LINK, origin xyz=-0.08687724 0.01225028 -0.08051472 rpy=-0.01399 -0.013054 1.570796
- added joint RIGHT_GRIPPER_Z_IMU_JOINT: type fixed, parent RIGHT_GRIPPER_Z_LINK, child RIGHT_GRIPPER_Z_IMU_LINK, origin xyz=0 0 0 rpy=0 0 0, axis 0 0 1
- added joint RIGHT_WRIST_Z_IMU_JOINT: type fixed, parent RIGHT_WRIST_Z_LINK, child RIGHT_WRIST_Z_IMU_LINK, origin xyz=-0.033554 0.010450 -0.148527 rpy=1.571  0.0 1.571, axis 0 0 1
- joint LEFT_ELBOW_Y: limit lower=-2.35619 upper=0.174532925 effort=71.28 velocity=4.47 -> lower=-2.35619 upper=0.174533 effort=71.28 velocity=4.47
- joint LEFT_HIP_X: limit lower=-0.3490658504 upper=0.872664626 effort=160.7 velocity=10.38 -> lower=-0.349066 upper=0.872664626 effort=160.7 velocity=10.38
- joint LEFT_HIP_Z: limit lower=-0.3490658504 upper=1.0472 effort=70.5 velocity=10.59 -> lower=-0.349066 upper=1.0472 effort=70.5 velocity=10.59
- joint LEFT_KNEE_Y: limit lower=0 upper=2.445206282 effort=217.2 velocity=9.3 -> lower=0 upper=2.44346 effort=217.2 velocity=9.3
- joint NECK_Y: limit lower=-0.49 upper=0.49 effort=20.86 velocity=17.3 -> lower=-0.488692 upper=0.488692 effort=20.86 velocity=17.3
- joint RIGHT_HIP_X: limit lower=-0.3490658504 upper=0.872664626 effort=160.7 velocity=10.38 -> lower=-1.0472 upper=0.349066 effort=70.5 velocity=10.59
- joint RIGHT_HIP_Z: limit lower=-0.3490658504 upper=1.0472 effort=70.5 velocity=10.59 -> lower=-2.61799 upper=0.785398 effort=217.2 velocity=9.3
- joint RIGHT_KNEE_Y: limit lower=0 upper=2.445206282 effort=217.2 velocity=9.3 -> lower=0 upper=2.44346 effort=217.2 velocity=9.3
- joint SPINE_Z: limit lower=-0.5235987756 upper=0.5235987756 effort=160.7 velocity=10.38 -> lower=-0.523599 upper=0.523599 effort=160.7 velocity=10.38

File: alex-models/alex_V1_description/rl_urdf/alex_v1.rlModel_nubForearms_robotAccurate_fullCollisions.urdf (robot description, URDF)
Before this commit: robot Alex, 39 links, 38 joints
Links:
- removed link LEFT_FOOT_IMU_LINK
- removed link PELVIS_STIM_IMU_LINK
- removed link RIGHT_FOOT_IMU_LINK
- added link PELVIS_IMU_LINK, mass 0.0
- link LEFT_ELBOW_Y_LINK: mass 0.69372585 -> 0.616
- link RIGHT_ELBOW_Y_LINK: mass 0.69372166  -> 0.616
- link TORSO_LINK: mass 10.878322779 -> 11.478322779
Joints:
- removed joint LEFT_FOOT_IMU_JOINT
- removed joint PELVIS_STIM_IMU_JOINT
- removed joint RIGHT_FOOT_IMU_JOINT
- added joint PELVIS_IMU_JOINT: type fixed, parent PELVIS_LINK, child PELVIS_IMU_LINK, origin xyz=-0.08687724 0.01225028 -0.08051472 rpy=-0.01399 -0.013054 1.570796
- joint LEFT_ELBOW_Y: limit lower=-2.35619 upper=0.174532925 effort=71.28 velocity=4.47 -> lower=-2.35619 upper=0.174533 effort=71.28 velocity=4.47
- joint LEFT_HIP_X: limit lower=-0.3490658504 upper=0.872664626 effort=160.7 velocity=10.38 -> lower=-0.349066 upper=0.872664626 effort=160.7 velocity=10.38
- joint LEFT_HIP_Z: limit lower=-0.3490658504 upper=1.0472 effort=70.5 velocity=10.59 -> lower=-0.349066 upper=1.0472 effort=70.5 velocity=10.59
- joint LEFT_KNEE_Y: limit lower=0 upper=2.445206282 effort=217.2 velocity=9.3 -> lower=0 upper=2.44346 effort=217.2 velocity=9.3
- joint NECK_Y: limit lower=-0.49 upper=0.49 effort=20.86 velocity=17.3 -> lower=-0.488692 upper=0.488692 effort=20.86 velocity=17.3
- joint RIGHT_HIP_X: limit lower=-0.3490658504 upper=0.872664626 effort=160.7 velocity=10.38 -> lower=-1.0472 upper=0.349066 effort=70.5 velocity=10.59
- joint RIGHT_HIP_Z: limit lower=-0.3490658504 upper=1.0472 effort=70.5 velocity=10.59 -> lower=-2.61799 upper=0.785398 effort=217.2 velocity=9.3
- joint SPINE_Z: limit lower=-0.5235987756 upper=0.5235987756 effort=160.7 velocity=10.38 -> lower=-0.523599 upper=0.523599 effort=160.7 velocity=10.38

File: alex-models/alex_V1_description/rl_urdf/alex_v1.rlModel_nubForearms_robotAccurate_fullCollisions_hanging.urdf (robot description, URDF)
Before this commit: robot Alex, 44 links, 43 joints
Links:
- removed link LEFT_FOOT_IMU_LINK
- removed link PELVIS_STIM_IMU_LINK
- removed link RIGHT_FOOT_IMU_LINK
- added link PELVIS_IMU_LINK, mass 0.0
- link LEFT_ELBOW_Y_LINK: mass 0.69372585 -> 0.616
- link RIGHT_ELBOW_Y_LINK: mass 0.69372166  -> 0.616
- link TORSO_LINK: mass 10.878322779 -> 11.478322779
Joints:
- removed joint LEFT_FOOT_IMU_JOINT
- removed joint PELVIS_STIM_IMU_JOINT
- removed joint RIGHT_FOOT_IMU_JOINT
- added joint PELVIS_IMU_JOINT: type fixed, parent PELVIS_LINK, child PELVIS_IMU_LINK, origin xyz=-0.08687724 0.01225028 -0.08051472 rpy=-0.01399 -0.013054 1.570796
- joint LEFT_ELBOW_Y: limit lower=-2.35619 upper=0.174532925 effort=71.28 velocity=4.47 -> lower=-2.35619 upper=0.174533 effort=71.28 velocity=4.47
- joint LEFT_HIP_X: limit lower=-0.3490658504 upper=0.872664626 effort=160.7 velocity=10.38 -> lower=-0.488692 upper=0.872665 effort=160.7 velocity=10.38
- joint LEFT_HIP_Z: limit lower=-0.3490658504 upper=1.0472 effort=70.5 velocity=10.59 -> lower=-0.349066 upper=1.0472 effort=70.5 velocity=10.59
- joint LEFT_KNEE_Y: limit lower=0 upper=2.445206282 effort=217.2 velocity=9.3 -> lower=0 upper=2.44346 effort=217.2 velocity=9.3
- joint NECK_Y: limit lower=-0.49 upper=0.49 effort=20.86 velocity=17.3 -> lower=-0.488692 upper=0.488692 effort=20.86 velocity=17.3
- joint RIGHT_ELBOW_Y: limit lower=-2.35619 upper=0.174532925 effort=71.28 velocity=4.47 -> lower=-2.35619 upper=0.174533 effort=71.28 velocity=4.47
- joint RIGHT_HIP_X: limit lower=-0.3490658504 upper=0.872664626 effort=160.7 velocity=10.38 -> lower=-0.872665 upper=0.488692 effort=160.7 velocity=10.38
- joint RIGHT_HIP_Z: limit lower=-0.3490658504 upper=1.0472 effort=70.5 velocity=10.59 -> lower=-1.0472 upper=0.349066 effort=70.5 velocity=10.59
- joint RIGHT_KNEE_Y: limit lower=0 upper=2.445206282 effort=217.2 velocity=9.3 -> lower=0 upper=2.44346 effort=217.2 velocity=9.3
- joint SPINE_Z: limit lower=-0.5235987756 upper=0.5235987756 effort=160.7 velocity=10.38 -> lower=-0.523599 upper=0.523599 effort=160.7 velocity=10.38

File: alex-models/alex_V1_description/rl_urdf/alex_v1.rlModel_nubForearms_robotAccurate_torsoFootCollisions.urdf (robot description, URDF)
Before this commit: robot Alex, 39 links, 38 joints
Links:
- removed link LEFT_FOOT_IMU_LINK
- removed link PELVIS_STIM_IMU_LINK
- removed link RIGHT_FOOT_IMU_LINK
- added link PELVIS_IMU_LINK, mass 0.0
- link LEFT_ELBOW_Y_LINK: mass 0.69372585 -> 0.616
- link RIGHT_ELBOW_Y_LINK: mass 0.69372166  -> 0.616
- link TORSO_LINK: mass 10.878322779 -> 11.478322779
Joints:
- removed joint LEFT_FOOT_IMU_JOINT
- removed joint PELVIS_STIM_IMU_JOINT
- removed joint RIGHT_FOOT_IMU_JOINT
- added joint PELVIS_IMU_JOINT: type fixed, parent PELVIS_LINK, child PELVIS_IMU_LINK, origin xyz=-0.08687724 0.01225028 -0.08051472 rpy=-0.01399 -0.013054 1.570796
- joint LEFT_ELBOW_Y: limit lower=-2.35619 upper=0.174532925 effort=67.72 velocity=5.29 -> lower=-2.35619 upper=0.174533 effort=71.28 velocity=4.47
- joint LEFT_HIP_X: limit lower=-0.3490658504 upper=0.872664626 effort=160.7 velocity=10.38 -> lower=-0.349066 upper=0.872664626 effort=160.7 velocity=10.38
- joint LEFT_HIP_Z: limit lower=-0.3490658504 upper=1.0472 effort=70.5 velocity=10.59 -> lower=-0.349066 upper=1.0472 effort=70.5 velocity=10.59
- joint LEFT_KNEE_Y: limit lower=0 upper=2.445206282 effort=217.2 velocity=9.3 -> lower=0 upper=2.44346 effort=217.2 velocity=9.3
- joint LEFT_SHOULDER_Z: limit lower=-1.91986 upper=1.22173 effort=67.72 velocity=5.29 -> lower=-1.91986 upper=1.22173 effort=71.28 velocity=4.47
- joint NECK_Y: limit lower=-1.0472 upper=1.0472 effort=20.86 velocity=17.3 -> lower=-0.488692 upper=0.488692 effort=20.86 velocity=17.3
- joint RIGHT_ELBOW_Y: limit lower=-2.35619 upper=0.174532925 effort=67.72 velocity=5.29 -> lower=-2.35619 upper=0.174532925 effort=71.28 velocity=4.47
- joint RIGHT_HIP_X: limit lower=-0.3490658504 upper=0.872664626 effort=160.7 velocity=10.38 -> lower=-1.0472 upper=0.349066 effort=70.5 velocity=10.59
- joint RIGHT_HIP_Z: limit lower=-0.3490658504 upper=1.0472 effort=70.5 velocity=10.59 -> lower=-2.61799 upper=0.785398 effort=217.2 velocity=9.3
- joint RIGHT_SHOULDER_Z: limit lower=-1.22173 upper=1.91986 effort=67.72 velocity=5.29 -> lower=-1.22173 upper=1.91986 effort=71.28 velocity=4.47
- joint SPINE_Z: limit lower=-0.5235987756 upper=0.5235987756 effort=160.7 velocity=10.38 -> lower=-0.523599 upper=0.523599 effort=160.7 velocity=10.38

File: alex-models/alex_V1_description/rl_urdf/alex_v1.rlModel_nubForearms_robotAccurate_torsoFootCollisions_hanging.urdf (robot description, URDF)
Before this commit: robot Alex, 45 links, 44 joints
Links:
- removed link LEFT_FOOT_IMU_LINK
- removed link PELVIS_STIM_IMU_LINK
- removed link RIGHT_FOOT_IMU_LINK
- added link PELVIS_IMU_LINK, mass 0.0
- link LEFT_ELBOW_Y_LINK: mass 0.69372585 -> 0.616
- link RIGHT_ELBOW_Y_LINK: mass 0.69372166  -> 0.616
- link TORSO_LINK: mass 10.878322779 -> 11.478322779
Joints:
- removed joint LEFT_FOOT_IMU_JOINT
- removed joint PELVIS_STIM_IMU_JOINT
- removed joint RIGHT_FOOT_IMU_JOINT
- added joint PELVIS_IMU_JOINT: type fixed, parent PELVIS_LINK, child PELVIS_IMU_LINK, origin xyz=-0.08687724 0.01225028 -0.08051472 rpy=-0.01399 -0.013054 1.570796
- joint LEFT_HIP_X: limit lower=-0.3490658504 upper=0.872664626 effort=160.7 velocity=10.38 -> lower=-0.488692 upper=0.872665 effort=160.7 velocity=10.38
- joint LEFT_HIP_Z: limit lower=-0.3490658504 upper=1.0472 effort=70.5 velocity=10.59 -> lower=-0.349066 upper=1.0472 effort=70.5 velocity=10.59
- joint LEFT_KNEE_Y: limit lower=0 upper=2.445206282 effort=217.2 velocity=9.3 -> lower=0 upper=2.44346 effort=217.2 velocity=9.3
- joint NECK_Y: limit lower=-1.0472 upper=1.0472 effort=20.86 velocity=17.3 -> lower=-0.488692 upper=0.488692 effort=20.86 velocity=17.3
- joint RIGHT_ELBOW_Y: limit lower=-2.35619 upper=0.174532925 effort=67.72 velocity=5.29 -> lower=-2.35619 upper=0.174533 effort=71.28 velocity=4.47
- joint RIGHT_HIP_X: limit lower=-0.3490658504 upper=0.872664626 effort=160.7 velocity=10.38 -> lower=-0.872665 upper=0.488692 effort=160.7 velocity=10.38
- joint RIGHT_HIP_Z: limit lower=-0.3490658504 upper=1.0472 effort=70.5 velocity=10.59 -> lower=-1.0472 upper=0.349066 effort=70.5 velocity=10.59
- joint RIGHT_KNEE_Y: limit lower=0 upper=2.445206282 effort=217.2 velocity=9.3 -> lower=0 upper=2.44346 effort=217.2 velocity=9.3
- joint RIGHT_SHOULDER_Z: limit lower=-1.22173 upper=1.91986 effort=67.72 velocity=5.29 -> lower=-1.22173 upper=1.91986 effort=71.28 velocity=4.47
- joint SPINE_Z: limit lower=-0.5235987756 upper=0.5235987756 effort=160.7 velocity=10.38 -> lower=-0.523599 upper=0.523599 effort=160.7 velocity=10.38

File: alex-models/alex_V1_description/urdf/alex_v1.fullBody.urdf (robot description, URDF)
Before this commit: robot Alex, 48 links, 47 joints
Links:
- added link RIGHT_SHOULDER_Z_IMU_LINK, mass 0
Joints:
- added joint RIGHT_SHOULDER_Z_IMU_JOINT: type fixed, parent RIGHT_SHOULDER_Z_LINK, child RIGHT_SHOULDER_Z_IMU_LINK, origin xyz=0.002 0.016 -0.318 rpy=1.570796 0 0.314159, axis 0 0 1

File: alex-models/alex_V1_description/urdf/alex_v1.fullBodyNubForearms.urdf (robot description, URDF)
Before this commit: robot Alex, 37 links, 36 joints
Joints:
- joint RIGHT_ELBOW_Y: limit lower=-2.35619 upper=0.174532925 effort=1000 velocity=100 -> lower=-2.35619 upper=0.174532925 effort=71.28 velocity=100
