Commit message: fixed copy paste errors

File: alex-models/alex_V1_description/rl_urdf/alex_v1.rlModel_fullBody_robotAccurate_fullCollisions.urdf (robot description, URDF)
Before this commit: robot Alex, 47 links, 46 joints
Joints:
- joint RIGHT_HIP_X: limit lower=-1.0472 upper=0.349066 effort=70.5 velocity=10.59 -> lower=-0.872665 upper=0.488692 effort=160.7 velocity=10.38
- joint RIGHT_HIP_Z: limit lower=-2.61799 upper=0.785398 effort=217.2 velocity=9.3 -> lower=-1.0472 upper=0.349066 effort=70.5 velocity=10.59

File: alex-models/alex_V1_description/rl_urdf/alex_v1.rlModel_fullBody_robotAccurate_torsoFootCollisions.urdf (robot description, URDF)
Before this commit: robot Alex, 47 links, 46 joints
Joints:
- joint RIGHT_HIP_X: limit lower=-1.0472 upper=0.349066 effort=70.5 velocity=10.59 -> lower=-0.872665 upper=0.488692 effort=160.7 velocity=10.38
- joint RIGHT_HIP_Z: limit lower=-2.61799 upper=0.785398 effort=217.2 velocity=9.3 -> lower=-1.0472 upper=0.349066 effort=70.5 velocity=10.59

File: alex-models/alex_V1_description/rl_urdf/alex_v1.rlModel_nubForearms_robotAccurate_fullCollisions.urdf (robot description, URDF)
Before this commit: robot Alex, 37 links, 36 joints
Joints:
- joint RIGHT_HIP_X: limit lower=-1.0472 upper=0.349066 effort=70.5 velocity=10.59 -> lower=-0.872665 upper=0.488692 effort=160.7 velocity=10.38
- joint RIGHT_HIP_Z: limit lower=-2.61799 upper=0.785398 effort=217.2 velocity=9.3 -> lower=-1.0472 upper=0.349066 effort=70.5 velocity=10.59

File: alex-models/alex_V1_description/rl_urdf/alex_v1.rlModel_nubForearms_robotAccurate_torsoFootCollisions.urdf (robot description, URDF)
Before this commit: robot Alex, 37 links, 36 joints
Joints:
- joint RIGHT_HIP_X: limit lower=-1.0472 upper=0.349066 effort=70.5 velocity=10.59 -> lower=-0.872665 upper=0.488692 effort=160.7 velocity=10.38
- joint RIGHT_HIP_Z: limit lower=-2.61799 upper=0.785398 effort=217.2 velocity=9.3 -> lower=-1.0472 upper=0.349066 effort=70.5 velocity=10.59

Commit message: fixed the last few little errors

File: alex-models/alex_V1_description/rl_urdf/alex_v1.rlModel_fullBody_robotAccurate_fullCollisions.urdf (robot description, URDF)
Before this commit: robot Alex, 47 links, 46 joints
Joints:
- joint LEFT_HIP_X: limit lower=-0.349066 upper=0.872664626 effort=160.7 velocity=10.38 -> lower=-0.488692 upper=0.872665 effort=160.7 velocity=10.38

File: alex-models/alex_V1_description/rl_urdf/alex_v1.rlModel_fullBody_robotAccurate_torsoFootCollisions.urdf (robot description, URDF)
Before this commit: robot Alex, 47 links, 46 joints
Joints:
- joint LEFT_HIP_X: limit lower=-0.349066 upper=0.872664626 effort=160.7 velocity=10.38 -> lower=-0.488692 upper=0.872665 effort=160.7 velocity=10.38

File: alex-models/alex_V1_description/rl_urdf/alex_v1.rlModel_nubForearms_robotAccurate_fullCollisions.urdf (robot description, URDF)
Before this commit: robot Alex, 37 links, 36 joints
Joints:
- joint LEFT_HIP_X: limit lower=-0.349066 upper=0.872664626 effort=160.7 velocity=10.38 -> lower=-0.488692 upper=0.872665 effort=160.7 velocity=10.38

File: alex-models/alex_V1_description/rl_urdf/alex_v1.rlModel_nubForearms_robotAccurate_torsoFootCollisions.urdf (robot description, URDF)
Before this commit: robot Alex, 37 links, 36 joints
Joints:
- joint LEFT_HIP_X: limit lower=-0.349066 upper=0.872664626 effort=160.7 velocity=10.38 -> lower=-0.488692 upper=0.872665 effort=160.7 velocity=10.38

File: alex-models/alex_V1_description/rl_urdf/alex_v1.rlModel_nubForearms_robotAccurate_torsoFootCollisions_hanging.urdf (robot description, URDF)
Before this commit: robot Alex, 43 links, 42 joints
Joints:
- joint LEFT_ELBOW_Y: limit lower=-2.35619 upper=0.174532925 effort=67.72 velocity=5.29 -> lower=-2.35619 upper=0.174533 effort=71.28 velocity=4.47
- joint LEFT_SHOULDER_Z: limit lower=-1.91986 upper=1.22173 effort=67.72 velocity=5.29 -> lower=-1.91986 upper=1.22173 effort=71.28 velocity=4.47
