Commit message: Fix bad velocity limits on right arm for old urdf

File: alex-models/alex_V1_description/urdf/old/alex_v1.rightFixedForearm.urdf (robot description, URDF)
Before this commit: robot Alex, 1 links, 1 joints
Joints:
- joint RIGHT_ELBOW_Y: limit lower=-2.35619 upper=0.174532925 effort=1000 velocity=100 -> lower=-2.35619 upper=0.174532925 effort=80.0 velocity=11.5

File: alex-models/alex_V1_description/urdf/old/alex_v1.rightForearm.urdf (robot description, URDF)
Before this commit: robot Alex, 6 links, 6 joints
Joints:
- joint RIGHT_ELBOW_Y: limit lower=-2.35619 upper=0.174532925 effort=1000 velocity=100 -> lower=-2.35619 upper=0.174532925 effort=80.0 velocity=11.5

File: alex-models/alex_V1_description/urdf/old/alex_v1.rightUpperArm.urdf (robot description, URDF)
Before this commit: robot Alex, 5 links, 5 joints
Joints:
- joint RIGHT_SHOULDER_X: limit lower=-2.79253 upper=0.349066 effort=1000 velocity=100 -> lower=-2.79253 upper=0.349066 effort=150.0 velocity=9.0
- joint RIGHT_SHOULDER_Y: limit lower=-3.141592 upper=1.22173 effort=1000 velocity=100 -> lower=-3.141592 upper=1.22173 effort=150.0 velocity=9.0
- joint RIGHT_SHOULDER_Z: limit lower=-1.22173 upper=1.91986 effort=1000 velocity=100 -> lower=-1.22173 upper=1.91986 effort=80.0 velocity=11.5
