Commit message: Fixed collisions on v2 lower body and upper arm urdfs

File: alex-models/alex_V2_description/urdf/alex_v2.leftUpperArm.urdf (robot description, URDF)
Before this commit: robot Alex, 5 links, 5 joints
Links:
- link LEFT_SHOULDER_Z_LINK: geometry collision cylinder length=0.22 radius=0.05; visual mesh filename=package://alex_V1_description/meshes/cycloidal_arm/LeftShou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

File: alex-models/alex_V2_description/urdf/alex_v2.lowerBody.urdf (robot description, URDF)
Before this commit: robot Alex, 21 links, 20 joints
Links:
- link LEFT_SHIN: geometry collision cylinder length=0.3 radius=0.06; visual mesh filename=package://alex_V1_description/meshes/legs/LeftShin.obj
- link LEFT_THIGH: geometry collision box size=0.13 0.13 0.29; visual mesh filename=package://alex_V1_description/meshes/legs/LeftThigh.obj
- link RIGHT_SHIN: geometry collision cylinder length=0.3 radius=0.06; visual mesh filename=package://alex_V1_description/meshes/legs/RightShin.obj
- link RIGHT_THIGH: geometry collision box size=0.13 0.13 0.29; visual mesh filename=package://alex_V1_description/meshes/legs/RightThigh.obj

File: alex-models/alex_V2_description/urdf/alex_v2.rightUpperArm.urdf (robot description, URDF)
Before this commit: robot Alex, 5 links, 5 joints
Links:
- link RIGHT_SHOULDER_Z_LINK: geometry collision cylinder length=0.22 radius=0.05; visual mesh filename=package://alex_V1_description/meshes/cycloidal_arm/RightSho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

Commit message: Fixed some of the masses to match the changes from v1

File: alex-models/alex_V2_description/urdf/alex_v2.leftUpperArm.urdf (robot description, URDF)
Before this commit: robot Alex, 5 links, 5 joints
Links:
- link LEFT_SHOULDER_X_LINK: mass 0.972 -> 1.16160776 
- link LEFT_SHOULDER_Y_LINK: mass 2.99 -> 3.0331992
- link LEFT_SHOULDER_Z_LINK: mass 2.91 -> 3.134 
Joints:
- joint LEFT_SHOULDER_X: limit lower=-0.349066 upper=2.79253 effort=150.0 velocity=9.0 -> lower=-0.349066 upper=2.79253 effort=160.7 velocity=10.38
- joint LEFT_SHOULDER_Y: limit lower=-3.141592 upper=1.22173 effort=150.0 velocity=9.0 -> lower=-3.141592 upper=1.22173 effort=160.7 velocity=10.38
- joint LEFT_SHOULDER_Z: limit lower=-1.91986 upper=1.22173 effort=80.0 velocity=11.5 -> lower=-1.91986 upper=1.22173 effort=71.28 velocity=4.47

File: alex-models/alex_V2_description/urdf/alex_v2.lowerBody.urdf (robot description, URDF)
Before this commit: robot Alex, 21 links, 20 joints
Links:
- link LEFT_FOOT: mass 1.28288609 -> 1.28831268
- link LEFT_HIP_X_LINK: mass 2.32977961 -> 2.332078
- link LEFT_HIP_Z_LINK: mass 0.77281362 -> 0.74972192 
- link LEFT_SHIN: mass 6.31087157 -> 6.3405718 
- link LEFT_THIGH: mass 7.75 -> 8.286
- link PELVIS_LINK: mass 9.50083635 -> 7.161
- link RIGHT_FOOT: mass 1.28288609 -> 1.28831268
- link RIGHT_HIP_X_LINK: mass 2.32977248 -> 2.33123426 
- link RIGHT_HIP_Z_LINK: mass 0.77281055 -> 0.77280715
- link RIGHT_SHIN: mass 6.31087157 -> 6.33633928 
- link RIGHT_THIGH: mass 7.75 -> 8.27617423 
Joints:
- joint LEFT_ANKLE_X: limit lower=-0.436332 upper=0.436332 effort=90 velocity=8 -> lower=-0.436332 upper=0.436332 effort=145.2 velocity=9.72
- joint LEFT_ANKLE_Y: limit lower=-1.0472 upper=0.523599 effort=180 velocity=8 -> lower=-1.0472 upper=0.523599 effort=193.6 velocity=9.72
- joint LEFT_HIP_X: limit lower=-0.3490658504 upper=0.872664626 effort=150 velocity=9 -> lower=-0.488692 upper=0.872665 effort=160.7 velocity=10.38
- joint LEFT_HIP_Y: limit lower=-2.61799 upper=0.785398 effort=200 velocity=8 -> lower=-2.61799 upper=0.785398 effort=217.2 velocity=9.3
- joint LEFT_HIP_Z: limit lower=-0.3490658504 upper=1.0472 effort=60 velocity=11 -> lower=-0.349066 upper=1.0472 effort=70.5 velocity=10.59
- joint LEFT_KNEE_Y: limit lower=0 upper=2.445206282 effort=200 velocity=8 -> lower=0 upper=2.44346 effort=217.2 velocity=9.3
- joint RIGHT_ANKLE_X: limit lower=-0.436332 upper=0.436332 effort=90 velocity=8 -> lower=-0.436332 upper=0.436332 effort=145.2 velocity=9.72
- joint RIGHT_ANKLE_Y: limit lower=-1.0472 upper=0.523599 effort=180 velocity=8 -> lower=-1.0472 upper=0.523599 effort=193.6 velocity=9.72
- joint RIGHT_HIP_X: limit lower=-0.872664626 upper=0.3490658504 effort=150 velocity=9 -> lower=-0.872665 upper=0.488692 effort=160.7 velocity=10.38
- joint RIGHT_HIP_Y: limit lower=-2.61799 upper=0.785398 effort=200 velocity=8 -> lower=-2.61799 upper=0.785398 effort=217.2 velocity=9.3
- joint RIGHT_HIP_Z: limit lower=-1.0472 upper=0.3490658504 effort=60 velocity=11 -> lower=-1.0472 upper=0.349066 effort=70.5 velocity=10.59
- joint RIGHT_KNEE_Y: limit lower=0 upper=2.445206282 effort=200 velocity=8 -> lower=0 upper=2.44346 effort=217.2 velocity=9.3
- joint SPINE_Z: limit lower=-0.5235987756 upper=0.5235987756 effort=150 velocity=9.0 -> lower=-0.523599 upper=0.523599 effort=160.7 velocity=10.38

File: alex-models/alex_V2_description/urdf/alex_v2.rightUpperArm.urdf (robot description, URDF)
Before this commit: robot Alex, 5 links, 5 joints
Links:
- link RIGHT_SHOULDER_X_LINK: mass 0.972 -> 1.1615873 
- link RIGHT_SHOULDER_Y_LINK: mass 2.99 -> 3.00752318
- link RIGHT_SHOULDER_Z_LINK: mass 2.91 -> 3.10111287
Joints:
- joint RIGHT_SHOULDER_X: limit lower=-2.79253 upper=0.349066 effort=1000 velocity=100 -> lower=-2.79253 upper=0.349066 effort=160.7 velocity=10.38
- joint RIGHT_SHOULDER_Y: limit lower=-3.141592 upper=1.22173 effort=1000 velocity=100 -> lower=-3.141592 upper=1.22173 effort=160.7 velocity=10.38
- joint RIGHT_SHOULDER_Z: limit lower=-1.22173 upper=1.91986 effort=1000 velocity=100 -> lower=-1.22173 upper=1.91986 effort=71.28 velocity=4.47

Commit message: Added modified mass and inertia to v2

File: alex-models/alex_V2_description/urdf/alex_v2.leftUpperArm.urdf (robot description, URDF)
Before this commit: robot Alex, 5 links, 5 joints
Links:
- link LEFT_SHOULDER_X_LINK: mass 0.972 -> 1.16159753
- link LEFT_SHOULDER_Y_LINK: mass 2.99 -> 3.02036119
- link LEFT_SHOULDER_Z_LINK: mass 2.91 -> 3.117556435

File: alex-models/alex_V2_description/urdf/alex_v2.lowerBody.urdf (robot description, URDF)
Before this commit: robot Alex, 21 links, 20 joints
Links:
- link LEFT_FOOT: mass 1.28288609 -> 1.28831268
- link LEFT_HIP_X_LINK: mass 2.32977961 -> 2.33165613
- link LEFT_HIP_Z_LINK: mass 0.77281362 -> 0.761264535
- link LEFT_SHIN: mass 6.31087157 -> 6.33845554
- link LEFT_THIGH: mass 7.75 -> 8.281087115
- link PELVIS_LINK: mass 9.50083635 -> 7.161
- link RIGHT_FOOT: mass 1.28288609 -> 1.28831268
- link RIGHT_HIP_X_LINK: mass 2.32977248 -> 2.33165613
- link RIGHT_HIP_Z_LINK: mass 0.77281055 -> 0.761264535
- link RIGHT_SHIN: mass 6.31087157 -> 6.33845554
- link RIGHT_THIGH: mass 7.75 -> 8.281087115

File: alex-models/alex_V2_description/urdf/alex_v2.rightForearm.urdf (robot description, URDF)
Before this commit: robot Alex, 6 links, 6 joints
Links:
- link RIGHT_GRIPPER_Z_LINK: mass 0.144 -> 0.287

File: alex-models/alex_V2_description/urdf/alex_v2.rightUpperArm.urdf (robot description, URDF)
Before this commit: robot Alex, 5 links, 5 joints
Links:
- link RIGHT_SHOULDER_X_LINK: mass 0.972 -> 1.16159753
- link RIGHT_SHOULDER_Y_LINK: mass 2.99 -> 3.02036119
- link RIGHT_SHOULDER_Z_LINK: mass 2.91 -> 3.117556435

Commit message: Fixed limits on v2

File: alex-models/alex_V2_description/urdf/alex_v2.leftUpperArm.urdf (robot description, URDF)
Before this commit: robot Alex, 5 links, 5 joints
Joints:
- joint LEFT_SHOULDER_X: limit lower=-0.349066 upper=2.79253 effort=150.0 velocity=9.0 -> lower=-0.349066 upper=2.79253 effort=160.7 velocity=10.38
- joint LEFT_SHOULDER_Y: limit lower=-3.141592 upper=1.22173 effort=150.0 velocity=9.0 -> lower=-3.141592 upper=1.22173 effort=160.7 velocity=10.38
- joint LEFT_SHOULDER_Z: limit lower=-1.91986 upper=1.22173 effort=80.0 velocity=11.5 -> lower=-1.91986 upper=1.22173 effort=71.28 velocity=4.47

File: alex-models/alex_V2_description/urdf/alex_v2.lowerBody.urdf (robot description, URDF)
Before this commit: robot Alex, 21 links, 20 joints
Joints:
- joint LEFT_ANKLE_X: limit lower=-0.436332 upper=0.436332 effort=90 velocity=8 -> lower=-0.436332 upper=0.436332 effort=145.2 velocity=9.72
- joint LEFT_ANKLE_Y: limit lower=-1.0472 upper=0.523599 effort=180 velocity=8 -> lower=-1.0472 upper=0.523599 effort=193.6 velocity=9.72
- joint LEFT_HIP_X: limit lower=-0.3490658504 upper=0.872664626 effort=150 velocity=9 -> lower=-0.488692 upper=0.872665 effort=160.7 velocity=10.38
- joint LEFT_HIP_Y: limit lower=-2.61799 upper=0.785398 effort=200 velocity=8 -> lower=-2.61799 upper=0.785398 effort=217.2 velocity=9.3
- joint LEFT_HIP_Z: limit lower=-0.3490658504 upper=1.0472 effort=60 velocity=11 -> lower=-0.349066 upper=1.0472 effort=70.5 velocity=10.59
- joint LEFT_KNEE_Y: limit lower=0 upper=2.445206282 effort=200 velocity=8 -> lower=0 upper=2.44346 effort=217.2 velocity=9.3
- joint RIGHT_ANKLE_X: limit lower=-0.436332 upper=0.436332 effort=90 velocity=8 -> lower=-0.436332 upper=0.436332 effort=145.2 velocity=9.72
- joint RIGHT_ANKLE_Y: limit lower=-1.0472 upper=0.523599 effort=180 velocity=8 -> lower=-1.0472 upper=0.523599 effort=193.6 velocity=9.72
- joint RIGHT_HIP_X: limit lower=-0.872664626 upper=0.3490658504 effort=150 velocity=9 -> lower=-0.872665 upper=0.488692 effort=160.7 velocity=10.38
- joint RIGHT_HIP_Y: limit lower=-2.61799 upper=0.785398 effort=200 velocity=8 -> lower=-2.61799 upper=0.785398 effort=217.2 velocity=9.3
- joint RIGHT_HIP_Z: limit lower=-1.0472 upper=0.3490658504 effort=60 velocity=11 -> lower=-1.0472 upper=0.349066 effort=70.5 velocity=10.59
- joint RIGHT_KNEE_Y: limit lower=0 upper=2.445206282 effort=200 velocity=8 -> lower=0 upper=2.44346 effort=217.2 velocity=9.3
- joint SPINE_Z: limit lower=-0.5235987756 upper=0.5235987756 effort=150 velocity=9.0 -> lower=-0.523599 upper=0.523599 effort=160.7 velocity=10.38

File: alex-models/alex_V2_description/urdf/alex_v2.rightUpperArm.urdf (robot description, URDF)
Before this commit: robot Alex, 5 links, 5 joints
Joints:
- joint RIGHT_SHOULDER_X: limit lower=-2.79253 upper=0.349066 effort=1000 velocity=100 -> lower=-2.79253 upper=0.349066 effort=160.7 velocity=10.38
- joint RIGHT_SHOULDER_Y: limit lower=-3.141592 upper=1.22173 effort=1000 velocity=100 -> lower=-3.141592 upper=1.22173 effort=160.7 velocity=10.38
- joint RIGHT_SHOULDER_Z: limit lower=-1.22173 upper=1.91986 effort=1000 velocity=100 -> lower=-1.22173 upper=1.91986 effort=71.28 velocity=4.47

Commit message: Fix mass and inertia assymetry (#82)
* Averaged left and right upper arm masses and inertias

* Fixed inertias in the forearms

* Fixed some very messed up inertias in forearms

* Averaged the lower body masses and inertias

* Added modified mass and inertia to v2

* Fixed limits on v2

File: alex-models/alex_V2_description/urdf/alex_v2.leftUpperArm.urdf (robot description, URDF)
Before this commit: robot Alex, 5 links, 5 joints
Links:
- link LEFT_SHOULDER_X_LINK: mass 0.972 -> 1.16159753
- link LEFT_SHOULDER_Y_LINK: mass 2.99 -> 3.02036119
- link LEFT_SHOULDER_Z_LINK: mass 2.91 -> 3.117556435
Joints:
- joint LEFT_SHOULDER_X: limit lower=-0.349066 upper=2.79253 effort=150.0 velocity=9.0 -> lower=-0.349066 upper=2.79253 effort=160.7 velocity=10.38
- joint LEFT_SHOULDER_Y: limit lower=-3.141592 upper=1.22173 effort=150.0 velocity=9.0 -> lower=-3.141592 upper=1.22173 effort=160.7 velocity=10.38
- joint LEFT_SHOULDER_Z: limit lower=-1.91986 upper=1.22173 effort=80.0 velocity=11.5 -> lower=-1.91986 upper=1.22173 effort=71.28 velocity=4.47

File: alex-models/alex_V2_description/urdf/alex_v2.lowerBody.urdf (robot description, URDF)
Before this commit: robot Alex, 21 links, 20 joints
Links:
- link LEFT_FOOT: mass 1.28288609 -> 1.28831268
- link LEFT_HIP_X_LINK: mass 2.32977961 -> 2.33165613
- link LEFT_HIP_Z_LINK: mass 0.77281362 -> 0.761264535
- link LEFT_SHIN: mass 6.31087157 -> 6.33845554
- link LEFT_THIGH: mass 7.75 -> 8.281087115
- link PELVIS_LINK: mass 9.50083635 -> 7.161
- link RIGHT_FOOT: mass 1.28288609 -> 1.28831268
- link RIGHT_HIP_X_LINK: mass 2.32977248 -> 2.33165613
- link RIGHT_HIP_Z_LINK: mass 0.77281055 -> 0.761264535
- link RIGHT_SHIN: mass 6.31087157 -> 6.33845554
- link RIGHT_THIGH: mass 7.75 -> 8.281087115
Joints:
- joint LEFT_ANKLE_X: limit lower=-0.436332 upper=0.436332 effort=90 velocity=8 -> lower=-0.436332 upper=0.436332 effort=145.2 velocity=9.72
- joint LEFT_ANKLE_Y: limit lower=-1.0472 upper=0.523599 effort=180 velocity=8 -> lower=-1.0472 upper=0.523599 effort=193.6 velocity=9.72
- joint LEFT_HIP_X: limit lower=-0.3490658504 upper=0.872664626 effort=150 velocity=9 -> lower=-0.488692 upper=0.872665 effort=160.7 velocity=10.38
- joint LEFT_HIP_Y: limit lower=-2.61799 upper=0.785398 effort=200 velocity=8 -> lower=-2.61799 upper=0.785398 effort=217.2 velocity=9.3
- joint LEFT_HIP_Z: limit lower=-0.3490658504 upper=1.0472 effort=60 velocity=11 -> lower=-0.349066 upper=1.0472 effort=70.5 velocity=10.59
- joint LEFT_KNEE_Y: limit lower=0 upper=2.445206282 effort=200 velocity=8 -> lower=0 upper=2.44346 effort=217.2 velocity=9.3
- joint RIGHT_ANKLE_X: limit lower=-0.436332 upper=0.436332 effort=90 velocity=8 -> lower=-0.436332 upper=0.436332 effort=145.2 velocity=9.72
- joint RIGHT_ANKLE_Y: limit lower=-1.0472 upper=0.523599 effort=180 velocity=8 -> lower=-1.0472 upper=0.523599 effort=193.6 velocity=9.72
- joint RIGHT_HIP_X: limit lower=-0.872664626 upper=0.3490658504 effort=150 velocity=9 -> lower=-0.872665 upper=0.488692 effort=160.7 velocity=10.38
- joint RIGHT_HIP_Y: limit lower=-2.61799 upper=0.785398 effort=200 velocity=8 -> lower=-2.61799 upper=0.785398 effort=217.2 velocity=9.3
- joint RIGHT_HIP_Z: limit lower=-1.0472 upper=0.3490658504 effort=60 velocity=11 -> lower=-1.0472 upper=0.349066 effort=70.5 velocity=10.59
- joint RIGHT_KNEE_Y: limit lower=0 upper=2.445206282 effort=200 velocity=8 -> lower=0 upper=2.44346 effort=217.2 velocity=9.3
- joint SPINE_Z: limit lower=-0.5235987756 upper=0.5235987756 effort=150 velocity=9.0 -> lower=-0.523599 upper=0.523599 effort=160.7 velocity=10.38

File: alex-models/alex_V2_description/urdf/alex_v2.rightUpperArm.urdf (robot description, URDF)
Before this commit: robot Alex, 5 links, 5 joints
Links:
- link RIGHT_SHOULDER_X_LINK: mass 0.972 -> 1.16159753
- link RIGHT_SHOULDER_Y_LINK: mass 2.99 -> 3.02036119
- link RIGHT_SHOULDER_Z_LINK: mass 2.91 -> 3.117556435
Joints:
- joint RIGHT_SHOULDER_X: limit lower=-2.79253 upper=0.349066 effort=1000 velocity=100 -> lower=-2.79253 upper=0.349066 effort=160.7 velocity=10.38
- joint RIGHT_SHOULDER_Y: limit lower=-3.141592 upper=1.22173 effort=1000 velocity=100 -> lower=-3.141592 upper=1.22173 effort=160.7 velocity=10.38
- joint RIGHT_SHOULDER_Z: limit lower=-1.22173 upper=1.91986 effort=1000 velocity=100 -> lower=-1.22173 upper=1.91986 effort=71.28 velocity=4.47

Commit message: Added arm and torso fixes

File: alex-models/alex_V2_description/urdf/alex_v2.leftUpperArm.urdf (robot description, URDF)
Before this commit: robot Alex, 5 links, 5 joints
Joints:
- joint LEFT_SHOULDER_Y: origin xyz=-0.017 0.115474 0.352984 rpy=0.698132 0.0 0.0 -> xyz=0.002 0.10350000 0.36000000 rpy=0.698132 0.0 0.0

File: alex-models/alex_V2_description/urdf/alex_v2.lowerBody.urdf (robot description, URDF)
Before this commit: robot Alex, 22 links, 21 joints
Links:
- link TORSO_LINK: mass 18.534 -> 22.210

File: alex-models/alex_V2_description/urdf/alex_v2.rightUpperArm.urdf (robot description, URDF)
Before this commit: robot Alex, 5 links, 5 joints
Joints:
- joint RIGHT_SHOULDER_Y: origin xyz=-0.017 -0.115474 0.352984 rpy=-0.698132 0.0 0.0 -> xyz=0.002 -0.10350000 0.36000000 rpy=-0.698132 0.0 0.0
