Commit message: changed collisions to capsules

File: alex-models/alex_V2_description/urdf/alex_v2.leftFixedForearm.urdf (robot description, URDF)
Before this commit: robot Alex, 1 links, 1 joints
Links:
- link LEFT_ELBOW_Y_LINK: geometry collision capsule length=0.28 radius=0.03; visual mesh filename=package://alex_V1_description/meshes/cycloidal_arm/LEFT_ELB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

File: alex-models/alex_V2_description/urdf/alex_v2.lowerBody.urdf (robot description, URDF)
Before this commit: robot Alex, 22 links, 21 joints
Links:
- link LEFT_SHIN: geometry collision capsule length=0.3 radius=0.06; visual mesh filename=package://alex_V1_description/meshes/legs/LeftShin.obj
- link LEFT_THIGH: geometry collision capsule length=0.18 radius=0.075; visual mesh filename=package://alex_V1_description/meshes/legs/LeftThigh.obj
- link RIGHT_SHIN: geometry collision capsule length=0.3 radius=0.06; visual mesh filename=package://alex_V1_description/meshes/legs/RightShin.obj
- link RIGHT_THIGH: geometry collision capsule length=0.18 radius=0.075; visual mesh filename=package://alex_V1_description/meshes/legs/RightThigh.obj
- link TORSO_LINK: geometry collision box size=0.11 0.31 0.32; collision capsule length=0.25 radius=0.15

File: alex-models/alex_V2_description/urdf/alex_v2.rightFixedForearm.urdf (robot description, URDF)
Before this commit: robot Alex, 1 links, 1 joints
Links:
- link RIGHT_ELBOW_Y_LINK: geometry collision capsule length=0.28 radius=0.03; visual mesh filename=package://alex_V1_description/meshes/cycloidal_arm/RIGHT_EL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
