Commit message: Update rightForearm

File: alex-models/alex_V2_description/urdf/alex_v2.rightForearm.urdf (robot description, URDF)
Before this commit: robot Alex, 6 links, 6 joints
Links:
- link RIGHT_ELBOW_Y_LINK: geometry collision capsule length=0.18 radius=0.05; visual mesh filename=package://alex_V1_description/meshes/cycloidal_arm/RightElb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
- link RIGHT_GRIPPER_Z_LINK: geometry collision box size=0.08 0.025 0.075; collision cylinder length=0.06 radius=0.047
