Commit message: changed v1 xml to have ALEX_PDO_LIGHT. renamed xml 'address' field to 'position' for all xmls

File: alex-models/alex_V2_description/urdf/alex_v2.lowerBody.urdf (robot description, URDF)
Before this commit: robot Alex, 22 links, 21 joints
Links:
- added link LEFT_FOOT_IMU_LINK, mass 0
- added link RIGHT_FOOT_IMU_LINK, mass 0
Joints:
- added joint LEFT_FOOT_IMU_JOINT: type fixed, parent LEFT_FOOT, child LEFT_FOOT_IMU_LINK, origin xyz=-0.03575526 0.01180178 -0.04979705 rpy=0 0 1.570796, axis 0 0 1
- added joint RIGHT_FOOT_IMU_JOINT: type fixed, parent RIGHT_FOOT, child RIGHT_FOOT_IMU_LINK, origin xyz=-0.03575526 0.01180178 -0.04979705 rpy=0 0 1.570796, axis 0 0 1

Commit message: Commented out torso IMU for V2

File: alex-models/alex_V2_description/urdf/alex_v2.lowerBody.urdf (robot description, URDF)
Before this commit: robot Alex, 24 links, 23 joints
Links:
- removed link TORSO_IMU_LINK
Joints:
- removed joint TORSO_IMU_JOINT

Commit message: added v2 arm xmls and their zeros

File: alex-models/alex_V2_description/urdf/alex_v2.lowerBody.urdf (robot description, URDF)
Before this commit: robot Alex, 23 links, 22 joints
Links:
- added link TORSO_IMU_LINK, mass 0
Joints:
- added joint TORSO_IMU_JOINT: type fixed, parent TORSO_LINK, child TORSO_IMU_LINK, origin xyz=-0.009753 -0.01075 0.373405 rpy=0.0 0.0 -1.5708, axis 0 0 1

Commit message: updated the urdfs to remove the force torques

File: alex-models/alex_V2_description/urdf/alex_v2.lowerBody.urdf (robot description, URDF)
Before this commit: robot Alex, 21 links, 20 joints
Links:
- link LEFT_FOOT: mass 1.28831268 -> 0.810
- link RIGHT_FOOT: mass 1.28831268 -> 0.810

Commit message: Updated the V2 torso collisions

File: alex-models/alex_V2_description/urdf/alex_v2.lowerBody.urdf (robot description, URDF)
Before this commit: robot Alex, 23 links, 22 joints
Links:
- link TORSO_LINK: geometry collision box size=0.11 0.31 0.32; collision box size=0.18 0.26 0.45

Commit message: Feature/pmb java code (#78)
* Added PMB fields to HardwareStatus

* added message type for fort robotics rc handheld

* added message type for fort robotics rc handheld pt2

* added new torso PMB for v2 to v2 xmls

* added secondary pmb ethersnacks to torso.xml for v2

* added v2 arm xmls and their zeros

* set torso imus to not present in xml and urdf. set do pd control on twitter to false for right elbow

* changed junction aliases back to what they should be. changed v2 head xml APs

* added alex SDK fields for safe startup and shutdown

* added extra fields for auto startup/shutdown

* added field for fort robotics handheld battery level

* added urdfs and xml for forearms. Temp removed neck pitch stuff bc of new head

* removed head and feet IMUs from V2 URDFs

---------

Co-authored-by: Alexander OCU <rosie@ihmc.org>

File: alex-models/alex_V2_description/urdf/alex_v2.lowerBody.urdf (robot description, URDF)
Before this commit: robot Alex, 23 links, 22 joints
Links:
- removed link LEFT_FOOT_IMU_LINK
- removed link RIGHT_FOOT_IMU_LINK
Joints:
- removed joint LEFT_FOOT_IMU_JOINT
- removed joint RIGHT_FOOT_IMU_JOINT

Commit message: Added proper torso imu, corrected orientations for IMUs using zero stand

File: alex-models/alex_V2_description/urdf/alex_v2.lowerBody.urdf (robot description, URDF)
Before this commit: robot Alex, 21 links, 20 joints
Links:
- added link TORSO_IMU_LINK, mass 0
Joints:
- added joint TORSO_IMU_JOINT: type fixed, parent TORSO_LINK, child TORSO_IMU_LINK, origin xyz=0.094766 0.018319 0.255014 rpy=-1.561264 -0.329453 -1.570796, axis 0 0 1
- joint LEFT_HIP_X_IMU_JOINT: origin xyz=-0.01922309 0.10145013 -0.01488788 rpy=-1.570796 0 1.570796 -> xyz=-0.01922309 0.10145013 -0.01488788 rpy=-1.5803397 -0.0019308 1.570796
- joint LEFT_SHIN_IMU_JOINT: origin xyz=0.05655120 0.00084826 -0.15664831 rpy=1.403695170631842 0 -1.570796 -> xyz=0.05655120 0.00084826 -0.15664831 rpy=1.396297 0.005288 -1.570796
- joint LEFT_THIGH_IMU_JOINT: origin xyz=0.10004 0.03746 -0.21194 rpy=1.437982 0 1.570796 -> xyz=0.10004 0.03746 -0.21194 rpy=1.6974894 -0.006992 1.570796
- joint PELVIS_IMU_JOINT: origin xyz=-0.08687724 0.01225028 -0.08051472 rpy=-0.01399 -0.013054 1.570796 -> xyz=-0.08687724 0.01225028 -0.08051472 rpy=0.005114 -0.0001262 1.570796
- joint RIGHT_HIP_X_IMU_JOINT: origin xyz=-0.01922309 -0.07694987 -0.01488788 rpy=-1.570796 0 1.570796 -> xyz=-0.01922309 -0.07694987 -0.01488788 rpy=-1.582622 0.00171 1.570796
- joint RIGHT_SHIN_IMU_JOINT: origin xyz=0.05673025 -0.00875818 -0.15674961 rpy=1.403695170631842 0 -1.570796 -> xyz=0.05673025 -0.00875818 -0.15674961 rpy=1.4114646 0.00076419 -1.570796
- joint RIGHT_THIGH_IMU_JOINT: origin xyz=0.10003618 -0.033541826 -0.21194191 rpy=1.6947717585 0 1.570796 -> xyz=0.10003618 -0.033541826 -0.21194191 rpy=1.69207 -0.005085 1.570796

Commit message: Bugfix/hip roll issues (#87)
* Fixed the limit of hip roll for both, updated some joint zeros for V2

* Rolled back v1 changes, added robot specific roll changes to v2

---------

Co-authored-by: Alexander OCU <rosie@ihmc.org>

File: alex-models/alex_V2_description/urdf/alex_v2.lowerBody.urdf (robot description, URDF)
Before this commit: robot Alex, 22 links, 21 joints
Joints:
- joint LEFT_HIP_X: limit lower=-0.488692 upper=0.872665 effort=160.7 velocity=10.38 -> lower=-0.349066 upper=0.872665 effort=160.7 velocity=10.38
- joint RIGHT_HIP_X: limit lower=-0.872665 upper=0.488692 effort=160.7 velocity=10.38 -> lower=-0.872665 upper=0.349066 effort=160.7 velocity=10.38

Commit message: Added arm and torso fixes (#86)

File: alex-models/alex_V2_description/urdf/alex_v2.lowerBody.urdf (robot description, URDF)
Before this commit: robot Alex, 22 links, 21 joints
Links:
- link TORSO_LINK: mass 18.534 -> 22.210

Commit message: Update lower body collisions

File: alex-models/alex_V2_description/urdf/alex_v2.lowerBody.urdf (robot description, URDF)
Before this commit: robot Alex, 22 links, 21 joints
Links:
- link LEFT_SHIN: geometry collision capsule length=0.3 radius=0.065; visual mesh filename=package://alex_V1_description/meshes/legs/LeftShin.obj
- link LEFT_THIGH: geometry collision capsule length=0.18 radius=0.08; visual mesh filename=package://alex_V1_description/meshes/legs/LeftThigh.obj
- link RIGHT_SHIN: geometry collision capsule length=0.3 radius=0.065; visual mesh filename=package://alex_V1_description/meshes/legs/RightShin.obj
- link RIGHT_THIGH: geometry collision capsule length=0.18 radius=0.08; visual mesh filename=package://alex_V1_description/meshes/legs/RightThigh.obj
- link TORSO_LINK: geometry collision box size=0.11 0.31 0.32; collision capsule length=0.25 radius=0.15

Commit message: contributed calf collision capsule

File: alex-models/alex_V2_description/urdf/alex_v2.lowerBody.urdf (robot description, URDF)
Before this commit: robot Alex, 22 links, 21 joints
Links:
- link LEFT_SHIN: geometry collision capsule length=0.15 radius=0.04; collision capsule length=0.3 radius=0.065
- link RIGHT_SHIN: geometry collision capsule length=0.15 radius=0.04; collision capsule length=0.3 radius=0.065

Commit message: modified the calf collisions

File: alex-models/alex_V2_description/urdf/alex_v2.lowerBody.urdf (robot description, URDF)
Before this commit: robot Alex, 22 links, 21 joints
Links:
- link LEFT_SHIN: geometry collision capsule length=0.11 radius=0.065; collision capsule length=0.3 radius=0.065
- link RIGHT_SHIN: geometry collision capsule length=0.11 radius=0.065; collision capsule length=0.3 radius=0.065

Commit message: updated thigh collisions

File: alex-models/alex_V2_description/urdf/alex_v2.lowerBody.urdf (robot description, URDF)
Before this commit: robot Alex, 22 links, 21 joints
Links:
- link LEFT_THIGH: geometry collision capsule length=0.26 radius=0.08; visual mesh filename=package://alex_V1_description/meshes/legs/LeftThigh.obj
- link RIGHT_THIGH: geometry collision capsule length=0.26 radius=0.08; visual mesh filename=package://alex_V1_description/meshes/legs/RightThigh.obj

Commit message: refine the collisions

File: alex-models/alex_V2_description/urdf/alex_v2.lowerBody.urdf (robot description, URDF)
Before this commit: robot Alex, 22 links, 21 joints
Links:
- link LEFT_SHIN: geometry collision capsule length=0.11 radius=0.065; collision capsule length=0.3 radius=0.06
- link LEFT_THIGH: geometry collision capsule length=0.26 radius=0.08; collision cylinder length=0.155 radius=0.03
- link RIGHT_SHIN: geometry collision capsule length=0.11 radius=0.065; collision capsule length=0.3 radius=0.06
- link RIGHT_THIGH: geometry collision capsule length=0.26 radius=0.08; collision cylinder length=0.155 radius=0.03
