Commit message: added urdfs and xml for forearms. Temp removed neck pitch stuff bc of new head

File: alex-models/alex_V2_description/urdf/alex_v2.head.urdf (robot description, URDF)
Before this commit: robot Alex, 3 links, 3 joints
Joints:
- joint NECK_Y: type revolute -> fixed

Commit message: removed head and feet IMUs from V2 URDFs

File: alex-models/alex_V2_description/urdf/alex_v2.head.urdf (robot description, URDF)
Before this commit: robot Alex, 3 links, 3 joints
Links:
- removed link HEAD_IMU_LINK
Joints:
- removed joint HEAD_IMU_JOINT

File: alex-models/alex_V2_description/urdf/alex_v2.lowerBody.urdf (robot description, URDF)
Before this commit: robot Alex, 23 links, 22 joints
Links:
- removed link LEFT_FOOT_IMU_LINK
- removed link RIGHT_FOOT_IMU_LINK
Joints:
- removed joint LEFT_FOOT_IMU_JOINT
- removed joint RIGHT_FOOT_IMU_JOINT

Commit message: New neck and head for V2

File: alex-models/alex_V2_description/urdf/alex_v2.head.urdf (robot description, URDF)
Before this commit: robot Alex, 3 links, 3 joints
Links:
- link HEAD_LINK: mass 1.27065932 -> 2.53238993; geometry collision sphere radius=0.14; visual mesh filename=package://alex_V2_description/meshes/head.obj
- link NECK_Z_LINK: mass 1.03172573 -> 0.50522843; geometry visual mesh filename=package://alex_V2_description/meshes/neck.obj
Joints:
- joint HEAD_IMU_JOINT: origin xyz=0.040556 -0.014155 0.057016 rpy=0.56723 0.0 1.5708  -> xyz=-0.02432603 -0.00225290 0.07425800 rpy=0.0 0.0 0.0
- joint NECK_Y: origin xyz=0.025 0.01 0.189597 rpy=0 0 0 -> xyz=0.015 -0.01 0.130 rpy=0 0 0
- joint NECK_Z: origin xyz=-0.015 0 0.450403 rpy=0 0 0 -> xyz=0.0072 0 0.4669 rpy=0 0 0

Commit message: updates for joint zeros, new option for using output from motor encoder

File: alex-models/alex_V2_description/urdf/alex_v2.head.urdf (robot description, URDF)
Before this commit: robot Alex, 3 links, 3 joints
Joints:
- joint NECK_Z: limit lower=-1.5708 upper=1.5708 effort=20.86 velocity=17.3 -> lower=-1.22173 upper=1.22173 effort=20.86 velocity=17.3

Commit message: Fix ZED URDF origins, OBJ files

File: alex-models/alex_V2_description/urdf/alex_v2.head.urdf (robot description, URDF)
Before this commit: robot Alex, 4 links, 4 joints
Joints:
- joint HEAD_ZED_X_MINI_JOINT: origin xyz=0.13041 -0.01079 0.02381 rpy=0.0 0.3633 0.0 -> xyz=0.11603 0.009965 -0.02983 rpy=0.0 0.3633 0.0

File: alex-models/alex_V2_description/urdf/alex_v2.lowerBody.urdf (robot description, URDF)
Before this commit: robot Alex, 23 links, 22 joints
Joints:
- joint TORSO_ZED_X_MINI_JOINT: origin xyz=0.1 0.0 0.05 rpy=0.0 0.907571 0.0 -> xyz=0.108969 0.0 0.035381 rpy=0.0 0.907571 0.0

Commit message: Use lower-poly meshes, include glb for RDX

File: alex-models/alex_V2_description/urdf/alex_v2.head.urdf (robot description, URDF)
Before this commit: robot Alex, 3 links, 3 joints
Links:
- link HEAD_LINK: geometry collision sphere radius=0.14; visual mesh filename=package://alex_V2_description/meshes/AlexV2Head.obj
- link NECK_Z_LINK: geometry visual mesh filename=package://alex_V2_description/meshes/AlexV2Neck.obj

File: alex-models/alex_V2_description/urdf/alex_v2.lowerBody.urdf (robot description, URDF)
Before this commit: robot Alex, 22 links, 21 joints
Links:
- link TORSO_LINK: geometry collision box size=0.11 0.31 0.32; collision capsule length=0.25 radius=0.15

Commit message: [Feature] ZEDs in URDF (#100)
* WIP - adding ZEDs to URDF

* Fix ZED URDF origins, OBJ files

* Defeature ZED X Mini mesh

File: alex-models/alex_V2_description/urdf/alex_v2.head.urdf (robot description, URDF)
Before this commit: robot Alex, 3 links, 3 joints
Links:
- added link HEAD_ZED_X_MINI_LINK, mass 0; visual mesh filename=package://alex_V1_description/meshes/ZEDXMini.obj
Joints:
- added joint HEAD_ZED_X_MINI_JOINT: type fixed, parent HEAD_LINK, child HEAD_ZED_X_MINI_LINK, origin xyz=0.11603 0.009965 -0.02983 rpy=0.0 0.3633 0.0

File: alex-models/alex_V2_description/urdf/alex_v2.lowerBody.urdf (robot description, URDF)
Before this commit: robot Alex, 22 links, 21 joints
Links:
- added link TORSO_ZED_X_MINI_LINK, mass 0; visual mesh filename=package://alex_V1_description/meshes/ZEDXMini.obj
Joints:
- added joint TORSO_ZED_X_MINI_JOINT: type fixed, parent TORSO_LINK, child TORSO_ZED_X_MINI_LINK, origin xyz=0.108969 0.0 0.035381 rpy=0.0 0.907571 0.0

Commit message: alex full convex

File: alex-models/alex_V2_description/urdf/alex_v2.head.urdf (robot description, URDF)
Before this commit: robot Alex, 3 links, 3 joints
Links:
- link HEAD_LINK: geometry collision mesh filename=package://alex_V2_description/meshes/head_convex.stl; visual mesh filename=package://alex_V2_description/meshes/head.obj

File: alex-models/alex_V2_description/urdf/alex_v2.leftForearm.urdf (robot description, URDF)
Before this commit: robot Alex, 6 links, 6 joints
Links:
- link LEFT_ELBOW_Y_LINK: geometry collision mesh filename=package://alex_V2_description/meshes/cycloidal_arm/LeftElbo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; visual mesh filename=package://alex_V2_description/meshes/cycloidal_arm/LeftElbo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
- link LEFT_GRIPPER_Z_LINK: geometry collision cylinder length=0.06 radius=0.047; collision mesh filename=package://alex_V2_description/meshes/cycloidal_arm/LeftGrip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
- link LEFT_WRIST_X_LINK: geometry visual mesh filename=package://alex_V2_description/meshes/cycloidal_arm/LeftWris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
- link LEFT_WRIST_Z_LINK: geometry collision mesh filename=package://alex_V2_description/meshes/cycloidal_arm/LeftWris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; visual mesh filename=package://alex_V2_description/meshes/cycloidal_arm/LeftWris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

File: alex-models/alex_V2_description/urdf/alex_v2.leftUpperArm.urdf (robot description, URDF)
Before this commit: robot Alex, 5 links, 5 joints
Links:
- link LEFT_SHOULDER_X_LINK: geometry visual mesh filename=package://alex_V2_description/meshes/cycloidal_arm/LeftShou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
- link LEFT_SHOULDER_Y_LINK: geometry visual mesh filename=package://alex_V2_description/meshes/cycloidal_arm/LeftShou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
- link LEFT_SHOULDER_Z_LINK: geometry collision mesh filename=package://alex_V2_description/meshes/cycloidal_arm/LeftShou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; visual mesh filename=package://alex_V2_description/meshes/cycloidal_arm/LeftShou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

File: alex-models/alex_V2_description/urdf/alex_v2.lowerBody.urdf (robot description, URDF)
Before this commit: robot Alex, 22 links, 21 joints
Links:
- link LEFT_ANKLE_Y_LINK: geometry visual mesh filename=package://alex_V2_description/meshes/legs/AnklePitchLink.obj
- link LEFT_FOOT: geometry collision mesh filename=package://alex_V2_description/meshes/legs/Foot_convex.stl; visual mesh filename=package://alex_V2_description/meshes/legs/Foot.obj
- link LEFT_HIP_X_LINK: geometry collision mesh filename=package://alex_V2_description/meshes/legs/LeftHipRollLink_c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; visual mesh filename=package://alex_V2_description/meshes/legs/LeftHipRollLink.o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
- link LEFT_HIP_Z_LINK: geometry visual mesh filename=package://alex_V2_description/meshes/legs/LeftHipYawLink.obj
- link LEFT_SHIN: geometry collision mesh filename=package://alex_V2_description/meshes/legs/LeftShin_convex.s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; visual mesh filename=package://alex_V2_description/meshes/legs/LeftShin.obj
- link LEFT_THIGH: geometry collision mesh filename=package://alex_V2_description/meshes/legs/LeftThigh_convex.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; visual mesh filename=package://alex_V2_description/meshes/legs/LeftThigh.obj
- link PELVIS_LINK: geometry collision mesh filename=package://alex_V2_description/meshes/legs/Pelvis_convex.stl; visual mesh filename=package://alex_V2_description/meshes/legs/Pelvis.obj
- link RIGHT_ANKLE_Y_LINK: geometry visual mesh filename=package://alex_V2_description/meshes/legs/AnklePitchLink.obj
- link RIGHT_FOOT: geometry collision mesh filename=package://alex_V2_description/meshes/legs/Foot_convex.stl; visual mesh filename=package://alex_V2_description/meshes/legs/Foot.obj
- link RIGHT_HIP_X_LINK: geometry collision mesh filename=package://alex_V2_description/meshes/legs/RightHipRollLink_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; visual mesh filename=package://alex_V2_description/meshes/legs/RightHipRollLink.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
- link RIGHT_HIP_Z_LINK: geometry visual mesh filename=package://alex_V2_description/meshes/legs/RightHipYawLink.o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
- link RIGHT_SHIN: geometry collision mesh filename=package://alex_V2_description/meshes/legs/RightShin_convex.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; visual mesh filename=package://alex_V2_description/meshes/legs/RightShin.obj
- link RIGHT_THIGH: geometry collision mesh filename=package://alex_V2_description/meshes/legs/RightThigh_convex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; visual mesh filename=package://alex_V2_description/meshes/legs/RightThigh.obj
- link TORSO_LINK: geometry collision mesh filename=package://alex_V2_description/meshes/torso_convex.stl; visual mesh filename=package://alex_V2_description/meshes/torso.obj

File: alex-models/alex_V2_description/urdf/alex_v2.rightForearm.urdf (robot description, URDF)
Before this commit: robot Alex, 6 links, 6 joints
Links:
- link RIGHT_ELBOW_Y_LINK: geometry collision mesh filename=package://alex_V2_description/meshes/cycloidal_arm/RightElb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; visual mesh filename=package://alex_V2_description/meshes/cycloidal_arm/RightElb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
- link RIGHT_GRIPPER_Z_LINK: geometry collision cylinder length=0.06 radius=0.047; collision mesh filename=package://alex_V2_description/meshes/cycloidal_arm/RightGri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
- link RIGHT_WRIST_X_LINK: geometry visual mesh filename=package://alex_V2_description/meshes/cycloidal_arm/RightWri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
- link RIGHT_WRIST_Z_LINK: geometry collision mesh filename=package://alex_V2_description/meshes/cycloidal_arm/RightWri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; visual mesh filename=package://alex_V2_description/meshes/cycloidal_arm/RightWri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

File: alex-models/alex_V2_description/urdf/alex_v2.rightUpperArm.urdf (robot description, URDF)
Before this commit: robot Alex, 5 links, 5 joints
Links:
- link RIGHT_SHOULDER_X_LINK: geometry visual mesh filename=package://alex_V2_description/meshes/cycloidal_arm/RightSho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
- link RIGHT_SHOULDER_Y_LINK: geometry visual mesh filename=package://alex_V2_description/meshes/cycloidal_arm/RightSho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
- link RIGHT_SHOULDER_Z_LINK: geometry collision mesh filename=package://alex_V2_description/meshes/cycloidal_arm/RightSho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; visual mesh filename=package://alex_V2_description/meshes/cycloidal_arm/RightSho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
