Commit message: Update leftForearm with new collsions

File: alex-models/alex_V2_description/urdf/alex_v2.leftForearm.urdf (robot description, URDF)
Before this commit: robot Alex, 6 links, 6 joints
Links:
- link LEFT_ELBOW_Y_LINK: geometry collision capsule length=0.18 radius=0.05; visual mesh filename=package://alex_V1_description/meshes/cycloidal_arm/LeftElbo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
- link LEFT_GRIPPER_Z_LINK: geometry collision box size=0.08 0.025 0.075; collision cylinder length=0.06 radius=0.047

Commit message: Feature/full body simple collisions (#91)
* Update lower body collisions

* Update leftForearm with new collsions

* Update rightForearm

* Fixed Urdu error in new collision

* Update alex_v2.leftForearm.urdf

removed closing ellipses

* Fix formatting of left gripper collision element

removed comment closer

* Fix formatting of right gripper collision element

removed comment closers

* fixed the right gripper z

* contributed calf collision capsule

* modified the calf collisions

* updated thigh collisions

---------

Co-authored-by: Geoffrey Clark <42682271+GeoffreyMClark@users.noreply.github.com>

File: alex-models/alex_V2_description/urdf/alex_v2.leftForearm.urdf (robot description, URDF)
Before this commit: robot Alex, 6 links, 6 joints
Links:
- link LEFT_ELBOW_Y_LINK: geometry collision capsule length=0.18 radius=0.05; visual mesh filename=package://alex_V1_description/meshes/cycloidal_arm/LeftElbo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
- link LEFT_GRIPPER_Z_LINK: geometry collision box size=0.08 0.025 0.075; collision cylinder length=0.06 radius=0.047

File: alex-models/alex_V2_description/urdf/alex_v2.lowerBody.urdf (robot description, URDF)
Before this commit: robot Alex, 22 links, 21 joints
Links:
- link LEFT_SHIN: geometry collision capsule length=0.11 radius=0.065; collision capsule length=0.3 radius=0.065
- link LEFT_THIGH: geometry collision capsule length=0.26 radius=0.08; visual mesh filename=package://alex_V1_description/meshes/legs/LeftThigh.obj
- link RIGHT_SHIN: geometry collision capsule length=0.11 radius=0.065; collision capsule length=0.3 radius=0.065
- link RIGHT_THIGH: geometry collision capsule length=0.26 radius=0.08; visual mesh filename=package://alex_V1_description/meshes/legs/RightThigh.obj
- link TORSO_LINK: geometry collision box size=0.11 0.31 0.32; collision capsule length=0.25 radius=0.15

File: alex-models/alex_V2_description/urdf/alex_v2.rightForearm.urdf (robot description, URDF)
Before this commit: robot Alex, 6 links, 6 joints
Links:
- link RIGHT_ELBOW_Y_LINK: geometry collision capsule length=0.18 radius=0.05; visual mesh filename=package://alex_V1_description/meshes/cycloidal_arm/RightElb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
- link RIGHT_GRIPPER_Z_LINK: geometry collision box size=0.08 0.025 0.075; collision cylinder length=0.06 radius=0.047

Commit message: updated the collision to capsules

File: alex-models/alex_V2_description/urdf/alex_v2.leftForearm.urdf (robot description, URDF)
Before this commit: robot Alex, 6 links, 6 joints
Links:
- link LEFT_GRIPPER_Z_LINK: geometry collision box size=0.08 0.025 0.075; collision capsule length=0.1 radius=0.04

File: alex-models/alex_V2_description/urdf/alex_v2.rightForearm.urdf (robot description, URDF)
Before this commit: robot Alex, 6 links, 6 joints
Links:
- link RIGHT_GRIPPER_Z_LINK: geometry collision box size=0.08 0.025 0.075; collision capsule length=0.1 radius=0.04

Commit message: meshes collisions

File: alex-models/alex_V2_description/urdf/alex_v2.leftForearm.urdf (robot description, URDF)
Before this commit: robot Alex, 6 links, 6 joints
Links:
- link LEFT_GRIPPER_Z_LINK: geometry collision cylinder length=0.11 radius=0.0285; visual mesh filename=package://alex_V2_description/meshes/cycloidal_arm/LeftGrip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
- link LEFT_WRIST_X_LINK: geometry collision mesh filename=package://alex_V2_description/meshes/cycloidal_arm/LeftWris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; visual mesh filename=package://alex_V2_description/meshes/cycloidal_arm/LeftWris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

File: alex-models/alex_V2_description/urdf/alex_v2.leftUpperArm.urdf (robot description, URDF)
Before this commit: robot Alex, 5 links, 5 joints
Links:
- link LEFT_SHOULDER_X_LINK: geometry collision mesh filename=package://alex_V2_description/meshes/cycloidal_arm/LeftShou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; visual mesh filename=package://alex_V2_description/meshes/cycloidal_arm/LeftShou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
- link LEFT_SHOULDER_Y_LINK: geometry collision mesh filename=package://alex_V2_description/meshes/cycloidal_arm/LeftShou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; visual mesh filename=package://alex_V2_description/meshes/cycloidal_arm/LeftShou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

File: alex-models/alex_V2_description/urdf/alex_v2.rightForearm.urdf (robot description, URDF)
Before this commit: robot Alex, 6 links, 6 joints
Links:
- link RIGHT_GRIPPER_Z_LINK: geometry collision cylinder length=0.11 radius=0.0285; visual mesh filename=package://alex_V2_description/meshes/cycloidal_arm/RightGri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
- link RIGHT_WRIST_X_LINK: geometry collision mesh filename=package://alex_V2_description/meshes/cycloidal_arm/RightWri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; visual mesh filename=package://alex_V2_description/meshes/cycloidal_arm/RightWri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

File: alex-models/alex_V2_description/urdf/alex_v2.rightUpperArm.urdf (robot description, URDF)
Before this commit: robot Alex, 5 links, 5 joints
Links:
- link RIGHT_SHOULDER_X_LINK: geometry collision mesh filename=package://alex_V2_description/meshes/cycloidal_arm/RightSho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; visual mesh filename=package://alex_V2_description/meshes/cycloidal_arm/RightSho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
- link RIGHT_SHOULDER_Y_LINK: geometry collision mesh filename=package://alex_V2_description/meshes/cycloidal_arm/RightSho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; visual mesh filename=package://alex_V2_description/meshes/cycloidal_arm/RightSho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

Commit message: convex meshes non colliding

File: alex-models/alex_V2_description/urdf/alex_v2.leftForearm.urdf (robot description, URDF)
Before this commit: robot Alex, 6 links, 6 joints
Links:
- link LEFT_GRIPPER_Z_LINK: geometry collision mesh filename=package://alex_V2_description/meshes/cycloidal_arm/LeftFist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; visual mesh filename=package://alex_V2_description/meshes/cycloidal_arm/LeftGrip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

File: alex-models/alex_V2_description/urdf/alex_v2.rightForearm.urdf (robot description, URDF)
Before this commit: robot Alex, 6 links, 6 joints
Links:
- link RIGHT_GRIPPER_Z_LINK: geometry collision mesh filename=package://alex_V2_description/meshes/cycloidal_arm/RightFis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; visual mesh filename=package://alex_V2_description/meshes/cycloidal_arm/RightGri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
