Commit message: convex meshes

File: alex-models/alex_V2_description/urdf/alex_v2.head_convex.urdf (robot description, URDF)
Before this commit: robot Alex, 4 links, 4 joints
Links:
- removed link HEAD_ZED_X_MINI_LINK
- link HEAD_LINK: geometry collision mesh filename=package://alex_V2_description/meshes/head_convex.stl; visual mesh filename=package://alex_V2_description/meshes/head.obj
- link NECK_Z_LINK: geometry visual mesh filename=package://alex_V2_description/meshes/neck.obj
Joints:
- removed joint HEAD_ZED_X_MINI_JOINT
- joint NECK_Z: limit lower=-1.22173 upper=1.22173 effort=20.86 velocity=17.3 -> lower=-1.5708 upper=1.5708 effort=20.86 velocity=17.3

File: alex-models/alex_V2_description/urdf/alex_v2.leftForearm.urdf (robot description, URDF)
Before this commit: robot Alex, 6 links, 6 joints
Links:
- link LEFT_ELBOW_Y_LINK: geometry collision capsule length=0.18 radius=0.05; visual mesh filename=package://alex_V1_description/meshes/cycloidal_arm/LeftElbo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
- link LEFT_GRIPPER_Z_LINK: geometry collision box size=0.08 0.025 0.075; collision capsule length=0.1 radius=0.04
- link LEFT_WRIST_X_LINK: geometry visual mesh filename=package://alex_V1_description/meshes/cycloidal_arm/LeftWris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
- link LEFT_WRIST_Z_LINK: geometry collision box size=0.01 0.06 0.1; collision cylinder length=0.12 radius=0.044

File: alex-models/alex_V2_description/urdf/alex_v2.leftForearm_convex.urdf (robot description, URDF)
Before this commit: robot Alex, 6 links, 6 joints
Links:
- removed link RIGHT_ELBOW_Y_LINK
- removed link RIGHT_GRIPPER_Z_IMU_LINK
- removed link RIGHT_GRIPPER_Z_LINK
- removed link RIGHT_WRIST_X_LINK
- removed link RIGHT_WRIST_Z_IMU_LINK
- removed link RIGHT_WRIST_Z_LINK
- added link LEFT_ELBOW_Y_LINK, mass 0.45; collision mesh filename=package://alex_V2_description/meshes/cycloidal_arm/LeftElbo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; visual mesh filename=package://alex_V2_description/meshes/cycloidal_arm/LeftElbo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
- added link LEFT_GRIPPER_Z_IMU_LINK, mass 0
- added link LEFT_GRIPPER_Z_LINK, mass 0.287; collision mesh filename=package://alex_V2_description/meshes/cycloidal_arm/LeftFist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; visual mesh filename=package://alex_V2_description/meshes/cycloidal_arm/LeftGrip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
- added link LEFT_WRIST_X_LINK, mass 0.909; collision mesh filename=package://alex_V2_description/meshes/cycloidal_arm/LeftWris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; visual mesh filename=package://alex_V2_description/meshes/cycloidal_arm/LeftWris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
- added link LEFT_WRIST_Z_IMU_LINK, mass 0
- added link LEFT_WRIST_Z_LINK, mass 1.547; collision mesh filename=package://alex_V2_description/meshes/cycloidal_arm/LeftWris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; visual mesh filename=package://alex_V2_description/meshes/cycloidal_arm/LeftWris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
Joints:
- removed joint RIGHT_ELBOW_Y
- removed joint RIGHT_GRIPPER_Z
- removed joint RIGHT_GRIPPER_Z_IMU_JOINT
- removed joint RIGHT_WRIST_X
- removed joint RIGHT_WRIST_Z
- removed joint RIGHT_WRIST_Z_IMU_JOINT
- added joint LEFT_ELBOW_Y: type revolute, parent LEFT_SHOULDER_Z_LINK, child LEFT_ELBOW_Y_LINK, origin xyz=0.015 0.0 -0.3127 rpy=0.0 0.0 0.0, axis 0.0 1.0 0.0, limit lower=-2.35619 upper=0.174533 effort=71.28 velocity=4.47
- added joint LEFT_GRIPPER_Z: type revolute, parent LEFT_WRIST_X_LINK, child LEFT_GRIPPER_Z_LINK, origin xyz=0.0 0.013 -0.031 rpy=0.0 0.0 0.0, axis 0.0 0.0 1.0, limit lower=-2.61799 upper=2.61799 effort=20.86 velocity=17.3
- added joint LEFT_GRIPPER_Z_IMU_JOINT: type fixed, parent LEFT_GRIPPER_Z_LINK, child LEFT_GRIPPER_Z_IMU_LINK, origin xyz=0 0 0 rpy=0 0 0, axis 0 0 1
- added joint LEFT_WRIST_X: type revolute, parent LEFT_WRIST_Z_LINK, child LEFT_WRIST_X_LINK, origin xyz=0.0 -0.013 -0.25 rpy=0.0 0.0 0.0, axis 1 0 0, limit lower=-1.8326 upper=0.610865 effort=20.86 velocity=17.3
- added joint LEFT_WRIST_Z: type revolute, parent LEFT_ELBOW_Y_LINK, child LEFT_WRIST_Z_LINK, origin xyz=-0.015 0.0 0.0 rpy=0.0 0.0 0.0, axis 0.0 0.0 1.0, limit lower=-2.61799 upper=2.61799 effort=20.86 velocity=17.3
- added joint LEFT_WRIST_Z_IMU_JOINT: type fixed, parent LEFT_WRIST_Z_LINK, child LEFT_WRIST_Z_IMU_LINK, origin xyz=-0.033554 0.010450 -0.148527 rpy=1.571 0.0 1.571, axis 0 0 1

File: alex-models/alex_V2_description/urdf/alex_v2.leftUpperArm_convex.urdf (robot description, URDF)
Before this commit: robot Alex, 5 links, 5 joints
Links:
- link LEFT_SHOULDER_X_LINK: geometry collision mesh filename=package://alex_V2_description/meshes/cycloidal_arm/LeftShou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; visual mesh filename=package://alex_V2_description/meshes/cycloidal_arm/LeftShou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
- link LEFT_SHOULDER_Y_LINK: geometry collision mesh filename=package://alex_V2_description/meshes/cycloidal_arm/LeftShou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; visual mesh filename=package://alex_V2_description/meshes/cycloidal_arm/LeftShou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
- link LEFT_SHOULDER_Z_LINK: geometry collision mesh filename=package://alex_V2_description/meshes/cycloidal_arm/LeftShou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; visual mesh filename=package://alex_V2_description/meshes/cycloidal_arm/LeftShou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

File: alex-models/alex_V2_description/urdf/alex_v2.lowerBody_convex.urdf (robot description, URDF)
Before this commit: robot Alex, 23 links, 22 joints
Links:
- removed link TORSO_ZED_X_MINI_LINK
- link LEFT_ANKLE_Y_LINK: geometry visual mesh filename=package://alex_V2_description/meshes/legs/AnklePitchLink.obj
- link LEFT_FOOT: geometry collision mesh filename=package://alex_V2_description/meshes/legs/Foot_convex.stl; visual mesh filename=package://alex_V2_description/meshes/legs/Foot.obj
- link LEFT_HIP_X_LINK: geometry collision mesh filename=package://alex_V2_description/meshes/legs/LeftHipRollLink_c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; visual mesh filename=package://alex_V2_description/meshes/legs/LeftHipRollLink.o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
- link LEFT_HIP_Z_LINK: geometry visual mesh filename=package://alex_V2_description/meshes/legs/LeftHipYawLink.obj
- link LEFT_SHIN: geometry collision mesh filename=package://alex_V2_description/meshes/legs/LeftShin_convex.s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; visual mesh filename=package://alex_V2_description/meshes/legs/LeftShin.obj
- link LEFT_THIGH: geometry collision mesh filename=package://alex_V2_description/meshes/legs/LeftThigh_convex.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; visual mesh filename=package://alex_V2_description/meshes/legs/LeftThigh.obj
- link PELVIS_LINK: geometry collision mesh filename=package://alex_V2_description/meshes/legs/Pelvis_convex.stl; visual mesh filename=package://alex_V2_description/meshes/legs/Pelvis.obj
- link RIGHT_ANKLE_Y_LINK: geometry visual mesh filename=package://alex_V2_description/meshes/legs/AnklePitchLink.obj
- link RIGHT_FOOT: geometry collision mesh filename=package://alex_V2_description/meshes/legs/Foot_convex.stl; visual mesh filename=package://alex_V2_description/meshes/legs/Foot.obj
- link RIGHT_HIP_X_LINK: geometry collision mesh filename=package://alex_V2_description/meshes/legs/RightHipRollLink_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; visual mesh filename=package://alex_V2_description/meshes/legs/RightHipRollLink.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
- link RIGHT_HIP_Z_LINK: geometry visual mesh filename=package://alex_V2_description/meshes/legs/RightHipYawLink.o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
- link RIGHT_SHIN: geometry collision mesh filename=package://alex_V2_description/meshes/legs/RightShin_convex.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; visual mesh filename=package://alex_V2_description/meshes/legs/RightShin.obj
- link RIGHT_THIGH: geometry collision mesh filename=package://alex_V2_description/meshes/legs/RightThigh_convex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; visual mesh filename=package://alex_V2_description/meshes/legs/RightThigh.obj
- link TORSO_LINK: geometry collision mesh filename=package://alex_V2_description/meshes/torso_convex.stl; visual mesh filename=package://alex_V2_description/meshes/torso.obj
Joints:
- removed joint TORSO_ZED_X_MINI_JOINT

File: alex-models/alex_V2_description/urdf/alex_v2.rightForearm_convex.urdf (robot description, URDF)
Before this commit: robot Alex, 6 links, 6 joints
Links:
- link RIGHT_ELBOW_Y_LINK: geometry collision mesh filename=package://alex_V2_description/meshes/cycloidal_arm/RightElb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; visual mesh filename=package://alex_V2_description/meshes/cycloidal_arm/RightElb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
- link RIGHT_GRIPPER_Z_LINK: geometry collision mesh filename=package://alex_V2_description/meshes/cycloidal_arm/RightFis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; visual mesh filename=package://alex_V2_description/meshes/cycloidal_arm/RightGri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
- link RIGHT_WRIST_X_LINK: geometry collision mesh filename=package://alex_V2_description/meshes/cycloidal_arm/RightWri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; visual mesh filename=package://alex_V2_description/meshes/cycloidal_arm/RightWri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
- link RIGHT_WRIST_Z_LINK: geometry collision mesh filename=package://alex_V2_description/meshes/cycloidal_arm/RightWri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; visual mesh filename=package://alex_V2_description/meshes/cycloidal_arm/RightWri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

File: alex-models/alex_V2_description/urdf/alex_v2.rightUpperArm_convex.urdf (robot description, URDF)
Before this commit: robot Alex, 5 links, 5 joints
Links:
- link RIGHT_SHOULDER_X_LINK: geometry collision mesh filename=package://alex_V2_description/meshes/cycloidal_arm/RightSho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; visual mesh filename=package://alex_V2_description/meshes/cycloidal_arm/RightSho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
- link RIGHT_SHOULDER_Y_LINK: geometry collision mesh filename=package://alex_V2_description/meshes/cycloidal_arm/RightSho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; visual mesh filename=package://alex_V2_description/meshes/cycloidal_arm/RightSho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
- link RIGHT_SHOULDER_Z_LINK: geometry collision mesh filename=package://alex_V2_description/meshes/cycloidal_arm/RightSho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; visual mesh filename=package://alex_V2_description/meshes/cycloidal_arm/RightSho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
