Commit message: Added actuator xmls and placeholder hardware xmls to be verified later

File: alex-models/alex_purdue_description/urdf/alex_purdue.rightForearm.urdf (robot description, URDF)
Before this commit: robot Alex, 6 links, 6 joints
Links:
- removed link LEFT_GRIPPER_Y_LINK
- added link RIGHT_GRIPPER_Y_LINK, mass 0.184; visual mesh filename=package://alex_purdue_description/meshes/left_arm/l_gripper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

File: alex-models/alex_purdue_description/urdf/alex_purdue.rightUpperArm.urdf (robot description, URDF)
Before this commit: robot Alex, 5 links, 5 joints
Links:
- removed link LEFT_SHOULDER_Z_LINK
- added link RIGHT_SHOULDER_Z_LINK, mass 3.67445507; visual mesh filename=package://alex_purdue_description/meshes/right_arm/r_should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

File: alex-models/alex_purdue_description/urdf/alex_purdue.sakeGripper.urdf (robot description, URDF)
Before this commit: robot Alex, 1 links, 2 joints
Links:
- removed link SAKE_GRIPPER
- added link LEFT_SAKE_GRIPPER_LINK, mass 0.43668602; visual mesh filename=package://alex_purdue_description/meshes/grippers/sake_grip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
- added link RIGHT_SAKE_GRIPPER_LINK, mass 0.43668602; visual mesh filename=package://alex_purdue_description/meshes/grippers/sake_grip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
Joints:
- joint LEFT_SAKE_GRIPPER: child SAKE_GRIPPER -> LEFT_SAKE_GRIPPER_LINK
- joint RIGHT_SAKE_GRIPPER: child SAKE_GRIPPER -> RIGHT_SAKE_GRIPPER_LINK
