Commit message: fixed some hardstop values in urdf and xmls, zerod robot

File: alex-models/alex_purdue_description/urdf/alex_purdue.leftForearm.urdf (robot description, URDF)
Before this commit: robot Alex, 6 links, 6 joints
Joints:
- joint LEFT_GRIPPER_Y: limit lower=-2.61799 upper=2.61799 effort=20.86 velocity=17.3 -> lower=-0.785398 upper=0.785398 effort=20.86 velocity=17.3
- joint LEFT_WRIST_X: limit lower=-1.8326 upper=0.610865 effort=20.86 velocity=17.3 -> lower=-1.48353 upper=0.959931 effort=20.86 velocity=17.3

File: alex-models/alex_purdue_description/urdf/alex_purdue.leftUpperArm.urdf (robot description, URDF)
Before this commit: robot Alex, 5 links, 5 joints
Joints:
- joint LEFT_SHOULDER_X: limit lower=-0.349066 upper=2.79253 effort=160.7 velocity=10.38 -> lower=-0.261799 upper=2.87979 effort=160.7 velocity=10.38

File: alex-models/alex_purdue_description/urdf/alex_purdue.rightForearm.urdf (robot description, URDF)
Before this commit: robot Alex, 6 links, 6 joints
Joints:
- joint RIGHT_GRIPPER_Y: limit lower=-2.61799 upper=2.61799 effort=20.86 velocity=17.3 -> lower=-0.785398 upper=0.785398 effort=20.86 velocity=17.3
- joint RIGHT_WRIST_X: limit lower=-1.8326 upper=0.610865 effort=20.86 velocity=17.3 -> lower=-0.959931 upper=1.48353 effort=20.86 velocity=17.3

File: alex-models/alex_purdue_description/urdf/alex_purdue.rightUpperArm.urdf (robot description, URDF)
Before this commit: robot Alex, 5 links, 5 joints
Joints:
- joint RIGHT_SHOULDER_X: limit lower=-0.349066 upper=2.79253 effort=160.7 velocity=10.38 -> lower=-2.87979 upper=0.261799 effort=160.7 velocity=10.38
- joint RIGHT_SHOULDER_Z: limit lower=-1.91986 upper=1.22173 effort=71.28 velocity=4.47 -> lower=-1.22173 upper=1.91986 effort=71.28 velocity=4.47
