Commit message: fixed urdf visualization and inertias

File: alex-models/alex_purdue_description/urdf/alex_purdue.leftUpperArm.urdf (robot description, URDF)
Before this commit: robot Alex, 5 links, 5 joints
Joints:
- joint LEFT_SHOULDER_X: origin xyz=0.0 0.01300000 0.11791000 rpy=-0.698132 0.0 0.0 -> xyz=0.0 0.01300000 0.11791000 rpy=0.698132 0.0 0.0
- joint LEFT_SHOULDER_Y: origin xyz=-0.00050000 0.12989023 0.38214403 rpy=0.698132 0.0 0.0 -> xyz=-0.00050000 0.12989023 0.38214403 rpy=-0.698132 0.0 0.0
- joint LEFT_SHOULDER_Z: origin xyz=0.0 0.03500000 -0.10400000 rpy=0.0 0.0 0.0 -> xyz=0.0 0.03500000 -0.10600000 rpy=0.0 0.0 0.0

File: alex-models/alex_purdue_description/urdf/alex_purdue.rightUpperArm.urdf (robot description, URDF)
Before this commit: robot Alex, 5 links, 5 joints
Joints:
- joint RIGHT_SHOULDER_X: origin xyz=0.0 -0.01300000 0.11791000 rpy=0.698132 0.0 0.0 -> xyz=0.0 -0.01300000 0.11791000 rpy=-0.698132 0.0 0.0
- joint RIGHT_SHOULDER_Y: origin xyz=-0.00050000 -0.12989023 0.38214403 rpy=-0.698132 0.0 0.0 -> xyz=-0.00050000 -0.12989023 0.38214403 rpy=0.698132 0.0 0.0

Commit message: fixed shoulder_y rotation issues

File: alex-models/alex_purdue_description/urdf/alex_purdue.leftUpperArm.urdf (robot description, URDF)
Before this commit: robot Alex, 5 links, 5 joints
Joints:
- joint LEFT_SHOULDER_Y: axis 0.0 1.0 0.0 -> 0.0 0.0 1.0

File: alex-models/alex_purdue_description/urdf/alex_purdue.rightUpperArm.urdf (robot description, URDF)
Before this commit: robot Alex, 5 links, 5 joints
Joints:
- joint RIGHT_SHOULDER_Y: axis 0.0 1.0 0.0 -> 0.0 0.0 1.0

Commit message: fixed shoulder y joints and added new decimated meshes

File: alex-models/alex_purdue_description/urdf/alex_purdue.leftUpperArm.urdf (robot description, URDF)
Before this commit: robot Alex, 5 links, 5 joints
Joints:
- joint LEFT_SHOULDER_X: limit lower=-0.261799 upper=2.87979 effort=160.7 velocity=10.38 -> lower=-0.349066 upper=2.79253 effort=160.7 velocity=10.38; origin xyz=0.0 0.01300000 0.11791000 rpy=0.872664626 0.0 0.0 -> xyz=0.0 0.11791000 -0.01300000 rpy=-0.698132 0.0 0.0
- joint LEFT_SHOULDER_Y: axis 0.0 0.0 1.0 -> 0.0 1.0 0.0; origin xyz=-0.00050000 0.12989023 0.38214403 rpy=-0.872664626 0.0 0.0 -> xyz=-0.00050000 0.12989023 0.38214403 rpy=0.698132 0.0 0.0

File: alex-models/alex_purdue_description/urdf/alex_purdue.rightUpperArm.urdf (robot description, URDF)
Before this commit: robot Alex, 5 links, 5 joints
Joints:
- joint RIGHT_SHOULDER_X: limit lower=-2.87979 upper=0.261799 effort=160.7 velocity=10.38 -> lower=-0.349066 upper=2.79253 effort=160.7 velocity=10.38; origin xyz=0.0 -0.01300000 0.11791000 rpy=-0.872664626 0.0 0.0 -> xyz=0.0 -0.11791000 -0.01300000 rpy=0.698132 0.0 0.0
- joint RIGHT_SHOULDER_Y: axis 0.0 0.0 1.0 -> 0.0 1.0 0.0; origin xyz=-0.00050000 -0.12989023 0.38214403 rpy=0.872664626 0.0 0.0 -> xyz=-0.00050000 -0.12989023 0.38214403 rpy=-0.698132 0.0 0.0
- joint RIGHT_SHOULDER_Z: limit lower=-1.22173 upper=1.91986 effort=71.28 velocity=4.47 -> lower=-1.91986 upper=1.22173 effort=71.28 velocity=4.47

Commit message: fixed joint limits in urdf

File: alex-models/alex_purdue_description/urdf/alex_purdue.leftUpperArm.urdf (robot description, URDF)
Before this commit: robot Alex, 5 links, 5 joints
Joints:
- joint LEFT_SHOULDER_X: limit lower=-0.349066 upper=2.79253 effort=160.7 velocity=10.38 -> lower=-0.261799 upper=2.87979 effort=160.7 velocity=10.38

File: alex-models/alex_purdue_description/urdf/alex_purdue.rightUpperArm.urdf (robot description, URDF)
Before this commit: robot Alex, 5 links, 5 joints
Joints:
- joint RIGHT_SHOULDER_X: limit lower=-0.349066 upper=2.79253 effort=160.7 velocity=10.38 -> lower=-2.87979 upper=0.261799 effort=160.7 velocity=10.38
- joint RIGHT_SHOULDER_Z: limit lower=-1.91986 upper=1.22173 effort=71.28 velocity=4.47 -> lower=-1.22173 upper=1.91986 effort=71.28 velocity=4.47

Commit message: fixed shoulder y joints and added new decimated meshes (#103)
* fixed shoulder y joints and added new decimated meshes

* fixed joint limits in urdf

---------

Co-authored-by: jaredihmc <jli@ihmc.org>
Co-authored-by: Alexander OCU <rosie@ihmc.org>

File: alex-models/alex_purdue_description/urdf/alex_purdue.leftUpperArm.urdf (robot description, URDF)
Before this commit: robot Alex, 5 links, 5 joints
Joints:
- joint LEFT_SHOULDER_X: origin xyz=0.0 0.01300000 0.11791000 rpy=0.872664626 0.0 0.0 -> xyz=0.0 0.11791000 -0.01300000 rpy=-0.698132 0.0 0.0
- joint LEFT_SHOULDER_Y: axis 0.0 0.0 1.0 -> 0.0 1.0 0.0; origin xyz=-0.00050000 0.12989023 0.38214403 rpy=-0.872664626 0.0 0.0 -> xyz=-0.00050000 0.12989023 0.38214403 rpy=0.698132 0.0 0.0

File: alex-models/alex_purdue_description/urdf/alex_purdue.rightUpperArm.urdf (robot description, URDF)
Before this commit: robot Alex, 5 links, 5 joints
Joints:
- joint RIGHT_SHOULDER_X: origin xyz=0.0 -0.01300000 0.11791000 rpy=-0.872664626 0.0 0.0 -> xyz=0.0 -0.11791000 -0.01300000 rpy=0.698132 0.0 0.0
- joint RIGHT_SHOULDER_Y: axis 0.0 0.0 1.0 -> 0.0 1.0 0.0; origin xyz=-0.00050000 -0.12989023 0.38214403 rpy=0.872664626 0.0 0.0 -> xyz=-0.00050000 -0.12989023 0.38214403 rpy=-0.698132 0.0 0.0
