Commit message: Adjust EZGripper adapter origin

File: alex-models/alex_purdue_description/urdf/alex_purdue.leftEZGripperAdapter.urdf (robot description, URDF)
Before this commit: robot Alex, 0 links, 1 joints
Joints:
- joint LEFT_EZGRIPPER_ADAPTER: origin xyz=0 0 -0.02 rpy=3.141592 1.570796 0 -> xyz=0 0 -0.0765 rpy=3.141592 1.570796 0

File: alex-models/alex_purdue_description/urdf/alex_purdue.rightEZGripperAdapter.urdf (robot description, URDF)
Before this commit: robot Alex, 0 links, 1 joints
Joints:
- joint RIGHT_EZGRIPPER_ADAPTER: origin xyz=0 0 -0.02 rpy=3.141592 1.570796 0 -> xyz=0 0 -0.0765 rpy=3.141592 1.570796 0
