Commit message: Fixed urdf files

File: alex-models/alex_purdue_description/urdf/alex_purdue.headTorso.urdf (robot description, URDF)
Before this commit: robot Alex, 5 links, 4 joints
Links:
- added link PEDESTAL_LINK, mass 0.72380912; visual mesh filename=package://alex_purdue_description/meshes/torso_head/pedesta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
- link TORSO_LINK: mass 15.84880155 -> 15.12587484
Joints:
- added joint PEDESTAL_F: type revolute, parent PEDESTAL_LINK, child TORSO_LINK, origin xyz=0 0 0 rpy=0 0 0, limit lower=0.0 upper=0.0 effort=0.0 velocity=0.0

File: alex-models/alex_purdue_description/urdf/alex_purdue.leftUpperArm.urdf (robot description, URDF)
Before this commit: robot Alex, 5 links, 5 joints
Joints:
- joint LEFT_SHOULDER_X: origin xyz=0.0 0.01300000 0.11791000 rpy=0.698132 0.0 0.0 -> xyz=0.0 0.01300000 0.11791000 rpy=0.872664626 0.0 0.0
- joint LEFT_SHOULDER_Y: origin xyz=-0.00050000 0.12989023 0.38214403 rpy=-0.698132 0.0 0.0 -> xyz=-0.00050000 0.12989023 0.38214403 rpy=-0.872664626 0.0 0.0

File: alex-models/alex_purdue_description/urdf/alex_purdue.rightUpperArm.urdf (robot description, URDF)
Before this commit: robot Alex, 5 links, 5 joints
Joints:
- joint RIGHT_SHOULDER_X: origin xyz=0.0 -0.01300000 0.11791000 rpy=-0.698132 0.0 0.0 -> xyz=0.0 -0.01300000 0.11791000 rpy=-0.872664626 0.0 0.0
- joint RIGHT_SHOULDER_Y: origin xyz=-0.00050000 -0.12989023 0.38214403 rpy=0.698132 0.0 0.0 -> xyz=-0.00050000 -0.12989023 0.38214403 rpy=0.872664626 0.0 0.0

Commit message: fixed things in purdue xmls and urdfs to get low-level process running

File: alex-models/alex_purdue_description/urdf/alex_purdue.headTorso.urdf (robot description, URDF)
Before this commit: robot Alex, 6 links, 5 joints
Links:
- added link TORSO_IMU_LINK, mass 0
Joints:
- added joint TORSO_IMU_JOINT: type fixed, parent TORSO_LINK, child TORSO_IMU_LINK, origin xyz=0.094766 0.018319 0.255014 rpy=-1.561264 -0.329453 -1.570796, axis 0 0 1

Commit message: purdue on rdx with legs

File: alex-models/alex_purdue_description/urdf/alex_purdue.headTorso.urdf (robot description, URDF)
Before this commit: robot Alex, 7 links, 6 joints
Joints:
- removed joint PEDESTAL_F
- added joint SPINE_Z: type revolute, parent PELVIS_LINK, child TORSO_LINK, origin xyz=0 0 0 rpy=0 0 0, limit lower=0.0 upper=0.0 effort=0.0 velocity=0.0

Commit message: fixed joint axis

File: alex-models/alex_purdue_description/urdf/alex_purdue.headTorso.urdf (robot description, URDF)
Before this commit: robot Alex, 7 links, 6 joints
Joints:
- joint PEDESTAL_F: origin xyz=0 0 0 rpy=0 0 0 -> xyz=0 0 1 rpy=0 0 0

Commit message: made pedestal urdf joint fixed

File: alex-models/alex_purdue_description/urdf/alex_purdue.headTorso.urdf (robot description, URDF)
Before this commit: robot Alex, 7 links, 6 joints
Joints:
- joint PEDESTAL_F: origin xyz=0 0 1 rpy=0 0 0 -> xyz=0 0 0 rpy=0 0 0; type revolute -> fixed
