Commit message: Shifted to a new structure

File: alex-models/alex_description/urdf/001/alex_v1.lowerBody.urdf (robot description, URDF)
Before this commit: robot Alex, 23 links, 22 joints
Links:
- link LEFT_ANKLE_Y_LINK: geometry visual mesh filename=package://alex_description/meshes/legs/AnklePitchLink.obj
- link LEFT_FOOT: geometry collision box size=0.22 0.1 0.02; visual mesh filename=package://alex_description/meshes/legs/Foot.obj
- link LEFT_HIP_X_LINK: geometry collision box size=0.02 0.12 0.10; visual mesh filename=package://alex_description/meshes/legs/LeftHipRollLink.obj
- link LEFT_HIP_Z_LINK: geometry visual mesh filename=package://alex_description/meshes/legs/LeftHipYawLink.obj
- link LEFT_SHIN: geometry collision capsule length=0.11 radius=0.065; collision capsule length=0.3 radius=0.06
- link LEFT_THIGH: geometry collision capsule length=0.26 radius=0.08; collision cylinder length=0.155 radius=0.03
- link PELVIS_LINK: geometry collision box size=0.15 0.10 0.12; visual mesh filename=package://alex_description/meshes/legs/Pelvis.obj
- link RIGHT_ANKLE_Y_LINK: geometry visual mesh filename=package://alex_description/meshes/legs/AnklePitchLink.obj
- link RIGHT_FOOT: geometry collision box size=0.22 0.1 0.02; visual mesh filename=package://alex_description/meshes/legs/Foot.obj
- link RIGHT_HIP_X_LINK: geometry collision box size=0.02 0.12 0.10; visual mesh filename=package://alex_description/meshes/legs/RightHipRollLink.obj
- link RIGHT_HIP_Z_LINK: geometry visual mesh filename=package://alex_description/meshes/legs/RightHipYawLink.obj
- link RIGHT_SHIN: geometry collision capsule length=0.11 radius=0.065; collision capsule length=0.3 radius=0.06
- link RIGHT_THIGH: geometry collision capsule length=0.26 radius=0.08; collision cylinder length=0.155 radius=0.03
- link TORSO_LINK: geometry collision box size=0.27 0.24 0.3; visual mesh filename=package://alex_description/meshes/V1/torso.obj
- link TORSO_ZED_X_MINI_LINK: geometry visual mesh filename=package://alex_description/meshes/ZEDXMini.obj
