Commit message: changed mesh directory in v1 urdfs

File: alex-models/alex_virtual_description/alex_v1_description/urdf/alex_v1.head.urdf (robot description, URDF)
Before this commit: robot Alex, 4 links, 4 joints
Links:
- link HEAD_LINK: geometry collision sphere radius=0.14; visual mesh filename=package://alex_virtual_description/alex_v1_description/mesh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
- link HEAD_ZED_X_MINI_LINK: geometry visual mesh filename=package://alex_virtual_description/alex_v1_description/mesh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

File: alex-models/alex_virtual_description/alex_v1_description/urdf/alex_v1.leftFixedForearm.urdf (robot description, URDF)
Before this commit: robot Alex, 1 links, 1 joints
Links:
- link LEFT_ELBOW_Y_LINK: geometry collision cylinder length=0.30 radius=0.04; visual mesh filename=package://alex_virtual_description/alex_v1_description/mesh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

File: alex-models/alex_virtual_description/alex_v1_description/urdf/alex_v1.leftForearm.urdf (robot description, URDF)
Before this commit: robot Alex, 6 links, 6 joints
Links:
- link LEFT_ELBOW_Y_LINK: geometry collision capsule length=0.18 radius=0.05; visual mesh filename=package://alex_virtual_description/alex_v1_description/mesh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
- link LEFT_GRIPPER_Z_LINK: geometry collision box size=0.08 0.025 0.075; collision capsule length=0.1 radius=0.04
- link LEFT_WRIST_X_LINK: geometry visual mesh filename=package://alex_virtual_description/alex_v1_description/mesh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
- link LEFT_WRIST_Z_LINK: geometry collision box size=0.01 0.06 0.1; collision cylinder length=0.12 radius=0.044

File: alex-models/alex_virtual_description/alex_v1_description/urdf/alex_v1.leftLongUpperArm.urdf (robot description, URDF)
Before this commit: robot Alex, 5 links, 5 joints
Links:
- link LEFT_SHOULDER_X_LINK: geometry visual mesh filename=package://alex_virtual_description/alex_v1_description/mesh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
- link LEFT_SHOULDER_Y_LINK: geometry visual mesh filename=package://alex_virtual_description/alex_v1_description/mesh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
- link LEFT_SHOULDER_Z_LINK: geometry visual mesh filename=package://alex_virtual_description/alex_v1_description/mesh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

File: alex-models/alex_virtual_description/alex_v1_description/urdf/alex_v1.leftNub.urdf (robot description, URDF)
Before this commit: robot Alex, 1 links, 1 joints
Links:
- link LEFT_NUB: geometry visual mesh filename=package://alex_virtual_description/alex_v1_description/mesh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

File: alex-models/alex_virtual_description/alex_v1_description/urdf/alex_v1.leftUpperArm.urdf (robot description, URDF)
Before this commit: robot Alex, 5 links, 5 joints
Links:
- link LEFT_SHOULDER_X_LINK: geometry visual mesh filename=package://alex_virtual_description/alex_v1_description/mesh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
- link LEFT_SHOULDER_Y_LINK: geometry visual mesh filename=package://alex_virtual_description/alex_v1_description/mesh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
- link LEFT_SHOULDER_Z_LINK: geometry collision cylinder length=0.22 radius=0.05; visual mesh filename=package://alex_virtual_description/alex_v1_description/mesh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

File: alex-models/alex_virtual_description/alex_v1_description/urdf/alex_v1.lowerBody.urdf (robot description, URDF)
Before this commit: robot Alex, 23 links, 22 joints
Links:
- link LEFT_ANKLE_Y_LINK: geometry visual mesh filename=package://alex_virtual_description/alex_v1_description/mesh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
- link LEFT_FOOT: geometry collision box size=0.22 0.1 0.02; visual mesh filename=package://alex_virtual_description/alex_v1_description/mesh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
- link LEFT_HIP_X_LINK: geometry collision box size=0.02 0.12 0.10; visual mesh filename=package://alex_virtual_description/alex_v1_description/mesh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
- link LEFT_HIP_Z_LINK: geometry visual mesh filename=package://alex_virtual_description/alex_v1_description/mesh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
- link LEFT_SHIN: geometry collision capsule length=0.11 radius=0.065; collision capsule length=0.3 radius=0.06
- link LEFT_THIGH: geometry collision capsule length=0.26 radius=0.08; collision cylinder length=0.155 radius=0.03
- link PELVIS_LINK: geometry collision box size=0.15 0.10 0.12; visual mesh filename=package://alex_virtual_description/alex_v1_description/mesh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
- link RIGHT_ANKLE_Y_LINK: geometry visual mesh filename=package://alex_virtual_description/alex_v1_description/mesh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
- link RIGHT_FOOT: geometry collision box size=0.22 0.1 0.02; visual mesh filename=package://alex_virtual_description/alex_v1_description/mesh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
- link RIGHT_HIP_X_LINK: geometry collision box size=0.02 0.12 0.10; visual mesh filename=package://alex_virtual_description/alex_v1_description/mesh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
- link RIGHT_HIP_Z_LINK: geometry visual mesh filename=package://alex_virtual_description/alex_v1_description/mesh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
- link RIGHT_SHIN: geometry collision capsule length=0.11 radius=0.065; collision capsule length=0.3 radius=0.06
- link RIGHT_THIGH: geometry collision capsule length=0.26 radius=0.08; collision cylinder length=0.155 radius=0.03
- link TORSO_LINK: geometry collision box size=0.27 0.24 0.3; visual mesh filename=package://alex_virtual_description/alex_v1_description/mesh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
- link TORSO_ZED_X_MINI_LINK: geometry visual mesh filename=package://alex_virtual_description/alex_v1_description/mesh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

File: alex-models/alex_virtual_description/alex_v1_description/urdf/alex_v1.miniFullBodyNubForearms.urdf (robot description, URDF)
Before this commit: robot Alex, 39 links, 38 joints
Links:
- link HEAD_LINK: geometry collision sphere radius=0.006500000000000001; visual mesh filename=package://alex_virtual_description/alex_v1_description/mesh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
- link LEFT_ANKLE_Y_LINK: geometry visual mesh filename=package://alex_virtual_description/alex_v1_description/mesh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
- link LEFT_ELBOW_Y_LINK: geometry collision cylinder length=0.017 radius=0.0016500000000000002; visual mesh filename=package://alex_virtual_description/alex_v1_description/mesh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
- link LEFT_FOOT: geometry collision box size=0.011000000000000001 0.005000000000000001 0.001; visual mesh filename=package://alex_virtual_description/alex_v1_description/mesh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
- link LEFT_HIP_X_LINK: geometry collision box size=0.001 0.006 0.005000000000000001; visual mesh filename=package://alex_virtual_description/alex_v1_description/mesh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
- link LEFT_HIP_Z_LINK: geometry visual mesh filename=package://alex_virtual_description/alex_v1_description/mesh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
- link LEFT_SHIN: geometry collision cylinder length=0.015 radius=0.004; visual mesh filename=package://alex_virtual_description/alex_v1_description/mesh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
- link LEFT_SHOULDER_X_LINK: geometry visual mesh filename=package://alex_virtual_description/alex_v1_description/mesh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
- link LEFT_SHOULDER_Y_LINK: geometry visual mesh filename=package://alex_virtual_description/alex_v1_description/mesh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
- link LEFT_SHOULDER_Z_LINK: geometry collision cylinder length=0.013000000000000001 radius=0.0025000000000000005; visual mesh filename=package://alex_virtual_description/alex_v1_description/mesh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
- link LEFT_THIGH: geometry collision box size=0.008 0.006500000000000001 0.014499999999999999; visual mesh filename=package://alex_virtual_description/alex_v1_description/mesh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
- link PELVIS_LINK: geometry collision box size=0.0075 0.005000000000000001 0.006; visual mesh filename=package://alex_virtual_description/alex_v1_description/mesh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
- link RIGHT_ANKLE_Y_LINK: geometry visual mesh filename=package://alex_virtual_description/alex_v1_description/mesh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
- link RIGHT_ELBOW_Y_LINK: geometry collision cylinder length=0.017 radius=0.0016500000000000002; visual mesh filename=package://alex_virtual_description/alex_v1_description/mesh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
- link RIGHT_FOOT: geometry collision box size=0.011000000000000001 0.005000000000000001 0.001; visual mesh filename=package://alex_virtual_description/alex_v1_description/mesh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
- link RIGHT_HIP_X_LINK: geometry collision box size=0.001 0.006 0.005000000000000001; visual mesh filename=package://alex_virtual_description/alex_v1_description/mesh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
- link RIGHT_HIP_Z_LINK: geometry visual mesh filename=package://alex_virtual_description/alex_v1_description/mesh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
- link RIGHT_SHIN: geometry collision cylinder length=0.015 radius=0.004; visual mesh filename=package://alex_virtual_description/alex_v1_description/mesh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
- link RIGHT_SHOULDER_X_LINK: geometry visual mesh filename=package://alex_virtual_description/alex_v1_description/mesh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
- link RIGHT_SHOULDER_Y_LINK: geometry visual mesh filename=package://alex_virtual_description/alex_v1_description/mesh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
- link RIGHT_SHOULDER_Z_LINK: geometry collision cylinder length=0.013000000000000001 radius=0.0025000000000000005; visual mesh filename=package://alex_virtual_description/alex_v1_description/mesh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
- link RIGHT_THIGH: geometry collision box size=0.008 0.006500000000000001 0.014499999999999999; visual mesh filename=package://alex_virtual_description/alex_v1_description/mesh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
- link TORSO_LINK: geometry collision box size=0.013750000000000002 0.0165 0.021500000000000002; visual mesh filename=package://alex_virtual_description/alex_v1_description/mesh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

File: alex-models/alex_virtual_description/alex_v1_description/urdf/alex_v1.mini_nubForearms.urdf (robot description, URDF)
Before this commit: robot Alex, 39 links, 38 joints
Links:
- link HEAD_LINK: geometry visual mesh filename=package://alex_virtual_description/alex_v1_description/mesh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
- link LEFT_ANKLE_Y_LINK: geometry visual mesh filename=package://alex_virtual_description/alex_v1_description/mesh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
- link LEFT_ELBOW_Y_LINK: geometry visual mesh filename=package://alex_virtual_description/alex_v1_description/mesh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
- link LEFT_FOOT: geometry collision box size=0.011 0.005 0.001; visual mesh filename=package://alex_virtual_description/alex_v1_description/mesh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
- link LEFT_HIP_X_LINK: geometry visual mesh filename=package://alex_virtual_description/alex_v1_description/mesh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
- link LEFT_HIP_Z_LINK: geometry visual mesh filename=package://alex_virtual_description/alex_v1_description/mesh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
- link LEFT_SHIN: geometry visual mesh filename=package://alex_virtual_description/alex_v1_description/mesh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
- link LEFT_SHOULDER_X_LINK: geometry visual mesh filename=package://alex_virtual_description/alex_v1_description/mesh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
- link LEFT_SHOULDER_Y_LINK: geometry visual mesh filename=package://alex_virtual_description/alex_v1_description/mesh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
- link LEFT_SHOULDER_Z_LINK: geometry visual mesh filename=package://alex_virtual_description/alex_v1_description/mesh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
- link LEFT_THIGH: geometry visual mesh filename=package://alex_virtual_description/alex_v1_description/mesh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
- link PELVIS_LINK: geometry collision box size=0.01 0.005 0.007; visual mesh filename=package://alex_virtual_description/alex_v1_description/mesh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
- link RIGHT_ANKLE_Y_LINK: geometry visual mesh filename=package://alex_virtual_description/alex_v1_description/mesh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
- link RIGHT_ELBOW_Y_LINK: geometry visual mesh filename=package://alex_virtual_description/alex_v1_description/mesh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
- link RIGHT_FOOT: geometry collision box size=0.011 0.005 0.001; visual mesh filename=package://alex_virtual_description/alex_v1_description/mesh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
- link RIGHT_HIP_X_LINK: geometry visual mesh filename=package://alex_virtual_description/alex_v1_description/mesh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
- link RIGHT_HIP_Z_LINK: geometry visual mesh filename=package://alex_virtual_description/alex_v1_description/mesh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
- link RIGHT_SHIN: geometry visual mesh filename=package://alex_virtual_description/alex_v1_description/mesh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
- link RIGHT_SHOULDER_X_LINK: geometry visual mesh filename=package://alex_virtual_description/alex_v1_description/mesh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
- link RIGHT_SHOULDER_Y_LINK: geometry visual mesh filename=package://alex_virtual_description/alex_v1_description/mesh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
- link RIGHT_SHOULDER_Z_LINK: geometry visual mesh filename=package://alex_virtual_description/alex_v1_description/mesh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
- link RIGHT_THIGH: geometry visual mesh filename=package://alex_virtual_description/alex_v1_description/mesh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
- link TORSO_LINK: geometry visual mesh filename=package://alex_virtual_description/alex_v1_description/mesh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

File: alex-models/alex_virtual_description/alex_v1_description/urdf/alex_v1.rightFixedForearm.urdf (robot description, URDF)
Before this commit: robot Alex, 1 links, 1 joints
Links:
- link RIGHT_ELBOW_Y_LINK: geometry collision cylinder length=0.30 radius=0.04; visual mesh filename=package://alex_virtual_description/alex_v1_description/mesh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

File: alex-models/alex_virtual_description/alex_v1_description/urdf/alex_v1.rightForearm.urdf (robot description, URDF)
Before this commit: robot Alex, 6 links, 6 joints
Links:
- link RIGHT_ELBOW_Y_LINK: geometry collision capsule length=0.18 radius=0.05; visual mesh filename=package://alex_virtual_description/alex_v1_description/mesh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
- link RIGHT_GRIPPER_Z_LINK: geometry collision box size=0.08 0.025 0.075; collision capsule length=0.1 radius=0.04
- link RIGHT_WRIST_X_LINK: geometry visual mesh filename=package://alex_virtual_description/alex_v1_description/mesh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
- link RIGHT_WRIST_Z_LINK: geometry collision box size=0.01 0.06 0.1; collision cylinder length=0.12 radius=0.044

File: alex-models/alex_virtual_description/alex_v1_description/urdf/alex_v1.rightLongUpperArm.urdf (robot description, URDF)
Before this commit: robot Alex, 5 links, 5 joints
Links:
- link RIGHT_SHOULDER_X_LINK: geometry visual mesh filename=package://alex_virtual_description/alex_v1_description/mesh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
- link RIGHT_SHOULDER_Y_LINK: geometry visual mesh filename=package://alex_virtual_description/alex_v1_description/mesh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
- link RIGHT_SHOULDER_Z_LINK: geometry visual mesh filename=package://alex_virtual_description/alex_v1_description/mesh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

File: alex-models/alex_virtual_description/alex_v1_description/urdf/alex_v1.rightNub.urdf (robot description, URDF)
Before this commit: robot Alex, 1 links, 1 joints
Links:
- link RIGHT_NUB: geometry visual mesh filename=package://alex_virtual_description/alex_v1_description/mesh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

File: alex-models/alex_virtual_description/alex_v1_description/urdf/alex_v1.rightUpperArm.urdf (robot description, URDF)
Before this commit: robot Alex, 5 links, 5 joints
Links:
- link RIGHT_SHOULDER_X_LINK: geometry visual mesh filename=package://alex_virtual_description/alex_v1_description/mesh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
- link RIGHT_SHOULDER_Y_LINK: geometry visual mesh filename=package://alex_virtual_description/alex_v1_description/mesh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
- link RIGHT_SHOULDER_Z_LINK: geometry collision cylinder length=0.22 radius=0.05; visual mesh filename=package://alex_virtual_description/alex_v1_description/mesh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
