Commit message: Fix JROS2 merge issues

File: alex-models/alex_virtual_description/alex_v2_description/urdf/alex_v2.leftFixedForearm_10lb.urdf (robot description, URDF)
Before this commit: robot Alex, 1 links, 1 joints
Links:
- link LEFT_ELBOW_Y_LINK: geometry collision cylinder length=0.30 radius=0.04; visual mesh filename=package://alex_virtual_description/alex_v1_description/mesh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

File: alex-models/alex_virtual_description/alex_v2_description/urdf/alex_v2.leftFixedForearm_5lb.urdf (robot description, URDF)
Before this commit: robot Alex, 1 links, 1 joints
Links:
- link LEFT_ELBOW_Y_LINK: geometry collision cylinder length=0.30 radius=0.04; visual mesh filename=package://alex_virtual_description/alex_v1_description/mesh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

File: alex-models/alex_virtual_description/alex_v2_description/urdf/alex_v2.leftFixedForearm_NoWeight.urdf (robot description, URDF)
Before this commit: robot Alex, 1 links, 1 joints
Links:
- link LEFT_ELBOW_Y_LINK: geometry collision cylinder length=0.30 radius=0.04; visual mesh filename=package://alex_virtual_description/alex_v1_description/mesh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

File: alex-models/alex_virtual_description/alex_v2_description/urdf/alex_v2.rightFixedForearm_10lb.urdf (robot description, URDF)
Before this commit: robot Alex, 1 links, 1 joints
Links:
- link RIGHT_ELBOW_Y_LINK: geometry collision cylinder length=0.30 radius=0.04; visual mesh filename=package://alex_virtual_description/alex_v1_description/mesh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

File: alex-models/alex_virtual_description/alex_v2_description/urdf/alex_v2.rightFixedForearm_5lb.urdf (robot description, URDF)
Before this commit: robot Alex, 1 links, 1 joints
Links:
- link RIGHT_ELBOW_Y_LINK: geometry collision cylinder length=0.30 radius=0.04; visual mesh filename=package://alex_virtual_description/alex_v1_description/mesh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

File: alex-models/alex_virtual_description/alex_v2_description/urdf/alex_v2.rightFixedForearm_NoWeight.urdf (robot description, URDF)
Before this commit: robot Alex, 1 links, 1 joints
Links:
- link RIGHT_ELBOW_Y_LINK: geometry collision cylinder length=0.30 radius=0.04; visual mesh filename=package://alex_virtual_description/alex_v1_description/mesh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
