Commit message: changed mesh directories in urdfs for v2

File: alex-models/alex_virtual_description/alex_v2_description/urdf/alex_v2.head.urdf (robot description, URDF)
Before this commit: robot Alex, 4 links, 4 joints
Links:
- link HEAD_LINK: geometry collision sphere radius=0.14; visual mesh filename=package://alex_virtual_description/alex_v2_description/mesh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
- link HEAD_ZED_X_MINI_LINK: geometry visual mesh filename=package://alex_virtual_description/alex_v1_description/mesh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
- link NECK_Z_LINK: geometry visual mesh filename=package://alex_virtual_description/alex_v2_description/mesh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

File: alex-models/alex_virtual_description/alex_v2_description/urdf/alex_v2.leftFixedForearm.urdf (robot description, URDF)
Before this commit: robot Alex, 1 links, 1 joints
Links:
- removed link RIGHT_ELBOW_Y_LINK
- added link LEFT_ELBOW_Y_LINK, mass 0.616; collision cylinder length=0.30 radius=0.04; visual mesh filename=package://alex_virtual_description/alex_v1_description/mesh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
Joints:
- removed joint RIGHT_ELBOW_Y
- added joint LEFT_ELBOW_Y: type revolute, parent LEFT_SHOULDER_Z_LINK, child LEFT_ELBOW_Y_LINK, origin xyz=0.015 0.0 -0.3127 rpy=0.0 0.0 0.0, axis 0.0 1.0 0.0, limit lower=-2.35619 upper=0.174533 effort=71.28 velocity=4.47

File: alex-models/alex_virtual_description/alex_v2_description/urdf/alex_v2.leftForearm.urdf (robot description, URDF)
Before this commit: robot Alex, 6 links, 6 joints
Links:
- removed link RIGHT_ELBOW_Y_LINK
- removed link RIGHT_GRIPPER_Z_IMU_LINK
- removed link RIGHT_GRIPPER_Z_LINK
- removed link RIGHT_WRIST_X_LINK
- removed link RIGHT_WRIST_Z_IMU_LINK
- removed link RIGHT_WRIST_Z_LINK
- added link LEFT_ELBOW_Y_LINK, mass 0.45; collision capsule length=0.18 radius=0.05; visual mesh filename=package://alex_virtual_description/alex_v1_description/mesh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
- added link LEFT_GRIPPER_Z_IMU_LINK, mass 0
- added link LEFT_GRIPPER_Z_LINK, mass 0.287; collision box size=0.08 0.025 0.075; collision capsule length=0.1 radius=0.04
- added link LEFT_WRIST_X_LINK, mass 0.909; visual mesh filename=package://alex_virtual_description/alex_v1_description/mesh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
- added link LEFT_WRIST_Z_IMU_LINK, mass 0
- added link LEFT_WRIST_Z_LINK, mass 1.547; collision box size=0.01 0.06 0.1; collision cylinder length=0.12 radius=0.044
Joints:
- removed joint RIGHT_ELBOW_Y
- removed joint RIGHT_GRIPPER_Z
- removed joint RIGHT_GRIPPER_Z_IMU_JOINT
- removed joint RIGHT_WRIST_X
- removed joint RIGHT_WRIST_Z
- removed joint RIGHT_WRIST_Z_IMU_JOINT
- added joint LEFT_ELBOW_Y: type revolute, parent LEFT_SHOULDER_Z_LINK, child LEFT_ELBOW_Y_LINK, origin xyz=0.015 0.0 -0.3127 rpy=0.0 0.0 0.0, axis 0.0 1.0 0.0, limit lower=-2.35619 upper=0.174533 effort=71.28 velocity=4.47
- added joint LEFT_GRIPPER_Z: type revolute, parent LEFT_WRIST_X_LINK, child LEFT_GRIPPER_Z_LINK, origin xyz=0.0 0.013 -0.031 rpy=0.0 0.0 0.0, axis 0.0 0.0 1.0, limit lower=-2.61799 upper=2.61799 effort=20.86 velocity=17.3
- added joint LEFT_GRIPPER_Z_IMU_JOINT: type fixed, parent LEFT_GRIPPER_Z_LINK, child LEFT_GRIPPER_Z_IMU_LINK, origin xyz=0 0 0 rpy=0 0 0, axis 0 0 1
- added joint LEFT_WRIST_X: type revolute, parent LEFT_WRIST_Z_LINK, child LEFT_WRIST_X_LINK, origin xyz=0.0 -0.013 -0.25 rpy=0.0 0.0 0.0, axis 1 0 0, limit lower=-1.8326 upper=0.610865 effort=20.86 velocity=17.3
- added joint LEFT_WRIST_Z: type revolute, parent LEFT_ELBOW_Y_LINK, child LEFT_WRIST_Z_LINK, origin xyz=-0.015 0.0 0.0 rpy=0.0 0.0 0.0, axis 0.0 0.0 1.0, limit lower=-2.61799 upper=2.61799 effort=20.86 velocity=17.3
- added joint LEFT_WRIST_Z_IMU_JOINT: type fixed, parent LEFT_WRIST_Z_LINK, child LEFT_WRIST_Z_IMU_LINK, origin xyz=-0.033554 0.010450 -0.148527 rpy=1.571 0.0 1.571, axis 0 0 1

File: alex-models/alex_virtual_description/alex_v2_description/urdf/alex_v2.leftUpperArm.urdf (robot description, URDF)
Before this commit: robot Alex, 5 links, 5 joints
Links:
- removed link RIGHT_SHOULDER_X_LINK
- removed link RIGHT_SHOULDER_Y_IMU_LINK
- removed link RIGHT_SHOULDER_Y_LINK
- removed link RIGHT_SHOULDER_Z_IMU_LINK
- removed link RIGHT_SHOULDER_Z_LINK
- added link LEFT_SHOULDER_X_LINK, mass 1.16159753; visual mesh filename=package://alex_virtual_description/alex_v1_description/mesh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
- added link LEFT_SHOULDER_Y_IMU_LINK, mass 0
- added link LEFT_SHOULDER_Y_LINK, mass 3.02036119; visual mesh filename=package://alex_virtual_description/alex_v1_description/mesh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
- added link LEFT_SHOULDER_Z_IMU_LINK, mass 0
- added link LEFT_SHOULDER_Z_LINK, mass 3.117556435; collision cylinder length=0.22 radius=0.05; visual mesh filename=package://alex_virtual_description/alex_v1_description/mesh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
Joints:
- removed joint RIGHT_SHOULDER_X
- removed joint RIGHT_SHOULDER_Y
- removed joint RIGHT_SHOULDER_Y_IMU_JOINT
- removed joint RIGHT_SHOULDER_Z
- removed joint RIGHT_SHOULDER_Z_IMU_JOINT
- added joint LEFT_SHOULDER_X: type revolute, parent LEFT_SHOULDER_Y_LINK, child LEFT_SHOULDER_X_LINK, origin xyz=0.0 0.15676000 -0.01300000 rpy=-0.698132 0.0 0.0, axis 1 0 0, limit lower=-0.349066 upper=2.79253 effort=160.7 velocity=10.38
- added joint LEFT_SHOULDER_Y: type revolute, parent TORSO_LINK, child LEFT_SHOULDER_Y_LINK, origin xyz=0.002 0.10350000 0.36000000 rpy=0.698132 0.0 0.0, axis 0.0 1.0 0.0, limit lower=-3.141592 upper=1.22173 effort=160.7 velocity=10.38
- added joint LEFT_SHOULDER_Y_IMU_JOINT: type fixed, parent LEFT_SHOULDER_Y_LINK, child LEFT_SHOULDER_Y_IMU_LINK, origin xyz=0.0174 0.06944 -0.03025 rpy=-1.570796 1.570796 0, axis 0 0 1
- added joint LEFT_SHOULDER_Z: type revolute, parent LEFT_SHOULDER_X_LINK, child LEFT_SHOULDER_Z_LINK, origin xyz=0.0 0.035 0.0 rpy=0.0 0.0 0.0, axis 0.0 0.0 1.0, limit lower=-1.91986 upper=1.22173 effort=71.28 velocity=4.47
- added joint LEFT_SHOULDER_Z_IMU_JOINT: type fixed, parent LEFT_SHOULDER_Z_LINK, child LEFT_SHOULDER_Z_IMU_LINK, origin xyz=-0.00763459 -0.0123324 -0.318 rpy=-1.570796 3.1415926 -0.314159, axis 0 0 1

File: alex-models/alex_virtual_description/alex_v2_description/urdf/alex_v2.lowerBody.urdf (robot description, URDF)
Before this commit: robot Alex, 23 links, 22 joints
Links:
- link LEFT_ANKLE_Y_LINK: geometry visual mesh filename=package://alex_virtual_description/alex_v1_description/mesh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
- link LEFT_FOOT: geometry collision box size=0.22 0.1 0.02; visual mesh filename=package://alex_virtual_description/alex_v1_description/mesh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
- link LEFT_HIP_X_LINK: geometry collision box size=0.02 0.12 0.10; visual mesh filename=package://alex_virtual_description/alex_v1_description/mesh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
- link LEFT_HIP_Z_LINK: geometry visual mesh filename=package://alex_virtual_description/alex_v1_description/mesh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
- link LEFT_SHIN: geometry collision capsule length=0.11 radius=0.065; collision capsule length=0.3 radius=0.06
- link LEFT_THIGH: geometry collision capsule length=0.26 radius=0.08; collision cylinder length=0.155 radius=0.03
- link PELVIS_LINK: geometry collision box size=0.15 0.10 0.12; visual mesh filename=package://alex_virtual_description/alex_v1_description/mesh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
- link RIGHT_ANKLE_Y_LINK: geometry visual mesh filename=package://alex_virtual_description/alex_v1_description/mesh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
- link RIGHT_FOOT: geometry collision box size=0.22 0.1 0.02; visual mesh filename=package://alex_virtual_description/alex_v1_description/mesh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
- link RIGHT_HIP_X_LINK: geometry collision box size=0.02 0.12 0.10; visual mesh filename=package://alex_virtual_description/alex_v1_description/mesh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
- link RIGHT_HIP_Z_LINK: geometry visual mesh filename=package://alex_virtual_description/alex_v1_description/mesh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
- link RIGHT_SHIN: geometry collision capsule length=0.11 radius=0.065; collision capsule length=0.3 radius=0.06
- link RIGHT_THIGH: geometry collision capsule length=0.26 radius=0.08; collision cylinder length=0.155 radius=0.03
- link TORSO_LINK: geometry collision box size=0.11 0.31 0.32; collision capsule length=0.25 radius=0.15
- link TORSO_ZED_X_MINI_LINK: geometry visual mesh filename=package://alex_virtual_description/alex_v1_description/mesh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

File: alex-models/alex_virtual_description/alex_v2_description/urdf/alex_v2.rightFixedForearm.urdf (robot description, URDF)
Before this commit: robot Alex, 1 links, 1 joints
Links:
- removed link LEFT_ELBOW_Y_LINK
- added link RIGHT_ELBOW_Y_LINK, mass 0.616; collision cylinder length=0.30 radius=0.04; visual mesh filename=package://alex_virtual_description/alex_v1_description/mesh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
Joints:
- removed joint LEFT_ELBOW_Y
- added joint RIGHT_ELBOW_Y: type revolute, parent RIGHT_SHOULDER_Z_LINK, child RIGHT_ELBOW_Y_LINK, origin xyz=0.015 0.0 -0.3127 rpy=0.0 0.0 0.0, axis 0.0 1.0 0.0, limit lower=-2.35619 upper=0.174533 effort=71.28 velocity=4.47

File: alex-models/alex_virtual_description/alex_v2_description/urdf/alex_v2.rightForearm.urdf (robot description, URDF)
Before this commit: robot Alex, 6 links, 6 joints
Links:
- removed link LEFT_ELBOW_Y_LINK
- removed link LEFT_GRIPPER_Z_IMU_LINK
- removed link LEFT_GRIPPER_Z_LINK
- removed link LEFT_WRIST_X_LINK
- removed link LEFT_WRIST_Z_IMU_LINK
- removed link LEFT_WRIST_Z_LINK
- added link RIGHT_ELBOW_Y_LINK, mass 0.45; collision capsule length=0.18 radius=0.05; visual mesh filename=package://alex_virtual_description/alex_v1_description/mesh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
- added link RIGHT_GRIPPER_Z_IMU_LINK, mass 0
- added link RIGHT_GRIPPER_Z_LINK, mass 0.287; collision box size=0.08 0.025 0.075; collision capsule length=0.1 radius=0.04
- added link RIGHT_WRIST_X_LINK, mass 0.909; visual mesh filename=package://alex_virtual_description/alex_v1_description/mesh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
- added link RIGHT_WRIST_Z_IMU_LINK, mass 0
- added link RIGHT_WRIST_Z_LINK, mass 1.547; collision box size=0.01 0.06 0.1; collision cylinder length=0.12 radius=0.044
Joints:
- removed joint LEFT_ELBOW_Y
- removed joint LEFT_GRIPPER_Z
- removed joint LEFT_GRIPPER_Z_IMU_JOINT
- removed joint LEFT_WRIST_X
- removed joint LEFT_WRIST_Z
- removed joint LEFT_WRIST_Z_IMU_JOINT
- added joint RIGHT_ELBOW_Y: type revolute, parent RIGHT_SHOULDER_Z_LINK, child RIGHT_ELBOW_Y_LINK, origin xyz=0.015 0.0 -0.3127 rpy=0.0 0.0 0.0, axis 0.0 1.0 0.0, limit lower=-2.35619 upper=0.174532925 effort=71.28 velocity=4.47
- added joint RIGHT_GRIPPER_Z: type revolute, parent RIGHT_WRIST_X_LINK, child RIGHT_GRIPPER_Z_LINK, origin xyz=0.0 -0.013 -0.031 rpy=0.0 0.0 0.0, axis 0.0 0.0 1.0, limit lower=-2.61799 upper=2.61799 effort=20.86 velocity=17.3
- added joint RIGHT_GRIPPER_Z_IMU_JOINT: type fixed, parent RIGHT_GRIPPER_Z_LINK, child RIGHT_GRIPPER_Z_IMU_LINK, origin xyz=0 0 0 rpy=0 0 0, axis 0 0 1
- added joint RIGHT_WRIST_X: type revolute, parent RIGHT_WRIST_Z_LINK, child RIGHT_WRIST_X_LINK, origin xyz=0.0 0.013 -0.25 rpy=0.0 0.0 0.0, axis 1 0 0, limit lower=-0.610865 upper=1.8326 effort=20.86 velocity=17.3
- added joint RIGHT_WRIST_Z: type revolute, parent RIGHT_ELBOW_Y_LINK, child RIGHT_WRIST_Z_LINK, origin xyz=-0.015 0.0 0.0 rpy=0.0 0.0 0.0, axis 0.0 0.0 1.0, limit lower=-2.61799 upper=2.61799 effort=20.86 velocity=17.3
- added joint RIGHT_WRIST_Z_IMU_JOINT: type fixed, parent RIGHT_WRIST_Z_LINK, child RIGHT_WRIST_Z_IMU_LINK, origin xyz=-0.033554 0.010450 -0.148527 rpy=1.571  0.0 1.571, axis 0 0 1

File: alex-models/alex_virtual_description/alex_v2_description/urdf/alex_v2.rightUpperArm.urdf (robot description, URDF)
Before this commit: robot Alex, 5 links, 5 joints
Links:
- removed link LEFT_SHOULDER_X_LINK
- removed link LEFT_SHOULDER_Y_IMU_LINK
- removed link LEFT_SHOULDER_Y_LINK
- removed link LEFT_SHOULDER_Z_IMU_LINK
- removed link LEFT_SHOULDER_Z_LINK
- added link RIGHT_SHOULDER_X_LINK, mass 1.16159753; visual mesh filename=package://alex_virtual_description/alex_v1_description/mesh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
- added link RIGHT_SHOULDER_Y_IMU_LINK, mass 0
- added link RIGHT_SHOULDER_Y_LINK, mass 3.02036119; visual mesh filename=package://alex_virtual_description/alex_v1_description/mesh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
- added link RIGHT_SHOULDER_Z_IMU_LINK, mass 0
- added link RIGHT_SHOULDER_Z_LINK, mass 3.117556435; collision cylinder length=0.22 radius=0.05; visual mesh filename=package://alex_virtual_description/alex_v1_description/mesh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
Joints:
- removed joint LEFT_SHOULDER_X
- removed joint LEFT_SHOULDER_Y
- removed joint LEFT_SHOULDER_Y_IMU_JOINT
- removed joint LEFT_SHOULDER_Z
- removed joint LEFT_SHOULDER_Z_IMU_JOINT
- added joint RIGHT_SHOULDER_X: type revolute, parent RIGHT_SHOULDER_Y_LINK, child RIGHT_SHOULDER_X_LINK, origin xyz=0.0 -0.15676000 -0.01300000 rpy=0.698132 0.0 0.0, axis 1 0 0, limit lower=-2.79253 upper=0.349066 effort=160.7 velocity=10.38
- added joint RIGHT_SHOULDER_Y: type revolute, parent TORSO_LINK, child RIGHT_SHOULDER_Y_LINK, origin xyz=0.002 -0.10350000 0.36000000 rpy=-0.698132 0.0 0.0, axis 0.0 1.0 0.0, limit lower=-3.141592 upper=1.22173 effort=160.7 velocity=10.38
- added joint RIGHT_SHOULDER_Y_IMU_JOINT: type fixed, parent RIGHT_SHOULDER_Y_LINK, child RIGHT_SHOULDER_Y_IMU_LINK, origin xyz=0.0175 -0.0704 -0.00778 rpy=1.570796 -1.570796 0, axis 0 0 1
- added joint RIGHT_SHOULDER_Z: type revolute, parent RIGHT_SHOULDER_X_LINK, child RIGHT_SHOULDER_Z_LINK, origin xyz=0.0 -0.035 0.0 rpy=0.0 0.0 0.0, axis 0.0 0.0 1.0, limit lower=-1.22173 upper=1.91986 effort=71.28 velocity=4.47
- added joint RIGHT_SHOULDER_Z_IMU_JOINT: type fixed, parent RIGHT_SHOULDER_Z_LINK, child RIGHT_SHOULDER_Z_IMU_LINK, origin xyz=0.002 0.016 -0.318 rpy=1.570796 0 0.314159, axis 0 0 1

Commit message: lowered neck joint effort limits in urdf down to 6Nm

File: alex-models/alex_virtual_description/alex_v2_description/urdf/alex_v2.head.urdf (robot description, URDF)
Before this commit: robot Alex, 4 links, 4 joints
Joints:
- joint NECK_Y: limit lower=-0.488692 upper=0.488692 effort=20.86 velocity=17.3 -> lower=-0.488692 upper=0.488692 effort=6.0 velocity=17.3
- joint NECK_Z: limit lower=-1.22173 upper=1.22173 effort=20.86 velocity=17.3 -> lower=-1.22173 upper=1.22173 effort=6.0 velocity=17.3
