Commit message: added new v2 feet meshes and edited v2 urdf

File: alex-models/alex_virtual_description/alex_v2_description/urdf/alex_v2.lowerBody.urdf (robot description, URDF)
Before this commit: robot Alex, 23 links, 22 joints
Links:
- link LEFT_FOOT: mass 0.810 -> 0.756; geometry collision box size=0.22 0.1 0.02; visual mesh filename=package://alex_virtual_description/alex_v2_description/mesh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
- link RIGHT_FOOT: mass 0.810 -> 0.756; geometry collision box size=0.22 0.1 0.02; visual mesh filename=package://alex_virtual_description/alex_v2_description/mesh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

Commit message: Added all the mesh's and updated the URDF's to get v2_description to be stand alone

File: alex-models/alex_virtual_description/alex_v2_description/urdf/alex_v2.lowerBody.urdf (robot description, URDF)
Before this commit: robot Alex, 23 links, 22 joints
Links:
- link LEFT_ANKLE_Y_LINK: geometry visual mesh filename=package://alex_virtual_description/alex_v2_description/mesh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
- link LEFT_FOOT: geometry collision box size=0.22 0.1 0.02; visual mesh filename=package://alex_virtual_description/alex_v2_description/mesh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
- link LEFT_HIP_X_LINK: geometry collision box size=0.02 0.12 0.10; visual mesh filename=package://alex_virtual_description/alex_v2_description/mesh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
- link LEFT_HIP_Z_LINK: geometry visual mesh filename=package://alex_virtual_description/alex_v2_description/mesh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
- link LEFT_SHIN: geometry collision capsule length=0.11 radius=0.065; collision capsule length=0.3 radius=0.06
- link LEFT_THIGH: geometry collision capsule length=0.26 radius=0.08; collision cylinder length=0.155 radius=0.03
- link PELVIS_LINK: geometry collision box size=0.15 0.10 0.12; visual mesh filename=package://alex_virtual_description/alex_v2_description/mesh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
- link RIGHT_ANKLE_Y_LINK: geometry visual mesh filename=package://alex_virtual_description/alex_v2_description/mesh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
- link RIGHT_FOOT: geometry collision box size=0.22 0.1 0.02; visual mesh filename=package://alex_virtual_description/alex_v2_description/mesh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
- link RIGHT_HIP_X_LINK: geometry collision box size=0.02 0.12 0.10; visual mesh filename=package://alex_virtual_description/alex_v2_description/mesh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
- link RIGHT_HIP_Z_LINK: geometry visual mesh filename=package://alex_virtual_description/alex_v2_description/mesh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
- link RIGHT_SHIN: geometry collision capsule length=0.11 radius=0.065; collision capsule length=0.3 radius=0.06
- link RIGHT_THIGH: geometry collision capsule length=0.26 radius=0.08; collision cylinder length=0.155 radius=0.03
- link TORSO_ZED_X_MINI_LINK: geometry visual mesh filename=package://alex_virtual_description/alex_v2_description/mesh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

File: alex-models/alex_virtual_description/alex_v2_description/urdf/alex_v2.lowerBody_convex.urdf (robot description, URDF)
Before this commit: robot Alex, 22 links, 21 joints
Links:
- link LEFT_ANKLE_Y_LINK: geometry visual mesh filename=package://alex_virtual_description/alex_v2_description/mesh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
- link LEFT_FOOT: geometry collision mesh filename=package://alex_virtual_description/alex_v2_description/mesh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; visual mesh filename=package://alex_virtual_description/alex_v2_description/mesh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
- link LEFT_HIP_X_LINK: geometry collision mesh filename=package://alex_virtual_description/alex_v2_description/mesh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; visual mesh filename=package://alex_virtual_description/alex_v2_description/mesh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
- link LEFT_HIP_Z_LINK: geometry visual mesh filename=package://alex_virtual_description/alex_v2_description/mesh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
- link LEFT_SHIN: geometry collision mesh filename=package://alex_virtual_description/alex_v2_description/mesh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; visual mesh filename=package://alex_virtual_description/alex_v2_description/mesh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
- link LEFT_THIGH: geometry collision mesh filename=package://alex_virtual_description/alex_v2_description/mesh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; visual mesh filename=package://alex_virtual_description/alex_v2_description/mesh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
- link PELVIS_LINK: geometry collision mesh filename=package://alex_virtual_description/alex_v2_description/mesh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; visual mesh filename=package://alex_virtual_description/alex_v2_description/mesh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
- link RIGHT_ANKLE_Y_LINK: geometry visual mesh filename=package://alex_virtual_description/alex_v2_description/mesh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
- link RIGHT_FOOT: geometry collision mesh filename=package://alex_virtual_description/alex_v2_description/mesh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; visual mesh filename=package://alex_virtual_description/alex_v2_description/mesh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
- link RIGHT_HIP_X_LINK: geometry collision mesh filename=package://alex_virtual_description/alex_v2_description/mesh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; visual mesh filename=package://alex_virtual_description/alex_v2_description/mesh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
- link RIGHT_HIP_Z_LINK: geometry visual mesh filename=package://alex_virtual_description/alex_v2_description/mesh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
- link RIGHT_SHIN: geometry collision mesh filename=package://alex_virtual_description/alex_v2_description/mesh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; visual mesh filename=package://alex_virtual_description/alex_v2_description/mesh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
- link RIGHT_THIGH: geometry collision mesh filename=package://alex_virtual_description/alex_v2_description/mesh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; visual mesh filename=package://alex_virtual_description/alex_v2_description/mesh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

Commit message: fixed mesh to be smaller and properly located

File: alex-models/alex_virtual_description/alex_v2_description/urdf/alex_v2.lowerBody.urdf (robot description, URDF)
Before this commit: robot Alex, 23 links, 22 joints
Links:
- link LEFT_FOOT: mass 0.756 -> 0.852
- link RIGHT_FOOT: mass 0.756 -> 0.852

Commit message: Feature/new feet urdf (#126)
* added new v2 feet meshes and edited v2 urdf

* forgot to add the meshes oof

* fixed mesh to be smaller and properly located

* Adjusted the foot collisions

* hands oddity

* rezero 001 right hip pitch

* Removed old edits

* Removed old comments

---------

Co-authored-by: Nikki Esposito <nesposito@ihmc.org>
Co-authored-by: ihmc-rosie <rosie@ihmc.org>

File: alex-models/alex_virtual_description/alex_v2_description/urdf/alex_v2.lowerBody.urdf (robot description, URDF)
Before this commit: robot Alex, 23 links, 22 joints
Links:
- link LEFT_FOOT: mass 0.810 -> 0.852
- link RIGHT_FOOT: mass 0.810 -> 0.852
