Commit message: convex feet and zed

File: alex-models/alex_virtual_description/alex_v2_description/urdf/alex_v2.lowerBody_convex.urdf (robot description, URDF)
Before this commit: robot Alex, 23 links, 22 joints
Links:
- link TORSO_ZED_X_MINI_LINK: geometry collision mesh filename=package://alex_virtual_description/alex_v2_description/mesh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; visual mesh filename=package://alex_virtual_description/alex_v2_description/mesh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
