Commit message: Adding meshes to Flappy Foot URDF model

File: alex-models/alex_virtual_description/alex_v2_description/urdf/alex_v2.lowerBody_flappyFoot.urdf (robot description, URDF)
Before this commit: robot Alex, 23 links, 22 joints
Links:
- link LEFT_FOOT_Y_INNER_LINK: geometry collision sphere radius=0.025; collision sphere radius=0.033
- link LEFT_FOOT_Y_OUTER_LINK: geometry collision sphere radius=0.025; visual mesh filename=package://alex_V2_description/meshes/LeftFlappyFootOuterLin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
- link RIGHT_FOOT_Y_INNER_LINK: geometry collision sphere radius=0.025; collision sphere radius=0.033
- link RIGHT_FOOT_Y_OUTER_LINK: geometry collision sphere radius=0.025; visual mesh filename=package://alex_V2_description/meshes/RightFlappyFootOuterLi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

Commit message: fixed mesh paths for flappy foot lower body urdf

File: alex-models/alex_virtual_description/alex_v2_description/urdf/alex_v2.lowerBody_flappyFoot.urdf (robot description, URDF)
Before this commit: robot Alex, 23 links, 22 joints
Links:
- link LEFT_FOOT_Y_INNER_LINK: geometry collision sphere radius=0.025; collision sphere radius=0.033
- link LEFT_FOOT_Y_OUTER_LINK: geometry collision sphere radius=0.025; visual mesh filename=package://alex_virtual_description/alex_v2_description/mesh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
- link LEFT_HIP_X_LINK: geometry collision box size=0.02 0.12 0.10; visual mesh filename=package://alex_virtual_description/alex_v2_description/mesh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
- link LEFT_HIP_Z_LINK: geometry visual mesh filename=package://alex_virtual_description/alex_v2_description/mesh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
- link LEFT_SHIN: geometry collision capsule length=0.11 radius=0.065; collision capsule length=0.3 radius=0.06
- link LEFT_THIGH: geometry collision capsule length=0.26 radius=0.08; collision cylinder length=0.155 radius=0.03
- link PELVIS_LINK: geometry collision box size=0.15 0.10 0.12; visual mesh filename=package://alex_virtual_description/alex_v2_description/mesh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
- link RIGHT_FOOT_Y_INNER_LINK: geometry collision sphere radius=0.025; collision sphere radius=0.033
- link RIGHT_FOOT_Y_OUTER_LINK: geometry collision sphere radius=0.025; visual mesh filename=package://alex_virtual_description/alex_v2_description/mesh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
- link RIGHT_HIP_X_LINK: geometry collision box size=0.02 0.12 0.10; visual mesh filename=package://alex_virtual_description/alex_v2_description/mesh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
- link RIGHT_HIP_Z_LINK: geometry visual mesh filename=package://alex_virtual_description/alex_v2_description/mesh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
- link RIGHT_SHIN: geometry collision capsule length=0.11 radius=0.065; collision capsule length=0.3 radius=0.06
- link RIGHT_THIGH: geometry collision capsule length=0.26 radius=0.08; collision cylinder length=0.155 radius=0.03
- link TORSO_LINK: geometry collision box size=0.11 0.31 0.32; collision capsule length=0.25 radius=0.15
- link TORSO_ZED_X_MINI_LINK: geometry visual mesh filename=package://alex_virtual_description/alex_v2_description/mesh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
