Commit message: fix forearm and hand collisions

File: alex-models/alex_virtual_description/alex_v2_description/urdf/alex_v2.leftForearm.urdf (robot description, URDF)
Before this commit: robot Alex, 6 links, 6 joints
Links:
- link LEFT_GRIPPER_Z_LINK: geometry visual mesh filename=package://alex_virtual_description/alex_v2_description/mesh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
- link LEFT_WRIST_X_LINK: geometry collision capsule length=0.03 radius=0.05; visual mesh filename=package://alex_virtual_description/alex_v2_description/mesh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

File: alex-models/alex_virtual_description/alex_v2_description/urdf/alex_v2.rightForearm.urdf (robot description, URDF)
Before this commit: robot Alex, 6 links, 6 joints
Links:
- link RIGHT_GRIPPER_Z_LINK: geometry visual mesh filename=package://alex_virtual_description/alex_v2_description/mesh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
- link RIGHT_WRIST_X_LINK: geometry collision capsule length=0.03 radius=0.05; visual mesh filename=package://alex_virtual_description/alex_v2_description/mesh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

Commit message: Re-adding removed hand collisions

File: alex-models/alex_virtual_description/alex_v2_description/urdf/alex_v2.leftForearm.urdf (robot description, URDF)
Before this commit: robot Alex, 6 links, 6 joints
Links:
- link LEFT_GRIPPER_Z_LINK: geometry collision capsule length=0.1 radius=0.04; visual mesh filename=package://alex_virtual_description/alex_v2_description/mesh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

File: alex-models/alex_virtual_description/alex_v2_description/urdf/alex_v2.rightForearm.urdf (robot description, URDF)
Before this commit: robot Alex, 6 links, 6 joints
Links:
- link RIGHT_GRIPPER_Z_LINK: geometry collision capsule length=0.1 radius=0.04; visual mesh filename=package://alex_virtual_description/alex_v2_description/mesh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

Commit message: Created hand stand-ins for training

File: alex-models/alex_virtual_description/alex_v2_description/urdf/alex_v2.leftForearm.urdf (robot description, URDF)
Before this commit: robot Alex, 6 links, 6 joints
Links:
- link LEFT_GRIPPER_Z_LINK: geometry visual mesh filename=package://alex_virtual_description/alex_v2_description/mesh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

File: alex-models/alex_virtual_description/alex_v2_description/urdf/alex_v2.rightForearm.urdf (robot description, URDF)
Before this commit: robot Alex, 6 links, 6 joints
Links:
- link RIGHT_GRIPPER_Z_LINK: geometry visual mesh filename=package://alex_virtual_description/alex_v2_description/mesh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

File: alex_description/urdf/alex_v2.wholeBody.urdf (robot description, URDF)
Before this commit: robot Alex, 49 links, 48 joints
Links:
- link LEFT_GRIPPER_Z_LINK: geometry visual mesh filename=package://alex_description/meshes/alex_v2/cycloidal_arm/Lef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
- link RIGHT_GRIPPER_Z_LINK: geometry visual mesh filename=package://alex_description/meshes/alex_v2/cycloidal_arm/Rig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

File: alex_description/urdf/alex_v2.wholeBody_abilityHands.urdf (robot description, URDF)
Before this commit: robot Alex, 141 links, 140 joints
Links:
- link LEFT_GRIPPER_Z_LINK: geometry visual mesh filename=package://alex_description/meshes/alex_v2/cycloidal_arm/Lef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
- link RIGHT_GRIPPER_Z_LINK: geometry visual mesh filename=package://alex_description/meshes/alex_v2/cycloidal_arm/Rig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
