Commit message: Put the correct capsule collisions

File: alex-models/alex_virtual_description/alex_v2_description/urdf/alex_v2.leftAbilityHandStandIn.urdf (robot description, URDF)
Before this commit: robot Alex, 1 links, 0 joints
Links:
- link left_ability_hand_base: geometry collision capsule length=0.1 radius=0.04; visual box size=0.157 0.053 0.184

File: alex-models/alex_virtual_description/alex_v2_description/urdf/alex_v2.rightAbilityHandStandIn.urdf (robot description, URDF)
Before this commit: robot Alex, 1 links, 0 joints
Links:
- link right_ability_hand_base: geometry collision capsule length=0.1 radius=0.04; visual box size=0.157 0.053 0.184

Commit message: Changed visual to match collision

File: alex-models/alex_virtual_description/alex_v2_description/urdf/alex_v2.leftAbilityHandStandIn.urdf (robot description, URDF)
Before this commit: robot Alex, 1 links, 0 joints
Links:
- link left_ability_hand_base: geometry collision capsule length=0.1 radius=0.04; visual capsule length=0.1 radius=0.04

File: alex-models/alex_virtual_description/alex_v2_description/urdf/alex_v2.rightAbilityHandStandIn.urdf (robot description, URDF)
Before this commit: robot Alex, 1 links, 0 joints
Links:
- link right_ability_hand_base: geometry collision capsule length=0.1 radius=0.04; visual capsule length=0.1 radius=0.04
