Commit message: Forgot to auto-generate models

File: alex_description/urdf/alex_v2.wholeBody.urdf (robot description, URDF)
Before this commit: robot Alex, 49 links, 48 joints
Links:
- link LEFT_GRIPPER_Z_LINK: geometry collision capsule length=0.1 radius=0.04; visual mesh filename=package://alex_description/meshes/alex_v2/cycloidal_arm/Lef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
- link LEFT_WRIST_X_LINK: geometry collision capsule length=0.03 radius=0.05; visual mesh filename=package://alex_description/meshes/alex_v2/cycloidal_arm/Lef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
- link RIGHT_GRIPPER_Z_LINK: geometry collision capsule length=0.1 radius=0.04; visual mesh filename=package://alex_description/meshes/alex_v2/cycloidal_arm/Rig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
- link RIGHT_WRIST_X_LINK: geometry collision capsule length=0.03 radius=0.05; visual mesh filename=package://alex_description/meshes/alex_v2/cycloidal_arm/Rig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
Joints:
- joint HEAD_IMU_JOINT: origin xyz=-0.02432603 -0.00225290 0.07425800 rpy=0.0 0.0 0.0 -> xyz=-0.02432603 -0.00225290 0.07425800 rpy=0.0 0.0 -1.5702
- joint LEFT_SHOULDER_Y_IMU_JOINT: origin xyz=0.0174 0.06944 -0.03025 rpy=-1.570796 1.570796 0 -> xyz=0.014320 0.079919 -0.002860 rpy=3.1415 0 -1.5702
- joint RIGHT_SHOULDER_Y_IMU_JOINT: origin xyz=0.0175 -0.0704 -0.00778 rpy=1.570796 -1.570796 0 -> xyz=0.014320 -0.104252 -0.002729 rpy=3.1415 0 -1.5702

File: alex_description/urdf/alex_v2.wholeBody_abilityHands.urdf (robot description, URDF)
Before this commit: robot Alex, 141 links, 140 joints
Links:
- link LEFT_GRIPPER_Z_LINK: geometry collision capsule length=0.1 radius=0.04; visual mesh filename=package://alex_description/meshes/alex_v2/cycloidal_arm/Lef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
- link LEFT_WRIST_X_LINK: geometry collision capsule length=0.03 radius=0.05; visual mesh filename=package://alex_description/meshes/alex_v2/cycloidal_arm/Lef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
- link RIGHT_GRIPPER_Z_LINK: geometry collision capsule length=0.1 radius=0.04; visual mesh filename=package://alex_description/meshes/alex_v2/cycloidal_arm/Rig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
- link RIGHT_WRIST_X_LINK: geometry collision capsule length=0.03 radius=0.05; visual mesh filename=package://alex_description/meshes/alex_v2/cycloidal_arm/Rig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
Joints:
- joint HEAD_IMU_JOINT: origin xyz=-0.02432603 -0.00225290 0.07425800 rpy=0.0 0.0 0.0 -> xyz=-0.02432603 -0.00225290 0.07425800 rpy=0.0 0.0 -1.5702
- joint LEFT_SHOULDER_Y_IMU_JOINT: origin xyz=0.0174 0.06944 -0.03025 rpy=-1.570796 1.570796 0 -> xyz=0.014320 0.079919 -0.002860 rpy=3.1415 0 -1.5702
- joint RIGHT_SHOULDER_Y_IMU_JOINT: origin xyz=0.0175 -0.0704 -0.00778 rpy=1.570796 -1.570796 0 -> xyz=0.014320 -0.104252 -0.002729 rpy=3.1415 0 -1.5702

File: alex_description/urdf/alex_v2.wholeBody_abilityHands_convex.urdf (robot description, URDF)
Before this commit: robot Alex, 141 links, 140 joints
Joints:
- joint HEAD_IMU_JOINT: origin xyz=-0.02432603 -0.00225290 0.07425800 rpy=0.0 0.0 0.0 -> xyz=-0.02432603 -0.00225290 0.07425800 rpy=0.0 0.0 -1.5702
- joint LEFT_SHOULDER_Y_IMU_JOINT: origin xyz=0.0174 0.06944 -0.03025 rpy=-1.570796 1.570796 0 -> xyz=0.014320 0.079919 -0.002860 rpy=3.1415 0 -1.5702
- joint RIGHT_SHOULDER_Y_IMU_JOINT: origin xyz=0.0175 -0.0704 -0.00778 rpy=1.570796 -1.570796 0 -> xyz=0.014320 -0.104252 -0.002729 rpy=3.1415 0 -1.5702

File: alex_description/urdf/alex_v2.wholeBody_convex.urdf (robot description, URDF)
Before this commit: robot Alex, 49 links, 48 joints
Joints:
- joint HEAD_IMU_JOINT: origin xyz=-0.02432603 -0.00225290 0.07425800 rpy=0.0 0.0 0.0 -> xyz=-0.02432603 -0.00225290 0.07425800 rpy=0.0 0.0 -1.5702
- joint LEFT_SHOULDER_Y_IMU_JOINT: origin xyz=0.0174 0.06944 -0.03025 rpy=-1.570796 1.570796 0 -> xyz=0.014320 0.079919 -0.002860 rpy=3.1415 0 -1.5702
- joint RIGHT_SHOULDER_Y_IMU_JOINT: origin xyz=0.0175 -0.0704 -0.00778 rpy=1.570796 -1.570796 0 -> xyz=0.014320 -0.104252 -0.002729 rpy=3.1415 0 -1.5702

Commit message: removed alex-models/alex_virtual_description and migrated everything into alex_description

File: alex_description/urdf/alex_v2.wholeBody.urdf (robot description, URDF)
Before this commit: robot Alex, 49 links, 48 joints
Links:
- link LEFT_GRIPPER_Z_LINK: geometry visual mesh filename=package://alex_description/meshes/alex_v2/cycloidal_arm/Lef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
- link LEFT_WRIST_X_LINK: geometry collision capsule length=0.03 radius=0.05; visual mesh filename=package://alex_description/meshes/alex_v2/cycloidal_arm/Lef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
- link RIGHT_GRIPPER_Z_LINK: geometry visual mesh filename=package://alex_description/meshes/alex_v2/cycloidal_arm/Rig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
- link RIGHT_WRIST_X_LINK: geometry collision capsule length=0.03 radius=0.05; visual mesh filename=package://alex_description/meshes/alex_v2/cycloidal_arm/Rig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
Joints:
- joint HEAD_IMU_JOINT: origin xyz=-0.02432603 -0.00225290 0.07425800 rpy=0.0 0.0 0.0 -> xyz=-0.02432603 -0.00225290 0.07425800 rpy=0.0 0.0 -1.5702
- joint LEFT_SHOULDER_Y_IMU_JOINT: origin xyz=0.0174 0.06944 -0.03025 rpy=-1.570796 1.570796 0 -> xyz=0.014320 0.079919 -0.002860 rpy=3.1415 0 -1.5702
- joint RIGHT_SHOULDER_Y_IMU_JOINT: origin xyz=0.0175 -0.0704 -0.00778 rpy=1.570796 -1.570796 0 -> xyz=0.014320 -0.104252 -0.002729 rpy=3.1415 0 -1.5702

File: alex_description/urdf/alex_v2.wholeBody_abilityHands.urdf (robot description, URDF)
Before this commit: robot Alex, 141 links, 140 joints
Links:
- link LEFT_GRIPPER_Z_LINK: geometry visual mesh filename=package://alex_description/meshes/alex_v2/cycloidal_arm/Lef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
- link LEFT_WRIST_X_LINK: geometry collision capsule length=0.03 radius=0.05; visual mesh filename=package://alex_description/meshes/alex_v2/cycloidal_arm/Lef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
- link RIGHT_GRIPPER_Z_LINK: geometry visual mesh filename=package://alex_description/meshes/alex_v2/cycloidal_arm/Rig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
- link RIGHT_WRIST_X_LINK: geometry collision capsule length=0.03 radius=0.05; visual mesh filename=package://alex_description/meshes/alex_v2/cycloidal_arm/Rig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
Joints:
- joint HEAD_IMU_JOINT: origin xyz=-0.02432603 -0.00225290 0.07425800 rpy=0.0 0.0 0.0 -> xyz=-0.02432603 -0.00225290 0.07425800 rpy=0.0 0.0 -1.5702
- joint LEFT_SHOULDER_Y_IMU_JOINT: origin xyz=0.0174 0.06944 -0.03025 rpy=-1.570796 1.570796 0 -> xyz=0.014320 0.079919 -0.002860 rpy=3.1415 0 -1.5702
- joint RIGHT_SHOULDER_Y_IMU_JOINT: origin xyz=0.0175 -0.0704 -0.00778 rpy=1.570796 -1.570796 0 -> xyz=0.014320 -0.104252 -0.002729 rpy=3.1415 0 -1.5702

File: alex_description/urdf/alex_v2.wholeBody_abilityHands_convex.urdf (robot description, URDF)
Before this commit: robot Alex, 141 links, 140 joints
Joints:
- joint HEAD_IMU_JOINT: origin xyz=-0.02432603 -0.00225290 0.07425800 rpy=0.0 0.0 0.0 -> xyz=-0.02432603 -0.00225290 0.07425800 rpy=0.0 0.0 -1.5702
- joint LEFT_SHOULDER_Y_IMU_JOINT: origin xyz=0.0174 0.06944 -0.03025 rpy=-1.570796 1.570796 0 -> xyz=0.014320 0.079919 -0.002860 rpy=3.1415 0 -1.5702
- joint RIGHT_SHOULDER_Y_IMU_JOINT: origin xyz=0.0175 -0.0704 -0.00778 rpy=1.570796 -1.570796 0 -> xyz=0.014320 -0.104252 -0.002729 rpy=3.1415 0 -1.5702

File: alex_description/urdf/alex_v2.wholeBody_convex.urdf (robot description, URDF)
Before this commit: robot Alex, 49 links, 48 joints
Joints:
- joint HEAD_IMU_JOINT: origin xyz=-0.02432603 -0.00225290 0.07425800 rpy=0.0 0.0 0.0 -> xyz=-0.02432603 -0.00225290 0.07425800 rpy=0.0 0.0 -1.5702
- joint LEFT_SHOULDER_Y_IMU_JOINT: origin xyz=0.0174 0.06944 -0.03025 rpy=-1.570796 1.570796 0 -> xyz=0.014320 0.079919 -0.002860 rpy=3.1415 0 -1.5702
- joint RIGHT_SHOULDER_Y_IMU_JOINT: origin xyz=0.0175 -0.0704 -0.00778 rpy=1.570796 -1.570796 0 -> xyz=0.014320 -0.104252 -0.002729 rpy=3.1415 0 -1.5702

Commit message: Re-adding removed hand collisions (#136)
* Re-adding removed hand collisions

* Forgot to auto-generate models

* Created hand stand-ins for training

* Put the correct capsule collisions

* Fixed the direction of the collision offset

* Changed visual to match collision

File: alex_description/urdf/alex_v2.wholeBody.urdf (robot description, URDF)
Before this commit: robot Alex, 49 links, 48 joints
Links:
- link LEFT_GRIPPER_Z_LINK: geometry visual mesh filename=package://alex_description/meshes/alex_v2/cycloidal_arm/Lef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
- link LEFT_WRIST_X_LINK: geometry collision capsule length=0.03 radius=0.05; visual mesh filename=package://alex_description/meshes/alex_v2/cycloidal_arm/Lef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
- link RIGHT_GRIPPER_Z_LINK: geometry visual mesh filename=package://alex_description/meshes/alex_v2/cycloidal_arm/Rig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
- link RIGHT_WRIST_X_LINK: geometry collision capsule length=0.03 radius=0.05; visual mesh filename=package://alex_description/meshes/alex_v2/cycloidal_arm/Rig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
Joints:
- joint HEAD_IMU_JOINT: origin xyz=-0.02432603 -0.00225290 0.07425800 rpy=0.0 0.0 0.0 -> xyz=-0.02432603 -0.00225290 0.07425800 rpy=0.0 0.0 -1.5702
- joint LEFT_SHOULDER_Y_IMU_JOINT: origin xyz=0.0174 0.06944 -0.03025 rpy=-1.570796 1.570796 0 -> xyz=0.014320 0.079919 -0.002860 rpy=3.1415 0 -1.5702
- joint RIGHT_SHOULDER_Y_IMU_JOINT: origin xyz=0.0175 -0.0704 -0.00778 rpy=1.570796 -1.570796 0 -> xyz=0.014320 -0.104252 -0.002729 rpy=3.1415 0 -1.5702

File: alex_description/urdf/alex_v2.wholeBody_abilityHands.urdf (robot description, URDF)
Before this commit: robot Alex, 141 links, 140 joints
Links:
- link LEFT_GRIPPER_Z_LINK: geometry visual mesh filename=package://alex_description/meshes/alex_v2/cycloidal_arm/Lef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
- link LEFT_WRIST_X_LINK: geometry collision capsule length=0.03 radius=0.05; visual mesh filename=package://alex_description/meshes/alex_v2/cycloidal_arm/Lef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
- link RIGHT_GRIPPER_Z_LINK: geometry visual mesh filename=package://alex_description/meshes/alex_v2/cycloidal_arm/Rig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
- link RIGHT_WRIST_X_LINK: geometry collision capsule length=0.03 radius=0.05; visual mesh filename=package://alex_description/meshes/alex_v2/cycloidal_arm/Rig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
Joints:
- joint HEAD_IMU_JOINT: origin xyz=-0.02432603 -0.00225290 0.07425800 rpy=0.0 0.0 0.0 -> xyz=-0.02432603 -0.00225290 0.07425800 rpy=0.0 0.0 -1.5702
- joint LEFT_SHOULDER_Y_IMU_JOINT: origin xyz=0.0174 0.06944 -0.03025 rpy=-1.570796 1.570796 0 -> xyz=0.014320 0.079919 -0.002860 rpy=3.1415 0 -1.5702
- joint RIGHT_SHOULDER_Y_IMU_JOINT: origin xyz=0.0175 -0.0704 -0.00778 rpy=1.570796 -1.570796 0 -> xyz=0.014320 -0.104252 -0.002729 rpy=3.1415 0 -1.5702
